File: Blank PCB/MS20-VCF.kicad_pcb (KiCad board)
At the start: 2 copper layers, 127.5 x 133 mm, 112 parts, among them J1 Conn_CircuitBoard, J10 Conn_CircuitBoard, J11 Conn_JackBoard, J12 Conn_JackBoard, J13 FilterCV2, J14 FilterIn2, J15 FilterOut2, J2 Conn_CircuitBoard, J3 Conn_JackBoard, J4 Conn_JackBoard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

Commit message: Finish ms20-VCF and create gerber files
Parts:
- removed H1, H2, H3, H4: MountingHole_Pad, Synth:Doepfer Mounting hole
Routing:
- net GND: vias 15 -> 8
- net (no net): vias 0 -> 7
Other:
- outline, holes or cut-outs redrawn
- board text removed: "JLCJLCJLCJLC"
