File: Blank PCB/Blank.kicad_pcb (KiCad board)
At the start: 2 copper layers, 127.5 x 133 mm, 108 parts, among them J1 Conn_CircuitBoard, J10 Conn_CircuitBoard, J11 Conn_JackBoard, J12 Conn_JackBoard, J13 FilterCV2, J14 FilterIn2, J15 FilterOut2, J2 Conn_CircuitBoard, J3 Conn_JackBoard, J4 Conn_JackBoard, J5 Power Input, J6 FilterCV1, J7 FilterIn1, J8 FilterOut1, J9 Conn_CircuitBoard, Q1 BC559, Q2 BC559, Q3 BC559, Q4 BC559, SW1 Hpass/Lpass Switch, SW2 Bandpass, SW3 Hpass/Lpass Switch, U1 LM13700, U2 TL072, U3 LM13700, U4 TL072

Commit message: finish snare + hihat
Parts:
- removed CUTCV1, CUTCV2, CUTOFF1, CUTOFF2, Res1, Res2: 100k, Potentiometer_THT:Potentiometer_Bourns_PTV09A-1_Single_Vertical
- removed D10, D11, D12, D13: 1N4148, Diode_THT:D_DO-35_SOD27_P7.62mm_Horizontal
- removed J10: Conn_CircuitBoard, Connector_PinSocket_2.54mm:PinSocket_1x06_P2.54mm_Vertical
- removed J11, J12: Conn_JackBoard, Connector_PinHeader_2.54mm:PinHeader_1x06_P2.54mm_Vertical
- removed J13: FilterCV2, Connector_Audio:Jack_3.5mm_QingPu_WQP-PJ398SM_Vertical_CircularHoles
- removed J14: FilterIn2, Connector_Audio:Jack_3.5mm_QingPu_WQP-PJ398SM_Vertical_CircularHoles
- removed J15: FilterOut2, Connector_Audio:Jack_3.5mm_QingPu_WQP-PJ398SM_Vertical_CircularHoles
- removed R22, R29, R42, R43: 1k, Resistor_THT:R_Axial_DIN0207_L6.3mm_D2.5mm_P10.16mm_Horizontal
- removed R23, R25, R33, R34: 470, Resistor_THT:R_Axial_DIN0207_L6.3mm_D2.5mm_P10.16mm_Horizontal
- removed R24, R27, R28, R32, R36, R37: 100k, Resistor_THT:R_Axial_DIN0207_L6.3mm_D2.5mm_P10.16mm_Horizontal
- removed R26, R30, R41: 2.2k, Resistor_THT:R_Axial_DIN0207_L6.3mm_D2.5mm_P10.16mm_Horizontal
- removed R31, R40: 1.8k, Resistor_THT:R_Axial_DIN0207_L6.3mm_D2.5mm_P10.16mm_Horizontal
- removed R35: 82k, Resistor_THT:R_Axial_DIN0207_L6.3mm_D2.5mm_P10.16mm_Horizontal
- removed R38: 33k, Resistor_THT:R_Axial_DIN0207_L6.3mm_D2.5mm_P10.16mm_Horizontal
- removed R39: 56k, Resistor_THT:R_Axial_DIN0207_L6.3mm_D2.5mm_P10.16mm_Horizontal
- removed ResLv1, ResLv2: 3.3k, Potentiometer_THT:Potentiometer_Bourns_3386C_Horizontal
- removed ResVol1, ResVol2: 10k, Potentiometer_THT:Potentiometer_Bourns_3386C_Horizontal
- removed SW1, SW3: Hpass/Lpass Switch, Synth:SW_DPDT_Toggle
- removed SW2: Bandpass, Synth:SW_Toggle_Blue_wSlots
- removed U2, U4: TL072, Package_DIP:DIP-8_W7.62mm_Socket
- removed U3: LM13700, Package_DIP:DIP-16_W7.62mm_Socket
- added C15: 10µF, Capacitor_THT:CP_Radial_D5.0mm_P2.00mm, F.Cu at (34.0, 94.5)
- added C16: 10µF, Capacitor_THT:CP_Radial_D5.0mm_P2.00mm, F.Cu at (39.5, 81.0)
- added C17: 1µF, Capacitor_THT:C_Disc_D7.0mm_W2.5mm_P5.00mm, F.Cu at (45.0, 132.0)
- added C18: 10nF, Capacitor_THT:C_Disc_D7.0mm_W2.5mm_P5.00mm, F.Cu at (45.0, 135.0)
- added C19: 680pF, Capacitor_THT:C_Disc_D7.0mm_W2.5mm_P5.00mm, F.Cu at (56.5, 69.0)
- added C20: .1µF, Capacitor_THT:C_Disc_D7.0mm_W2.5mm_P5.00mm, F.Cu at (66.5, 71.0)
- added C21: 10µF, Capacitor_THT:C_Disc_D7.0mm_W2.5mm_P5.00mm, F.Cu at (56.5, 66.0)
- added C22: 100µ, Capacitor_THT:CP_Radial_D5.0mm_P2.00mm, F.Cu at (46.5, 116.0)
- added C23: 100µ, Capacitor_THT:CP_Radial_D5.0mm_P2.00mm, F.Cu at (53.5, 116.0)
- added DECAY1: 100k, Potentiometer_THT:Potentiometer_Bourns_PTV09A-1_Single_Vertical, F.Cu at (106.5, 45.5)
- added DECAY2: 100k, Potentiometer_THT:Potentiometer_Bourns_PTV09A-1_Single_Vertical, F.Cu at (84.5, 45.5)
- added Depth1: SW_Push_DPDT, Synth:SW_DPDT_Toggle, F.Cu at (104.0, 90.0)
- added Depth2: SW_Push_DPDT, Synth:SW_DPDT_Toggle, F.Cu at (82.0, 90.0)
- added Q5: BC546, Package_TO_SOT_THT:TO-92_Inline, F.Cu at (36.5, 122.5)
- added Q6: BC546, Package_TO_SOT_THT:TO-92_Inline, F.Cu at (41.5, 122.5)
- added Q7: BC546, Package_TO_SOT_THT:TO-92_Inline, F.Cu at (41.5, 128.0)
- added Q8: 2N3904, Package_TO_SOT_THT:TO-92_Inline, F.Cu at (80.7, 101.0)
- added REF**: Doepfer Mounting hole, Synth:Doepfer Mounting hole, F.Cu at (148.5, 22.5)
- added REF**: Doepfer Mounting hole, Synth:Doepfer Mounting hole, F.Cu at (127.0, 22.5)
- added REF**: Doepfer Mounting hole, Synth:Doepfer Mounting hole, F.Cu at (126.5, 149.5)
- added REF**: Doepfer Mounting hole, Synth:Doepfer Mounting hole, F.Cu at (148.5, 149.5)
- added Strike1: 100k, Potentiometer_THT:Potentiometer_Bourns_PTV09A-1_Single_Vertical, F.Cu at (106.5, 61.5)
- added Strike2: 100k, Potentiometer_THT:Potentiometer_Bourns_PTV09A-1_Single_Vertical, F.Cu at (84.5, 61.5)
- added VOL1: 10k, Potentiometer_THT:Potentiometer_Bourns_PTV09A-1_Single_Vertical, F.Cu at (106.5, 77.5)
- added VOL2: 10k, Potentiometer_THT:Potentiometer_Bourns_PTV09A-1_Single_Vertical, F.Cu at (84.5, 77.5)
- C1, C11, C12: value 1nF -> 10µF
- C10: value 0.1µ -> .1µF; footprint Capacitor_THT:CP_Radial_D5.0mm_P2.00mm -> Capacitor_THT:C_Disc_D7.0mm_W2.5mm_P5.00mm
- C13: value 1nF -> 1µF
- C14: value 10µF -> 0.1µF; footprint Capacitor_THT:CP_Radial_D5.0mm_P2.00mm -> Capacitor_THT:C_Disc_D7.0mm_W2.5mm_P5.00mm
- C2: value 10µ -> 1µF; footprint Capacitor_THT:CP_Radial_D5.0mm_P2.00mm -> Capacitor_THT:C_Disc_D7.0mm_W2.5mm_P5.00mm
- C3: value 10µ -> 0.1µF; footprint Capacitor_THT:CP_Radial_D5.0mm_P2.00mm -> Capacitor_THT:C_Disc_D7.0mm_W2.5mm_P5.00mm
- C4: value 1nF -> 10µF; footprint Capacitor_THT:C_Disc_D7.0mm_W2.5mm_P5.00mm -> Capacitor_THT:CP_Radial_D5.0mm_P2.00mm
- C5: value 1nF -> 10µ; footprint Capacitor_THT:C_Disc_D7.0mm_W2.5mm_P5.00mm -> Capacitor_THT:CP_Radial_D5.0mm_P2.00mm
- C6: value 10µF -> 10µ
- C7: value 0.1µ -> 10µF
- C8: value 0.1µ -> 1µF; footprint Capacitor_THT:CP_Radial_D5.0mm_P2.00mm -> Capacitor_THT:C_Disc_D7.0mm_W2.5mm_P5.00mm
- C9: value 0.1µ -> 0.1µF; footprint Capacitor_THT:CP_Radial_D5.0mm_P2.00mm -> Capacitor_THT:C_Disc_D7.0mm_W2.5mm_P5.00mm
- D1: value LED-12V -> 1N4148; footprint LED_THT:LED_D4.0mm -> Diode_THT:D_DO-35_SOD27_P7.62mm_Horizontal
- D4: value 1N4148 -> LED-12V; footprint Diode_THT:D_DO-35_SOD27_P7.62mm_Horizontal -> LED_THT:LED_D4.0mm; moved to B.Cu
- D5: value 1N4148 -> Trig Snare; footprint Diode_THT:D_DO-35_SOD27_P7.62mm_Horizontal -> LED_THT:LED_D4.0mm
- D9: value 1N4148 -> Trig_HiHat; footprint Diode_THT:D_DO-35_SOD27_P7.62mm_Horizontal -> LED_THT:LED_D4.0mm
- J1: value Conn_CircuitBoard -> Snare IN; footprint Connector_PinSocket_2.54mm:PinSocket_1x06_P2.54mm_Vertical -> Connector_Audio:Jack_3.5mm_QingPu_WQP-PJ398SM_Vertical_CircularHoles
- J2: value Conn_CircuitBoard -> Power Input; footprint Connector_PinSocket_2.54mm:PinSocket_1x06_P2.54mm_Vertical -> Connector_PinHeader_2.54mm:PinHeader_2x05_P2.54mm_Vertical; moved to B.Cu
- J3: value Conn_JackBoard -> HiHat IN; footprint Connector_PinHeader_2.54mm:PinHeader_1x06_P2.54mm_Vertical -> Connector_Audio:Jack_3.5mm_QingPu_WQP-PJ398SM_Vertical_CircularHoles; moved to F.Cu
- J4: value Conn_JackBoard -> Snare OUT; footprint Connector_PinHeader_2.54mm:PinHeader_1x06_P2.54mm_Vertical -> Connector_Audio:Jack_3.5mm_QingPu_WQP-PJ398SM_Vertical_CircularHoles; moved to F.Cu
- J5: value Power Input -> Conn_01x08_Male; footprint Connector_PinHeader_2.54mm:PinHeader_2x05_P2.54mm_Vertical -> Connector_PinHeader_2.54mm:PinHeader_1x08_P2.54mm_Vertical; moved to F.Cu
- J6: value FilterCV1 -> Conn_01x08_Female; footprint Connector_Audio:Jack_3.5mm_QingPu_WQP-PJ398SM_Vertical_CircularHoles -> Connector_PinSocket_2.54mm:PinSocket_1x08_P2.54mm_Vertical; moved to B.Cu
- J7: value FilterIn1 -> Conn_01x08_Male; footprint Connector_Audio:Jack_3.5mm_QingPu_WQP-PJ398SM_Vertical_CircularHoles -> Connector_PinHeader_2.54mm:PinHeader_1x08_P2.54mm_Vertical
- J8: value FilterOut1 -> Conn_01x08_Female; footprint Connector_Audio:Jack_3.5mm_QingPu_WQP-PJ398SM_Vertical_CircularHoles -> Connector_PinSocket_2.54mm:PinSocket_1x08_P2.54mm_Vertical; moved to B.Cu
- J9: value Conn_CircuitBoard -> HiHat OUT; footprint Connector_PinSocket_2.54mm:PinSocket_1x06_P2.54mm_Vertical -> Connector_Audio:Jack_3.5mm_QingPu_WQP-PJ398SM_Vertical_CircularHoles
- Q1, Q2, Q3: value BC559 -> BC546
- Q4: value BC559 -> 2N3904
- R1, R12, R3: value 470 -> 4k7
- R10: value 1.8k -> 100k
- R11, R15, R7: value 100k -> 1M
- R13: value 470 -> 47k
- R14: value 82k -> 4k7
- R17: value 33k -> 1M
- R18: value 56k -> 6.8k
- R19: value 1.8k -> 1k
- R2: value 100k -> 47k
- R20, R5: value 2.2k -> 100k
- R21: value 1k -> 1M
- R4: value 2.2k -> 1M
- R6: value 100k -> 2.2k
- R8: value 1k -> 6.8k
- R9: value 2.2k -> 1k
- U1: value LM13700 -> TL072; footprint Package_DIP:DIP-16_W7.62mm_Socket -> Package_DIP:DIP-8_W7.62mm_Socket
- moved J1 83.0 mm to (104.0, 112.0)
- moved R13 82.1 mm to (36.5, 125.5), turned to 270 degrees
- moved R3 80.7 mm to (52.0, 120.0)
- moved R15 80.2 mm to (32.0, 119.5), turned to 270 degrees
- moved R9 79.2 mm to (99.5, 99.3), turned to 270 degrees
- moved Q4 78.4 mm to (102.7, 101.0), turned to 0 degrees
- moved D3 77.3 mm to (55.0, 127.6)
- moved D5 77.1 mm to (102.7, 106.5), turned to 0 degrees
- moved Q2 75.4 mm to (59.0, 123.0), turned to 90 degrees
- moved Q1 75.2 mm to (64.0, 123.0), turned to 90 degrees
- moved R16 73.5 mm to (86.5, 99.3), turned to 270 degrees
- moved R5 71.4 mm to (96.5, 99.3), turned to 270 degrees
- moved R14 70.2 mm to (48.0, 120.0), turned to 270 degrees
- moved C14 70.2 mm to (90.0, 83.5), turned to 270 degrees
- moved R2 68.9 mm to (64.0, 126.0), turned to 270 degrees
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Connections:
- C1 pad 1: Net-(C1-Pad1) -> /DeH
- C10 pad 1: Net-(C10-Pad1) -> /So
- C10 pad 2: -12V -> Net-(C10-Pad2)
- C11 pad 1: Net-(C11-Pad1) -> /HiDH
- C13 pad 1: Net-(C13-Pad1) -> /HiDH
- C13 pad 2: /Filtre2/HPass -> Net-(C13-Pad2)
- C14 pad 1: /Filtre2/Out1 -> /HiDH
- C2 pad 1: +12V -> /DeH
- C2 pad 2: GND -> Net-(C2-Pad2)
- C3 pad 1: GND -> /DeH
- C3 pad 2: -12V -> Net-(C3-Pad2)
- C4 pad 1: Net-(C4-Pad1) -> /SnI
- C5 pad 1: Net-(C5-Pad1) -> +12V
- C5 pad 2: /HPass -> GND
- C6 pad 1: /Out1 -> GND
- C6 pad 2: Net-(C6-Pad2) -> -12V
- C7 pad 1: +12V -> /SnH
- C7 pad 2: Net-(C7-Pad2) -> GND
- C8 pad 2: -12V -> Net-(C8-Pad2)
- C9 pad 1: +12V -> GND
- C9 pad 2: Net-(C9-Pad2) -> Net-(C8-Pad2)
- D1 pad 1: GND -> Net-(C4-Pad2)
- D1 pad 2: Net-(D1-Pad2) -> GND
- D2 pad 1: Net-(D2-Pad1) -> /SnH
- D2 pad 2: Net-(D2-Pad2) -> Net-(C4-Pad2)
- D3 pad 1: Net-(D2-Pad2) -> Net-(D3-Pad1)
- D3 pad 2: Net-(D3-Pad2) -> /So
- D4 pad 1: Net-(D4-Pad1) -> GND
- D4 pad 2: Net-(D2-Pad1) -> Net-(D4-Pad2)
- D5 pad 1: Net-(D3-Pad2) -> GND
- D6 pad 1: Net-(D6-Pad1) -> Net-(C15-Pad2)
- D6 pad 2: Net-(D4-Pad1) -> GND
- D7 pad 1: Net-(D5-Pad2) -> /HiH
- D7 pad 2: Net-(D6-Pad1) -> Net-(C15-Pad2)
- D8 pad 2: Net-(D8-Pad2) -> /Ho
- D9 pad 1: Net-(D8-Pad2) -> GND
- J2 pad 1: /ResOut -> Net-(FB1-Pad2)
- J2 pad 2: Net-(J2-Pad2) -> Net-(FB1-Pad2)
- J2 pad 3: -12V -> GND
- J2 pad 6: +12V -> GND
- J5 pad 1: Net-(FB1-Pad2) -> +12V
- J5 pad 2: Net-(FB1-Pad2) -> GND
- J5 pad 3: GND -> /SnI
- J5 pad 4: GND -> /SnH
- J5 pad 5: GND -> /SnO
- J5 pad 6: GND -> /So
- J5 pad 8: GND -> /DeH
- Q1 pad 2: GND -> Net-(Q1-Pad2)
- Q1 pad 3: Net-(Q1-Pad3) -> /DeH
- Q2 pad 1: Net-(C4-Pad2) -> Net-(C8-Pad1)
- Q2 pad 2: /Cutoff -> Net-(Q1-Pad2)
- Q2 pad 3: Net-(Q1-Pad3) -> GND
- Q3 pad 1: Net-(Q3-Pad1) -> Net-(D3-Pad1)
- Q3 pad 2: GND -> Net-(C8-Pad2)
- Q3 pad 3: Net-(Q3-Pad3) -> GND
- Q4 pad 1: Net-(C12-Pad2) -> Net-(D5-Pad2)
- Q4 pad 2: /Filtre2/Cutoff -> Net-(Q4-Pad2)
- Q4 pad 3: Net-(Q3-Pad3) -> Net-(Q4-Pad3)
- R1 pad 1: GND -> /SnI
- R1 pad 2: Net-(R1-Pad2) -> GND
- R10 pad 1: -12V -> Net-(C12-Pad1)
- R11 pad 1: Net-(R10-Pad2) -> /SnO
- R11 pad 2: Net-(R11-Pad2) -> Net-(C12-Pad2)
- R12 pad 1: GND -> /HiI
- R12 pad 2: Net-(R12-Pad2) -> GND
- R13 pad 1: GND -> /HiDH
- R13 pad 2: Net-(R11-Pad2) -> Net-(C17-Pad1)
- R14 pad 1: /Cutoff -> +12V
- R14 pad 2: Net-(CUTCV1-Pad2) -> Net-(C17-Pad1)
- R15 pad 1: /Cutoff -> +12V
- R16 pad 1: Net-(R12-Pad2) -> /HiH
- R16 pad 2: Net-(C6-Pad2) -> Net-(Q8-Pad2)
- R17 pad 1: Net-(CUTOFF1-Pad3) -> Net-(C20-Pad2)
- R17 pad 2: +12V -> GND
- R18 pad 1: -12V -> Net-(R18-Pad1)
- R18 pad 2: Net-(CUTOFF1-Pad1) -> GND
- R19 pad 1: -12V -> +12V
- R19 pad 2: Net-(C6-Pad2) -> Net-(Q8-Pad3)
- R2 pad 1: /LPass -> /DeH
- R2 pad 2: Net-(R2-Pad2) -> Net-(C8-Pad1)
- R20 pad 1: GND -> Net-(C21-Pad1)
- R20 pad 2: Net-(D6-Pad1) -> Net-(R18-Pad1)
- R21 pad 1: Net-(R21-Pad1) -> /HiO
- R21 pad 2: /Out1 -> Net-(C21-Pad2)
- R3 pad 1: GND -> +12V
- R3 pad 2: Net-(R2-Pad2) -> Net-(C8-Pad1)
- R4 pad 2: Net-(D1-Pad2) -> Net-(C8-Pad2)
- R5 pad 1: Net-(Q1-Pad1) -> /SnH
- R5 pad 2: Net-(R5-Pad2) -> Net-(Q4-Pad2)
- R6 pad 1: Net-(R1-Pad2) -> +12V
- R6 pad 2: Net-(R10-Pad2) -> Net-(D4-Pad2)
- R7 pad 1: -12V -> Net-(C10-Pad2)
- R7 pad 2: Net-(C4-Pad2) -> GND
- R8 pad 1: Net-(Q1-Pad3) -> Net-(R10-Pad2)
- R8 pad 2: Net-(C4-Pad1) -> GND
- R9 pad 1: GND -> +12V
- R9 pad 2: /Cutoff -> Net-(Q4-Pad3)
- U1 pad 1: Net-(R5-Pad2) -> Net-(C12-Pad1)
- U1 pad 2: Net-(U1-Pad2) -> Net-(R10-Pad2)
- U1 pad 3: Net-(R2-Pad2) -> Net-(C10-Pad2)
- U1 pad 4: Net-(R1-Pad2) -> -12V
- U1 pad 5: Net-(C1-Pad1) -> Net-(C20-Pad2)
- U1 pad 6: Net-(C8-Pad1) -> Net-(R18-Pad1)
- U1 pad 7: Net-(C1-Pad1) -> Net-(C21-Pad1)
- U1 pad 8: Net-(R10-Pad2) -> +12V
Routing:
- net -12V: track 206.2 -> 21.0 mm, vias 2 -> 0
- net /So: track 0.00 -> 130.1 mm
- net /Ho: track 0.00 -> 125.3 mm
- net /SnH: track 0.00 -> 111.1 mm
- net /HiH: track 0.00 -> 103.9 mm
- net /HiO: track 0.00 -> 94.1 mm
- net /Cutoff: track 85.7 -> 0.00 mm
- net /Filtre2/LPass: track 83.1 -> 0.00 mm
- net /SnO: track 0.00 -> 81.5 mm
- net Net-(R5-Pad2): track 79.4 -> 0.00 mm
- net /HPass: track 79.1 -> 0.00 mm
- net /Out1: track 77.4 -> 0.00 mm
- net Net-(J4-PadT): track 0.00 -> 74.4 mm
- net Net-(J9-PadT): track 0.00 -> 73.4 mm
- net Net-(R24-Pad2): track 71.8 -> 0.00 mm, vias 2 -> 0
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Other:
- outline, holes or cut-outs redrawn
- board text added: "JLCJLCJLCJLC"

Commit message: update blank
Routing:
- net (no net): vias 12 -> 14
Other:
- net class Default removed
- net class Power removed
