File: Drumbox/HiHat + Snare/CircuitBoard/Snare+Hihat.kicad_pcb (KiCad board)
At the start: 2 copper layers, 40 x 110 mm, 53 parts, among them J2 Power Input, J5 Conn_01x08_Male, J7 Conn_01x08_Male, Q1 BC546, Q2 BC546, Q3 BC546, Q5 BC546, Q6 BC546, Q7 BC546, U1 TL072

Commit message: gerber files for snare + hihat
Parts:
- removed C12, C21: 10µF, Capacitor_THT:C_Disc_D7.0mm_W2.5mm_P5.00mm
- removed C5, C6: 10µ, Capacitor_THT:CP_Radial_D5.0mm_P2.00mm
- removed R11, R21: 1M, Resistor_THT:R_Axial_DIN0207_L6.3mm_D2.5mm_P10.16mm_Horizontal
- removed R18: 6.8k, Resistor_THT:R_Axial_DIN0207_L6.3mm_D2.5mm_P10.16mm_Horizontal
- removed R20: 100k, Resistor_THT:R_Axial_DIN0207_L6.3mm_D2.5mm_P10.16mm_Horizontal
- removed U1: TL072, Package_DIP:DIP-8_W7.62mm_Socket
- added J11: Conn_01x03_Male, Connector_PinHeader_2.54mm:PinHeader_1x03_P2.54mm_Vertical, F.Cu at (52.5, 137.5)
- R10: value 100k -> 0R
- R8: value 6.8k -> 0R
- moved D4 107.5 mm to (34.9, 137.0), turned to 90 degrees
- moved J2 86.5 mm to (44.9, 130.0), turned to -90 degrees
- moved R6 76.9 mm to (34.0, 120.3), turned to -90 degrees
- moved FB2 69.2 mm to (60.5, 120.0), turned to -90 degrees
- moved FB1 69.1 mm to (39.5, 120.0), turned to -90 degrees
- moved R10 64.0 mm to (61.5, 114.5), turned to 180 degrees
- moved R8 54.6 mm to (38.8, 114.5), turned to 0 degrees
- moved R7 48.3 mm to (61.6, 108.0)
- moved C10 47.7 mm to (54.5, 111.2)
- moved R17 46.7 mm to (35.2, 104.5)
- moved C19 45.8 mm to (39.0, 111.2)
- moved C20 43.3 mm to (44.0, 108.0), turned to 180 degrees
- moved D3 39.4 mm to (55.0, 88.2)
- moved D8 39.4 mm to (45.0, 88.2)
- moved Q1 39.4 mm to (64.0, 83.6)
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Connections:
- C10 pad 2: Net-(C10-Pad2) -> /SnO
- C20 pad 2: Net-(C20-Pad2) -> /HiO
- J5 pad 1: +12V -> GND
- Q1 pad 1: Net-(Q1-Pad1) -> unconnected-(Q1-Pad1)
- Q5 pad 1: Net-(Q5-Pad1) -> unconnected-(Q5-Pad1)
- R10 pad 1: Net-(C12-Pad1) -> /SnO
- R10 pad 2: Net-(R10-Pad2) -> /So
- R17 pad 1: Net-(C20-Pad2) -> /HiO
- R7 pad 1: Net-(C10-Pad2) -> /SnO
- R8 pad 1: Net-(R10-Pad2) -> /HiO
- R8 pad 2: GND -> Net-(C19-Pad2)
Routing:
- net +12V: track 142.2 -> 112.0 mm
- net /Ho: track 69.9 -> 41.4 mm
- net /SnO: track 45.9 -> 17.8 mm
- net /DeH: track 12.6 -> 37.9 mm
- net /HiO: track 45.8 -> 20.8 mm
- net Net-(C12-Pad1): track 24.3 -> 0.00 mm
- net /So: track 73.8 -> 51.7 mm
- net /HiDH: track 14.8 -> 36.1 mm
- net /HiI: track 14.4 -> 35.4 mm
- net /HiH: track 31.3 -> 51.3 mm
- net /SnI: track 15.6 -> 34.2 mm
- net /SnH: track 32.6 -> 51.2 mm
- net Net-(R18-Pad1): track 14.9 -> 0.00 mm
- net Net-(C20-Pad2): track 14.5 -> 0.00 mm
- net Net-(C21-Pad1): track 14.1 -> 0.00 mm
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- added copper zone on F.Cu, net GND
Other:
- net class Default removed
- net class Power removed
- board text added: "8HP"
- board text added: "Board 1/2"
- board text added: "Snare + HiHat V1.0 BleepSound 2022"

Commit message: update each board
Parts:
- added C1: 10µF, Capacitor_THT:C_Disc_D7.0mm_W2.5mm_P5.00mm, F.Cu at (103.0, 80.5)
- added C11: 10µF, Capacitor_THT:C_Disc_D7.0mm_W2.5mm_P5.00mm, F.Cu at (80.0, 80.5)
- added C12: 10µF, Capacitor_THT:C_Disc_D7.0mm_W2.5mm_P5.00mm, F.Cu at (111.0, 121.0)
- added C13: 1µF, Capacitor_THT:C_Disc_D7.0mm_W2.5mm_P5.00mm, F.Cu at (83.0, 80.5)
- added C14: 0.1µF, Capacitor_THT:C_Disc_D7.0mm_W2.5mm_P5.00mm, F.Cu at (90.0, 83.5)
- added C2: 1µF, Capacitor_THT:C_Disc_D7.0mm_W2.5mm_P5.00mm, F.Cu at (105.5, 80.5)
- added C21: 10µF, Capacitor_THT:C_Disc_D7.0mm_W2.5mm_P5.00mm, F.Cu at (75.0, 121.0)
- added C3: 0.1µF, Capacitor_THT:C_Disc_D7.0mm_W2.5mm_P5.00mm, F.Cu at (96.0, 83.5)
- added C5: 10µ, Capacitor_THT:CP_Radial_D5.0mm_P2.00mm, F.Cu at (94.5, 129.5)
- added C6: 10µ, Capacitor_THT:CP_Radial_D5.0mm_P2.00mm, F.Cu at (90.0, 126.5)
- added D5: Trig Snare, LED_THT:LED_D4.0mm, F.Cu at (102.7, 106.5)
- added D9: Trig_HiHat, LED_THT:LED_D4.0mm, F.Cu at (80.7, 106.5)
- added DECAY1: 100k, Potentiometer_THT:Potentiometer_Bourns_PTV09A-1_Single_Vertical, F.Cu at (106.5, 45.5)
- added DECAY2: 100k, Potentiometer_THT:Potentiometer_Bourns_PTV09A-1_Single_Vertical, F.Cu at (84.5, 45.5)
- added Depth1: SW_Push_DPDT, Synth:SW_DPDT_Toggle, F.Cu at (104.0, 90.0)
- added Depth2: SW_Push_DPDT, Synth:SW_DPDT_Toggle, F.Cu at (82.0, 90.0)
- added J1: Snare IN, Connector_Audio:Jack_3.5mm_QingPu_WQP-PJ398SM_Vertical_CircularHoles, F.Cu at (104.0, 112.0)
- added J10: Conn_01x03_Female, Connector_PinSocket_2.54mm:PinSocket_1x03_P2.54mm_Vertical, B.Cu at (95.5, 137.5)
- added J3: HiHat IN, Connector_Audio:Jack_3.5mm_QingPu_WQP-PJ398SM_Vertical_CircularHoles, F.Cu at (82.0, 112.0)
- added J4: Snare OUT, Connector_Audio:Jack_3.5mm_QingPu_WQP-PJ398SM_Vertical_CircularHoles, F.Cu at (104.0, 126.6)
- added J6: Conn_01x08_Female, Connector_PinSocket_2.54mm:PinSocket_1x08_P2.54mm_Vertical, B.Cu at (111.0, 98.5)
- added J8: Conn_01x08_Female, Connector_PinSocket_2.54mm:PinSocket_1x08_P2.54mm_Vertical, B.Cu at (75.0, 98.5)
- added J9: HiHat OUT, Connector_Audio:Jack_3.5mm_QingPu_WQP-PJ398SM_Vertical_CircularHoles, F.Cu at (82.0, 126.6)
- added Q4: 2N3904, Package_TO_SOT_THT:TO-92_Inline, F.Cu at (102.7, 101.0)
- added Q8: 2N3904, Package_TO_SOT_THT:TO-92_Inline, F.Cu at (80.7, 101.0)
- added R11: 1k, Resistor_THT:R_Axial_DIN0207_L6.3mm_D2.5mm_P10.16mm_Horizontal, F.Cu at (111.0, 138.5)
- added R16: 100k, Resistor_THT:R_Axial_DIN0207_L6.3mm_D2.5mm_P10.16mm_Horizontal, F.Cu at (86.5, 99.3)
- added R19: 1k, Resistor_THT:R_Axial_DIN0207_L6.3mm_D2.5mm_P10.16mm_Horizontal, F.Cu at (89.5, 99.3)
- added R21: 1k, Resistor_THT:R_Axial_DIN0207_L6.3mm_D2.5mm_P10.16mm_Horizontal, F.Cu at (75.0, 138.6)
- added R5: 100k, Resistor_THT:R_Axial_DIN0207_L6.3mm_D2.5mm_P10.16mm_Horizontal, F.Cu at (96.5, 99.3)
- added R9: 1k, Resistor_THT:R_Axial_DIN0207_L6.3mm_D2.5mm_P10.16mm_Horizontal, F.Cu at (99.5, 99.3)
- added REF**: Doepfer Mounting hole, Synth:Doepfer Mounting hole, F.Cu at (150.0, 149.5)
- added REF**: Doepfer Mounting hole, Synth:Doepfer Mounting hole, F.Cu at (124.5, 22.5)
- added REF**: Doepfer Mounting hole, Synth:Doepfer Mounting hole, F.Cu at (150.0, 22.5)
- added REF**: Doepfer Mounting hole, Synth:Doepfer Mounting hole, F.Cu at (125.0, 149.5)
- added Strike1: 100k, Potentiometer_THT:Potentiometer_Bourns_PTV09A-1_Single_Vertical, F.Cu at (106.5, 61.5)
- added Strike2: 100k, Potentiometer_THT:Potentiometer_Bourns_PTV09A-1_Single_Vertical, F.Cu at (84.5, 61.5)
- added U1: TL072, Package_DIP:DIP-8_W7.62mm_Socket, F.Cu at (89.2, 113.2)
- added VOL1: 10k, Potentiometer_THT:Potentiometer_Bourns_PTV09A-1_Single_Vertical, F.Cu at (106.5, 77.5)
- added VOL2: 10k, Potentiometer_THT:Potentiometer_Bourns_PTV09A-1_Single_Vertical, F.Cu at (84.5, 77.5)
Routing:
- net /SnH: track 51.2 -> 130.1 mm
- net /HiH: track 51.3 -> 126.0 mm
- net /Ho: track 41.4 -> 107.9 mm
- net /So: track 51.7 -> 110.0 mm, vias 0 -> 1
- net Net-(VOL1-Pad2): track 0.00 -> 55.9 mm, vias 0 -> 1
- net Net-(VOL2-Pad2): track 0.00 -> 55.5 mm
- net /DeH: track 37.9 -> 92.7 mm
- net +12V: track 112.0 -> 162.4 mm
- net /HiDH: track 36.1 -> 83.6 mm
- net /SnO: track 17.8 -> 54.3 mm, vias 0 -> 1
- net /HiO: track 20.8 -> 56.0 mm
- net Net-(U1-Pad2): track 0.00 -> 26.5 mm
- net Net-(C21-Pad1): track 0.00 -> 25.5 mm
- net /HiI: track 35.4 -> 60.4 mm
- net /SnI: track 34.2 -> 58.9 mm
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Other:
- board size 40 x 110 mm -> 127.5 x 133 mm
- board text added: "Board 2/2"

Commit message: update gerber for all boards on hihat + snare
Parts:
- removed C1, C11, C12, C21: 10µF, Capacitor_THT:C_Disc_D7.0mm_W2.5mm_P5.00mm
- removed C13, C2: 1µF, Capacitor_THT:C_Disc_D7.0mm_W2.5mm_P5.00mm
- removed C14, C3: 0.1µF, Capacitor_THT:C_Disc_D7.0mm_W2.5mm_P5.00mm
- removed C5, C6: 10µ, Capacitor_THT:CP_Radial_D5.0mm_P2.00mm
- removed D5: Trig Snare, LED_THT:LED_D4.0mm
- removed D9: Trig_HiHat, LED_THT:LED_D4.0mm
- removed DECAY1, DECAY2, Strike1, Strike2: 100k, Potentiometer_THT:Potentiometer_Bourns_PTV09A-1_Single_Vertical
- removed Depth1, Depth2: SW_Push_DPDT, Synth:SW_DPDT_Toggle
- removed J1: Snare IN, Connector_Audio:Jack_3.5mm_QingPu_WQP-PJ398SM_Vertical_CircularHoles
- removed J10: Conn_01x03_Female, Connector_PinSocket_2.54mm:PinSocket_1x03_P2.54mm_Vertical
- removed J3: HiHat IN, Connector_Audio:Jack_3.5mm_QingPu_WQP-PJ398SM_Vertical_CircularHoles
- removed J4: Snare OUT, Connector_Audio:Jack_3.5mm_QingPu_WQP-PJ398SM_Vertical_CircularHoles
- removed J6, J8: Conn_01x08_Female, Connector_PinSocket_2.54mm:PinSocket_1x08_P2.54mm_Vertical
- removed J9: HiHat OUT, Connector_Audio:Jack_3.5mm_QingPu_WQP-PJ398SM_Vertical_CircularHoles
- removed Q4, Q8: 2N3904, Package_TO_SOT_THT:TO-92_Inline
- removed R11, R19, R21, R9: 1k, Resistor_THT:R_Axial_DIN0207_L6.3mm_D2.5mm_P10.16mm_Horizontal
- removed R16, R5: 100k, Resistor_THT:R_Axial_DIN0207_L6.3mm_D2.5mm_P10.16mm_Horizontal
- removed REF** (x4): Doepfer Mounting hole, Synth:Doepfer Mounting hole
- removed U1: TL072, Package_DIP:DIP-8_W7.62mm_Socket
- removed VOL1, VOL2: 10k, Potentiometer_THT:Potentiometer_Bourns_PTV09A-1_Single_Vertical
Routing:
- net /SnH: track 130.1 -> 51.2 mm
- net /HiH: track 126.0 -> 51.3 mm
- net /Ho: track 107.9 -> 41.4 mm
- net /So: track 110.0 -> 51.7 mm, vias 1 -> 0
- net Net-(VOL1-Pad2): track 55.9 -> 0.00 mm, vias 1 -> 0
- net Net-(VOL2-Pad2): track 55.5 -> 0.00 mm
- net /DeH: track 92.7 -> 37.9 mm
- net +12V: track 162.4 -> 112.0 mm
- net /HiDH: track 83.6 -> 36.1 mm
- net /SnO: track 54.3 -> 17.8 mm, vias 1 -> 0
- net /HiO: track 56.0 -> 20.8 mm
- net Net-(U1-Pad2): track 26.5 -> 0.00 mm
- net Net-(C21-Pad1): track 25.5 -> 0.00 mm
- net /HiI: track 60.4 -> 35.4 mm
- net /SnI: track 58.9 -> 34.2 mm
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Other:
- board size 127.5 x 133 mm -> 40 x 110 mm
- board text removed: "Board 2/2"
