File: Drumbox/HiHat + Snare/Front/Snare+Hihat.kicad_pcb (KiCad board)
At the start: 2 copper layers, 40 x 133 mm, 4 parts

Commit message: update each board
Parts:
- added C1: 10µF, Capacitor_THT:C_Disc_D7.0mm_W2.5mm_P5.00mm, F.Cu at (103.0, 80.5)
- added C10: .1µF, Capacitor_THT:C_Disc_D7.0mm_W2.5mm_P5.00mm, F.Cu at (54.5, 111.2)
- added C11: 10µF, Capacitor_THT:C_Disc_D7.0mm_W2.5mm_P5.00mm, F.Cu at (80.0, 80.5)
- added C12: 10µF, Capacitor_THT:C_Disc_D7.0mm_W2.5mm_P5.00mm, F.Cu at (111.0, 121.0)
- added C13: 1µF, Capacitor_THT:C_Disc_D7.0mm_W2.5mm_P5.00mm, F.Cu at (83.0, 80.5)
- added C14: 0.1µF, Capacitor_THT:C_Disc_D7.0mm_W2.5mm_P5.00mm, F.Cu at (90.0, 83.5)
- added C15: 10µF, Capacitor_THT:CP_Radial_D5.0mm_P2.00mm, F.Cu at (34.0, 74.5)
- added C16: 10µF, Capacitor_THT:CP_Radial_D5.0mm_P2.00mm, F.Cu at (39.5, 61.0)
- added C17: 1µF, Capacitor_THT:C_Disc_D7.0mm_W2.5mm_P5.00mm, F.Cu at (45.0, 92.6)
- added C18: 10nF, Capacitor_THT:C_Disc_D7.0mm_W2.5mm_P5.00mm, F.Cu at (45.0, 95.6)
- added C19: 680pF, Capacitor_THT:C_Disc_D7.0mm_W2.5mm_P5.00mm, F.Cu at (39.0, 111.2)
- added C2: 1µF, Capacitor_THT:C_Disc_D7.0mm_W2.5mm_P5.00mm, F.Cu at (105.5, 80.5)
- added C20: .1µF, Capacitor_THT:C_Disc_D7.0mm_W2.5mm_P5.00mm, F.Cu at (44.0, 108.0)
- added C21: 10µF, Capacitor_THT:C_Disc_D7.0mm_W2.5mm_P5.00mm, F.Cu at (75.0, 121.0)
- added C22: 100µ, Capacitor_THT:CP_Radial_D5.0mm_P2.00mm, F.Cu at (47.2, 99.2)
- added C23: 100µ, Capacitor_THT:CP_Radial_D5.0mm_P2.00mm, F.Cu at (53.0, 99.2)
- added C3: 0.1µF, Capacitor_THT:C_Disc_D7.0mm_W2.5mm_P5.00mm, F.Cu at (96.0, 83.5)
- added C4: 10µF, Capacitor_THT:CP_Radial_D5.0mm_P2.00mm, F.Cu at (60.8, 75.0)
- added C5: 10µ, Capacitor_THT:CP_Radial_D5.0mm_P2.00mm, F.Cu at (94.5, 129.5)
- added C6: 10µ, Capacitor_THT:CP_Radial_D5.0mm_P2.00mm, F.Cu at (90.0, 126.5)
- added C7: 10µF, Capacitor_THT:CP_Radial_D5.0mm_P2.00mm, F.Cu at (66.2, 61.5)
- added C8: 1µF, Capacitor_THT:C_Disc_D7.0mm_W2.5mm_P5.00mm, F.Cu at (55.0, 92.6)
- added C9: 0.1µF, Capacitor_THT:C_Disc_D7.0mm_W2.5mm_P5.00mm, F.Cu at (55.0, 95.6)
- added D1: 1N4148, Diode_THT:D_DO-35_SOD27_P7.62mm_Horizontal, F.Cu at (58.8, 70.0)
- added D2: 1N4148, Diode_THT:D_DO-35_SOD27_P7.62mm_Horizontal, F.Cu at (61.8, 62.4)
- added D3: 1N4148, Diode_THT:D_DO-35_SOD27_P7.62mm_Horizontal, F.Cu at (55.0, 88.2)
- added D4: LED-12V, LED_THT:LED_D4.0mm, B.Cu at (34.9, 137.0)
- added D5: Trig Snare, LED_THT:LED_D4.0mm, F.Cu at (102.7, 106.5)
- added D6: 1N4148, Diode_THT:D_DO-35_SOD27_P7.62mm_Horizontal, F.Cu at (32.5, 69.5)
- added D7: 1N4148, Diode_THT:D_DO-35_SOD27_P7.62mm_Horizontal, F.Cu at (35.0, 61.9)
- added D8: 1N4148, Diode_THT:D_DO-35_SOD27_P7.62mm_Horizontal, F.Cu at (45.0, 88.2)
- added D9: Trig_HiHat, LED_THT:LED_D4.0mm, F.Cu at (80.7, 106.5)
- added DECAY1: 100k, Potentiometer_THT:Potentiometer_Bourns_PTV09A-1_Single_Vertical, F.Cu at (106.5, 45.5)
- added DECAY2: 100k, Potentiometer_THT:Potentiometer_Bourns_PTV09A-1_Single_Vertical, F.Cu at (84.5, 45.5)
- added Depth1: SW_Push_DPDT, Synth:SW_DPDT_Toggle, F.Cu at (104.0, 90.0)
- added Depth2: SW_Push_DPDT, Synth:SW_DPDT_Toggle, F.Cu at (82.0, 90.0)
- added FB1: 10R, Inductor_THT:L_Axial_L9.5mm_D4.0mm_P12.70mm_Horizontal_Fastron_SMCC, F.Cu at (39.5, 120.0)
- added FB2: 10R, Inductor_THT:L_Axial_L9.5mm_D4.0mm_P12.70mm_Horizontal_Fastron_SMCC, F.Cu at (60.5, 120.0)
- added J1: Snare IN, Connector_Audio:Jack_3.5mm_QingPu_WQP-PJ398SM_Vertical_CircularHoles, F.Cu at (104.0, 112.0)
- added J10: Conn_01x03_Female, Connector_PinSocket_2.54mm:PinSocket_1x03_P2.54mm_Vertical, B.Cu at (95.5, 137.5)
- added J11: Conn_01x03_Male, Connector_PinHeader_2.54mm:PinHeader_1x03_P2.54mm_Vertical, F.Cu at (52.5, 137.5)
- added J2: Power Input, Connector_PinHeader_2.54mm:PinHeader_2x05_P2.54mm_Vertical, B.Cu at (44.9, 130.0)
- added J3: HiHat IN, Connector_Audio:Jack_3.5mm_QingPu_WQP-PJ398SM_Vertical_CircularHoles, F.Cu at (82.0, 112.0)
- added J4: Snare OUT, Connector_Audio:Jack_3.5mm_QingPu_WQP-PJ398SM_Vertical_CircularHoles, F.Cu at (104.0, 126.6)
- added J5: Conn_01x08_Male, Connector_PinHeader_2.54mm:PinHeader_1x08_P2.54mm_Vertical, F.Cu at (68.0, 98.5)
- added J6: Conn_01x08_Female, Connector_PinSocket_2.54mm:PinSocket_1x08_P2.54mm_Vertical, B.Cu at (111.0, 98.5)
- added J7: Conn_01x08_Male, Connector_PinHeader_2.54mm:PinHeader_1x08_P2.54mm_Vertical, F.Cu at (32.0, 98.5)
- added J8: Conn_01x08_Female, Connector_PinSocket_2.54mm:PinSocket_1x08_P2.54mm_Vertical, B.Cu at (75.0, 98.5)
- added J9: HiHat OUT, Connector_Audio:Jack_3.5mm_QingPu_WQP-PJ398SM_Vertical_CircularHoles, F.Cu at (82.0, 126.6)
- added Q1: BC546, Package_TO_SOT_THT:TO-92_Inline, F.Cu at (64.0, 83.6)
- added Q2: BC546, Package_TO_SOT_THT:TO-92_Inline, F.Cu at (59.0, 83.6)
- added Q3: BC546, Package_TO_SOT_THT:TO-92_Inline, F.Cu at (59.0, 89.1)
- added Q4: 2N3904, Package_TO_SOT_THT:TO-92_Inline, F.Cu at (102.7, 101.0)
- added Q5: BC546, Package_TO_SOT_THT:TO-92_Inline, F.Cu at (36.5, 83.1)
- added Q6: BC546, Package_TO_SOT_THT:TO-92_Inline, F.Cu at (41.5, 83.1)
- added Q7: BC546, Package_TO_SOT_THT:TO-92_Inline, F.Cu at (41.5, 88.6)
- added Q8: 2N3904, Package_TO_SOT_THT:TO-92_Inline, F.Cu at (80.7, 101.0)
- added R1: 4k7, Resistor_THT:R_Axial_DIN0207_L6.3mm_D2.5mm_P10.16mm_Horizontal, F.Cu at (65.2, 75.0)
- added R10: 0R, Resistor_THT:R_Axial_DIN0207_L6.3mm_D2.5mm_P10.16mm_Horizontal, F.Cu at (61.5, 114.5)
- added R11: 1k, Resistor_THT:R_Axial_DIN0207_L6.3mm_D2.5mm_P10.16mm_Horizontal, F.Cu at (111.0, 138.5)
- added R12: 4k7, Resistor_THT:R_Axial_DIN0207_L6.3mm_D2.5mm_P10.16mm_Horizontal, F.Cu at (38.5, 74.5)
- added R13: 47k, Resistor_THT:R_Axial_DIN0207_L6.3mm_D2.5mm_P10.16mm_Horizontal, F.Cu at (36.5, 86.1)
- added R14: 4k7, Resistor_THT:R_Axial_DIN0207_L6.3mm_D2.5mm_P10.16mm_Horizontal, F.Cu at (48.0, 80.6)
- added R15: 1M, Resistor_THT:R_Axial_DIN0207_L6.3mm_D2.5mm_P10.16mm_Horizontal, F.Cu at (35.8, 117.3)
- added R16: 100k, Resistor_THT:R_Axial_DIN0207_L6.3mm_D2.5mm_P10.16mm_Horizontal, F.Cu at (86.5, 99.3)
- added R17: 1M, Resistor_THT:R_Axial_DIN0207_L6.3mm_D2.5mm_P10.16mm_Horizontal, F.Cu at (35.2, 104.5)
- added R19: 1k, Resistor_THT:R_Axial_DIN0207_L6.3mm_D2.5mm_P10.16mm_Horizontal, F.Cu at (89.5, 99.3)
- added R2: 47k, Resistor_THT:R_Axial_DIN0207_L6.3mm_D2.5mm_P10.16mm_Horizontal, F.Cu at (64.0, 86.6)
- added R21: 1k, Resistor_THT:R_Axial_DIN0207_L6.3mm_D2.5mm_P10.16mm_Horizontal, F.Cu at (75.0, 138.6)
- added R3: 4k7, Resistor_THT:R_Axial_DIN0207_L6.3mm_D2.5mm_P10.16mm_Horizontal, F.Cu at (52.0, 80.6)
- added R4: 1M, Resistor_THT:R_Axial_DIN0207_L6.3mm_D2.5mm_P10.16mm_Horizontal, F.Cu at (64.2, 117.0)
- added R5: 100k, Resistor_THT:R_Axial_DIN0207_L6.3mm_D2.5mm_P10.16mm_Horizontal, F.Cu at (96.5, 99.3)
- added R6: 2.2k, Resistor_THT:R_Axial_DIN0207_L6.3mm_D2.5mm_P10.16mm_Horizontal, F.Cu at (34.0, 120.3)
- added R7: 1M, Resistor_THT:R_Axial_DIN0207_L6.3mm_D2.5mm_P10.16mm_Horizontal, F.Cu at (61.6, 108.0)
- added R8: 0R, Resistor_THT:R_Axial_DIN0207_L6.3mm_D2.5mm_P10.16mm_Horizontal, F.Cu at (38.8, 114.5)
- added R9: 1k, Resistor_THT:R_Axial_DIN0207_L6.3mm_D2.5mm_P10.16mm_Horizontal, F.Cu at (99.5, 99.3)
- added Strike1: 100k, Potentiometer_THT:Potentiometer_Bourns_PTV09A-1_Single_Vertical, F.Cu at (106.5, 61.5)
- added Strike2: 100k, Potentiometer_THT:Potentiometer_Bourns_PTV09A-1_Single_Vertical, F.Cu at (84.5, 61.5)
- added U1: TL072, Package_DIP:DIP-8_W7.62mm_Socket, F.Cu at (89.2, 113.2)
- added VOL1: 10k, Potentiometer_THT:Potentiometer_Bourns_PTV09A-1_Single_Vertical, F.Cu at (106.5, 77.5)
- added VOL2: 10k, Potentiometer_THT:Potentiometer_Bourns_PTV09A-1_Single_Vertical, F.Cu at (84.5, 77.5)
Routing:
- net +12V: track 0.00 -> 162.4 mm
- net /SnH: track 0.00 -> 130.1 mm
- net /HiH: track 0.00 -> 126.0 mm
- net /So: track 0.00 -> 110.0 mm, vias 0 -> 1
- net /Ho: track 0.00 -> 107.9 mm
- net /DeH: track 0.00 -> 92.7 mm
- net /HiDH: track 0.00 -> 83.6 mm
- net /HiI: track 0.00 -> 60.4 mm
- net /SnI: track 0.00 -> 58.9 mm
- net /HiO: track 0.00 -> 56.0 mm
- net Net-(VOL1-Pad2): track 0.00 -> 55.9 mm, vias 0 -> 1
- net Net-(VOL2-Pad2): track 0.00 -> 55.5 mm
- net /SnO: track 0.00 -> 54.3 mm, vias 0 -> 1
- net -12V: track 0.00 -> 51.9 mm
- net Net-(U1-Pad2): track 0.00 -> 26.5 mm
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- added copper zone on B.Cu, net GND
- added copper zone on F.Cu, net GND
Other:
- board size 40 x 133 mm -> 127.5 x 133 mm
- board text added: "8HP"
- board text added: "Board 1/2"
- board text added: "Board 2/2"
- board text added: "Snare + HiHat V1.0 BleepSound 2022"

Commit message: update gerber for all boards on hihat + snare
Parts:
- removed C1, C11, C12, C21: 10µF, Capacitor_THT:C_Disc_D7.0mm_W2.5mm_P5.00mm
- removed C10, C20: .1µF, Capacitor_THT:C_Disc_D7.0mm_W2.5mm_P5.00mm
- removed C13, C17, C2, C8: 1µF, Capacitor_THT:C_Disc_D7.0mm_W2.5mm_P5.00mm
- removed C14, C3, C9: 0.1µF, Capacitor_THT:C_Disc_D7.0mm_W2.5mm_P5.00mm
- removed C15, C16, C4, C7: 10µF, Capacitor_THT:CP_Radial_D5.0mm_P2.00mm
- removed C18: 10nF, Capacitor_THT:C_Disc_D7.0mm_W2.5mm_P5.00mm
- removed C19: 680pF, Capacitor_THT:C_Disc_D7.0mm_W2.5mm_P5.00mm
- removed C22, C23: 100µ, Capacitor_THT:CP_Radial_D5.0mm_P2.00mm
- removed C5, C6: 10µ, Capacitor_THT:CP_Radial_D5.0mm_P2.00mm
- removed D1, D2, D3, D6, D7, D8: 1N4148, Diode_THT:D_DO-35_SOD27_P7.62mm_Horizontal
- removed D4: LED-12V, LED_THT:LED_D4.0mm
- removed D5: Trig Snare, LED_THT:LED_D4.0mm
- removed D9: Trig_HiHat, LED_THT:LED_D4.0mm
- removed DECAY1, DECAY2, Strike1, Strike2: 100k, Potentiometer_THT:Potentiometer_Bourns_PTV09A-1_Single_Vertical
- removed Depth1, Depth2: SW_Push_DPDT, Synth:SW_DPDT_Toggle
- removed FB1, FB2: 10R, Inductor_THT:L_Axial_L9.5mm_D4.0mm_P12.70mm_Horizontal_Fastron_SMCC
- removed J1: Snare IN, Connector_Audio:Jack_3.5mm_QingPu_WQP-PJ398SM_Vertical_CircularHoles
- removed J10: Conn_01x03_Female, Connector_PinSocket_2.54mm:PinSocket_1x03_P2.54mm_Vertical
- removed J11: Conn_01x03_Male, Connector_PinHeader_2.54mm:PinHeader_1x03_P2.54mm_Vertical
- removed J2: Power Input, Connector_PinHeader_2.54mm:PinHeader_2x05_P2.54mm_Vertical
- removed J3: HiHat IN, Connector_Audio:Jack_3.5mm_QingPu_WQP-PJ398SM_Vertical_CircularHoles
- removed J4: Snare OUT, Connector_Audio:Jack_3.5mm_QingPu_WQP-PJ398SM_Vertical_CircularHoles
- removed J5, J7: Conn_01x08_Male, Connector_PinHeader_2.54mm:PinHeader_1x08_P2.54mm_Vertical
- removed J6, J8: Conn_01x08_Female, Connector_PinSocket_2.54mm:PinSocket_1x08_P2.54mm_Vertical
- removed J9: HiHat OUT, Connector_Audio:Jack_3.5mm_QingPu_WQP-PJ398SM_Vertical_CircularHoles
- removed Q1, Q2, Q3, Q5, Q6, Q7: BC546, Package_TO_SOT_THT:TO-92_Inline
- removed Q4, Q8: 2N3904, Package_TO_SOT_THT:TO-92_Inline
- removed R1, R12, R14, R3: 4k7, Resistor_THT:R_Axial_DIN0207_L6.3mm_D2.5mm_P10.16mm_Horizontal
- removed R10, R8: 0R, Resistor_THT:R_Axial_DIN0207_L6.3mm_D2.5mm_P10.16mm_Horizontal
- removed R11, R19, R21, R9: 1k, Resistor_THT:R_Axial_DIN0207_L6.3mm_D2.5mm_P10.16mm_Horizontal
- removed R13, R2: 47k, Resistor_THT:R_Axial_DIN0207_L6.3mm_D2.5mm_P10.16mm_Horizontal
- removed R15, R17, R4, R7: 1M, Resistor_THT:R_Axial_DIN0207_L6.3mm_D2.5mm_P10.16mm_Horizontal
- removed R16, R5: 100k, Resistor_THT:R_Axial_DIN0207_L6.3mm_D2.5mm_P10.16mm_Horizontal
- removed R6: 2.2k, Resistor_THT:R_Axial_DIN0207_L6.3mm_D2.5mm_P10.16mm_Horizontal
- removed U1: TL072, Package_DIP:DIP-8_W7.62mm_Socket
- removed VOL1, VOL2: 10k, Potentiometer_THT:Potentiometer_Bourns_PTV09A-1_Single_Vertical
Routing:
- net +12V: track 162.4 -> 0.00 mm
- net /SnH: track 130.1 -> 0.00 mm
- net /HiH: track 126.0 -> 0.00 mm
- net /So: track 110.0 -> 0.00 mm, vias 1 -> 0
- net /Ho: track 107.9 -> 0.00 mm
- net /DeH: track 92.7 -> 0.00 mm
- net /HiDH: track 83.6 -> 0.00 mm
- net /HiI: track 60.4 -> 0.00 mm
- net /SnI: track 58.9 -> 0.00 mm
- net /HiO: track 56.0 -> 0.00 mm
- net Net-(VOL1-Pad2): track 55.9 -> 0.00 mm, vias 1 -> 0
- net Net-(VOL2-Pad2): track 55.5 -> 0.00 mm
- net /SnO: track 54.3 -> 0.00 mm, vias 1 -> 0
- net -12V: track 51.9 -> 0.00 mm
- net Net-(U1-Pad2): track 26.5 -> 0.00 mm
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- removed copper zone on B.Cu, net GND
- removed copper zone on F.Cu, net GND
Other:
- board size 127.5 x 133 mm -> 40 x 133 mm
- board text removed: "8HP"
- board text removed: "Board 1/2"
- board text removed: "Board 2/2"
- board text removed: "Snare + HiHat V1.0 BleepSound 2022"
