File: MS20-VCF/Front/MS20-VCF.kicad_pcb (KiCad board)
At the start: 2 copper layers, 40 x 133 mm, 4 parts

Commit message: Update gerber MS20-VCF
Routing:
- removed copper zone on B.Cu, net GND
Other:
- net class Default removed
- net class Power removed

Commit message: update bom + gerber for jackboard
Parts:
- added C1: 1nF, Capacitor_THT:C_Disc_D7.0mm_W2.5mm_P5.00mm, F.Cu at (66.5, 83.5)
- added C10: 0.1µ, Capacitor_THT:CP_Radial_D5.0mm_P2.00mm, F.Cu at (81.5, 126.0)
- added C11: 1nF, Capacitor_THT:C_Disc_D7.0mm_W2.5mm_P5.00mm, F.Cu at (64.5, 103.0)
- added C12: 1nF, Capacitor_THT:C_Disc_D7.0mm_W2.5mm_P5.00mm, F.Cu at (69.5, 107.5)
- added C13: 1nF, Capacitor_THT:C_Disc_D7.0mm_W2.5mm_P5.00mm, F.Cu at (34.0, 113.0)
- added C14: 10µF, Capacitor_THT:CP_Radial_D5.0mm_P2.00mm, F.Cu at (33.5, 123.0)
- added C15: 0.1µ, Capacitor_THT:CP_Radial_D5.0mm_P2.00mm, F.Cu at (34.0, 107.5)
- added C16: 0.1µ, Capacitor_THT:CP_Radial_D5.0mm_P2.00mm, F.Cu at (34.0, 103.5)
- added C17: 0.1µ, Capacitor_THT:CP_Radial_D5.0mm_P2.00mm, F.Cu at (34.0, 91.5)
- added C18: 0.1µ, Capacitor_THT:CP_Radial_D5.0mm_P2.00mm, F.Cu at (37.0, 98.0)
- added C2: 10µ, Capacitor_THT:CP_Radial_D5.0mm_P2.00mm, F.Cu at (66.5, 89.0)
- added C3: 10µ, Capacitor_THT:CP_Radial_D5.0mm_P2.00mm, F.Cu at (68.5, 95.5)
- added C4: 1nF, Capacitor_THT:C_Disc_D7.0mm_W2.5mm_P5.00mm, F.Cu at (87.0, 60.5)
- added C5: 1nF, Capacitor_THT:C_Disc_D7.0mm_W2.5mm_P5.00mm, F.Cu at (38.0, 70.0)
- added C6: 10µF, Capacitor_THT:CP_Radial_D5.0mm_P2.00mm, F.Cu at (45.0, 61.5)
- added C7: 0.1µ, Capacitor_THT:CP_Radial_D5.0mm_P2.00mm, F.Cu at (83.0, 73.5)
- added C8: 0.1µ, Capacitor_THT:CP_Radial_D5.0mm_P2.00mm, F.Cu at (75.0, 73.5)
- added C9: 0.1µ, Capacitor_THT:CP_Radial_D5.0mm_P2.00mm, F.Cu at (75.5, 128.0)
- added CUTCV1: 100k, Potentiometer_THT:Potentiometer_Bourns_PTV09A-1_Single_Vertical, F.Cu at (140.5, 71.0)
- added CUTCV2: 100k, Potentiometer_THT:Potentiometer_Bourns_PTV09A-1_Single_Vertical, F.Cu at (114.5, 130.0)
- added CUTOFF1: 100k, Potentiometer_THT:Potentiometer_Bourns_PTV09A-1_Single_Vertical, F.Cu at (112.5, 51.0)
- added CUTOFF2: 100k, Potentiometer_THT:Potentiometer_Bourns_PTV09A-1_Single_Vertical, F.Cu at (142.5, 110.0)
- added D1: LED-12V, LED_THT:LED_D4.0mm, F.Cu at (148.3, 86.5)
- added D10: 1N4148, Diode_THT:D_DO-35_SOD27_P7.62mm_Horizontal, F.Cu at (73.0, 95.5)
- added D11: 1N4148, Diode_THT:D_DO-35_SOD27_P7.62mm_Horizontal, F.Cu at (80.0, 98.9)
- added D12: 1N4148, Diode_THT:D_DO-35_SOD27_P7.62mm_Horizontal, F.Cu at (73.0, 106.5)
- added D13: 1N4148, Diode_THT:D_DO-35_SOD27_P7.62mm_Horizontal, F.Cu at (76.5, 98.9)
- added D2: 1N4148, Diode_THT:D_DO-35_SOD27_P7.62mm_Horizontal, F.Cu at (81.5, 38.9)
- added D3: 1N4148, Diode_THT:D_DO-35_SOD27_P7.62mm_Horizontal, F.Cu at (81.5, 58.0)
- added D4: 1N4148, Diode_THT:D_DO-35_SOD27_P7.62mm_Horizontal, F.Cu at (78.0, 46.5)
- added D5: 1N4148, Diode_THT:D_DO-35_SOD27_P7.62mm_Horizontal, F.Cu at (78.0, 50.4)
- added D6: 1N4148, Diode_THT:D_DO-35_SOD27_P7.62mm_Horizontal, F.Cu at (74.5, 46.5)
- added D7: 1N4148, Diode_THT:D_DO-35_SOD27_P7.62mm_Horizontal, F.Cu at (74.5, 58.0)
- added D8: 1N4148, Diode_THT:D_DO-35_SOD27_P7.62mm_Horizontal, F.Cu at (76.5, 87.9)
- added D9: 1N4148, Diode_THT:D_DO-35_SOD27_P7.62mm_Horizontal, F.Cu at (80.0, 87.9)
- added FB1: 10R, Inductor_THT:L_Axial_L9.5mm_D4.0mm_P12.70mm_Horizontal_Fastron_SMCC, B.Cu at (62.0, 87.2)
- added FB2: 10R, Inductor_THT:L_Axial_L9.5mm_D4.0mm_P12.70mm_Horizontal_Fastron_SMCC, B.Cu at (57.0, 99.8)
- added J1: Conn_CircuitBoard, Connector_PinSocket_2.54mm:PinSocket_1x06_P2.54mm_Vertical, F.Cu at (33.0, 69.0)
- added J10: Conn_CircuitBoard, Connector_PinSocket_2.54mm:PinSocket_1x06_P2.54mm_Vertical, F.Cu at (87.0, 130.0)
- added J11: Conn_JackBoard, Connector_PinHeader_2.54mm:PinHeader_1x06_P2.54mm_Vertical, B.Cu at (98.0, 130.0)
- added J12: Conn_JackBoard, Connector_PinHeader_2.54mm:PinHeader_1x06_P2.54mm_Vertical, B.Cu at (152.0, 130.0)
- added J13: FilterCV2, Connector_Audio:Jack_3.5mm_QingPu_WQP-PJ398SM_Vertical_CircularHoles, F.Cu at (115.0, 133.0)
- added J14: FilterIn2, Connector_Audio:Jack_3.5mm_QingPu_WQP-PJ398SM_Vertical_CircularHoles, F.Cu at (125.0, 133.0)
- added J15: FilterOut2, Connector_Audio:Jack_3.5mm_QingPu_WQP-PJ398SM_Vertical_CircularHoles, F.Cu at (135.0, 133.0)
- added J2: Conn_CircuitBoard, Connector_PinSocket_2.54mm:PinSocket_1x06_P2.54mm_Vertical, F.Cu at (87.0, 69.0)
- added J3: Conn_JackBoard, Connector_PinHeader_2.54mm:PinHeader_1x06_P2.54mm_Vertical, B.Cu at (98.0, 69.0)
- added J4: Conn_JackBoard, Connector_PinHeader_2.54mm:PinHeader_1x06_P2.54mm_Vertical, B.Cu at (152.0, 69.0)
- added J5: Power Input, Connector_PinHeader_2.54mm:PinHeader_2x05_P2.54mm_Vertical, B.Cu at (41.9, 93.2)
- added J6: FilterCV1, Connector_Audio:Jack_3.5mm_QingPu_WQP-PJ398SM_Vertical_CircularHoles, F.Cu at (135.0, 74.0)
- added J7: FilterIn1, Connector_Audio:Jack_3.5mm_QingPu_WQP-PJ398SM_Vertical_CircularHoles, F.Cu at (125.0, 74.0)
- added J8: FilterOut1, Connector_Audio:Jack_3.5mm_QingPu_WQP-PJ398SM_Vertical_CircularHoles, F.Cu at (115.0, 74.0)
- added J9: Conn_CircuitBoard, Connector_PinSocket_2.54mm:PinSocket_1x06_P2.54mm_Vertical, F.Cu at (33.0, 130.0)
- added Q1: BC559, Package_TO_SOT_THT:TO-92_Inline, F.Cu at (71.0, 75.3)
- added Q2: BC559, Package_TO_SOT_THT:TO-92_Inline, F.Cu at (65.1, 72.7)
- added Q3: BC559, Package_TO_SOT_THT:TO-92_Inline, F.Cu at (57.4, 121.8)
- added Q4: BC559, Package_TO_SOT_THT:TO-92_Inline, F.Cu at (63.0, 121.8)
- added R1: 470, Resistor_THT:R_Axial_DIN0207_L6.3mm_D2.5mm_P10.16mm_Horizontal, F.Cu at (57.5, 59.8)
- added R10: 1.8k, Resistor_THT:R_Axial_DIN0207_L6.3mm_D2.5mm_P10.16mm_Horizontal, F.Cu at (57.5, 83.0)
- added R11: 100k, Resistor_THT:R_Axial_DIN0207_L6.3mm_D2.5mm_P10.16mm_Horizontal, F.Cu at (51.1, 66.0)
- added R12: 470, Resistor_THT:R_Axial_DIN0207_L6.3mm_D2.5mm_P10.16mm_Horizontal, F.Cu at (51.1, 49.5)
- added R13: 470, Resistor_THT:R_Axial_DIN0207_L6.3mm_D2.5mm_P10.16mm_Horizontal, F.Cu at (51.1, 56.5)
- added R14: 82k, Resistor_THT:R_Axial_DIN0207_L6.3mm_D2.5mm_P10.16mm_Horizontal, F.Cu at (104.0, 84.1)
- added R15: 100k, Resistor_THT:R_Axial_DIN0207_L6.3mm_D2.5mm_P10.16mm_Horizontal, F.Cu at (99.9, 55.0)
- added R16: 100k, Resistor_THT:R_Axial_DIN0207_L6.3mm_D2.5mm_P10.16mm_Horizontal, F.Cu at (40.9, 53.0)
- added R17: 33k, Resistor_THT:R_Axial_DIN0207_L6.3mm_D2.5mm_P10.16mm_Horizontal, F.Cu at (120.0, 45.0)
- added R18: 56k, Resistor_THT:R_Axial_DIN0207_L6.3mm_D2.5mm_P10.16mm_Horizontal, F.Cu at (130.2, 41.0)
- added R19: 1.8k, Resistor_THT:R_Axial_DIN0207_L6.3mm_D2.5mm_P10.16mm_Horizontal, F.Cu at (61.0, 72.9)
- added R2: 100k, Resistor_THT:R_Axial_DIN0207_L6.3mm_D2.5mm_P10.16mm_Horizontal, F.Cu at (39.5, 77.4)
- added R20: 2.2k, Resistor_THT:R_Axial_DIN0207_L6.3mm_D2.5mm_P10.16mm_Horizontal, F.Cu at (70.0, 38.9)
- added R21: 1k, Resistor_THT:R_Axial_DIN0207_L6.3mm_D2.5mm_P10.16mm_Horizontal, F.Cu at (107.5, 73.9)
- added R22: 1k, Resistor_THT:R_Axial_DIN0207_L6.3mm_D2.5mm_P10.16mm_Horizontal, F.Cu at (130.1, 69.0)
- added R23: 470, Resistor_THT:R_Axial_DIN0207_L6.3mm_D2.5mm_P10.16mm_Horizontal, F.Cu at (60.5, 137.1)
- added R24: 100k, Resistor_THT:R_Axial_DIN0207_L6.3mm_D2.5mm_P10.16mm_Horizontal, F.Cu at (41.5, 141.1)
- added R25: 470, Resistor_THT:R_Axial_DIN0207_L6.3mm_D2.5mm_P10.16mm_Horizontal, F.Cu at (38.0, 141.1)
- added R26: 2.2k, Resistor_THT:R_Axial_DIN0207_L6.3mm_D2.5mm_P10.16mm_Horizontal, F.Cu at (51.0, 109.1)
- added R27: 100k, Resistor_THT:R_Axial_DIN0207_L6.3mm_D2.5mm_P10.16mm_Horizontal, F.Cu at (57.0, 126.9)
- added R28: 100k, Resistor_THT:R_Axial_DIN0207_L6.3mm_D2.5mm_P10.16mm_Horizontal, F.Cu at (58.0, 102.4)
- added R29: 1k, Resistor_THT:R_Axial_DIN0207_L6.3mm_D2.5mm_P10.16mm_Horizontal, F.Cu at (77.9, 122.5)
- added R3: 470, Resistor_THT:R_Axial_DIN0207_L6.3mm_D2.5mm_P10.16mm_Horizontal, F.Cu at (36.4, 77.4)
- added R30: 2.2k, Resistor_THT:R_Axial_DIN0207_L6.3mm_D2.5mm_P10.16mm_Horizontal, F.Cu at (64.0, 137.1)
- added R31: 1.8k, Resistor_THT:R_Axial_DIN0207_L6.3mm_D2.5mm_P10.16mm_Horizontal, F.Cu at (54.5, 102.4)
- added R32: 100k, Resistor_THT:R_Axial_DIN0207_L6.3mm_D2.5mm_P10.16mm_Horizontal, F.Cu at (53.5, 137.1)
- added R33: 470, Resistor_THT:R_Axial_DIN0207_L6.3mm_D2.5mm_P10.16mm_Horizontal, F.Cu at (46.5, 137.1)
- added R34: 470, Resistor_THT:R_Axial_DIN0207_L6.3mm_D2.5mm_P10.16mm_Horizontal, F.Cu at (50.0, 137.1)
- added R35: 82k, Resistor_THT:R_Axial_DIN0207_L6.3mm_D2.5mm_P10.16mm_Horizontal, F.Cu at (102.5, 118.4)
- added R36: 100k, Resistor_THT:R_Axial_DIN0207_L6.3mm_D2.5mm_P10.16mm_Horizontal, F.Cu at (97.0, 109.5)
- added R37: 100k, Resistor_THT:R_Axial_DIN0207_L6.3mm_D2.5mm_P10.16mm_Horizontal, F.Cu at (50.0, 124.6)
- added R38: 33k, Resistor_THT:R_Axial_DIN0207_L6.3mm_D2.5mm_P10.16mm_Horizontal, F.Cu at (152.0, 113.9)
- added R39: 56k, Resistor_THT:R_Axial_DIN0207_L6.3mm_D2.5mm_P10.16mm_Horizontal, F.Cu at (148.0, 124.1)
- added R4: 2.2k, Resistor_THT:R_Axial_DIN0207_L6.3mm_D2.5mm_P10.16mm_Horizontal, F.Cu at (147.0, 71.9)
- added R40: 1.8k, Resistor_THT:R_Axial_DIN0207_L6.3mm_D2.5mm_P10.16mm_Horizontal, F.Cu at (61.5, 102.4)
- added R41: 2.2k, Resistor_THT:R_Axial_DIN0207_L6.3mm_D2.5mm_P10.16mm_Horizontal, F.Cu at (73.0, 119.6)
- added R42: 1k, Resistor_THT:R_Axial_DIN0207_L6.3mm_D2.5mm_P10.16mm_Horizontal, F.Cu at (129.0, 130.0)
- added R43: 1k, Resistor_THT:R_Axial_DIN0207_L6.3mm_D2.5mm_P10.16mm_Horizontal, F.Cu at (108.0, 144.1)
- added R5: 2.2k, Resistor_THT:R_Axial_DIN0207_L6.3mm_D2.5mm_P10.16mm_Horizontal, F.Cu at (54.0, 72.8)
- added R6: 100k, Resistor_THT:R_Axial_DIN0207_L6.3mm_D2.5mm_P10.16mm_Horizontal, F.Cu at (54.0, 70.0)
- added R7: 100k, Resistor_THT:R_Axial_DIN0207_L6.3mm_D2.5mm_P10.16mm_Horizontal, F.Cu at (61.0, 70.0)
- added R8: 1k, Resistor_THT:R_Axial_DIN0207_L6.3mm_D2.5mm_P10.16mm_Horizontal, F.Cu at (70.5, 70.1)
- added R9: 2.2k, Resistor_THT:R_Axial_DIN0207_L6.3mm_D2.5mm_P10.16mm_Horizontal, F.Cu at (74.1, 80.0)
- added Res1: 100k, Potentiometer_THT:Potentiometer_Bourns_PTV09A-1_Single_Vertical, F.Cu at (114.5, 71.0)
- added Res2: 100k, Potentiometer_THT:Potentiometer_Bourns_PTV09A-1_Single_Vertical, F.Cu at (140.5, 130.1)
- added ResLv1: 3.3k, Potentiometer_THT:Potentiometer_Bourns_3386C_Horizontal, B.Cu at (86.1, 45.1)
- added ResLv2: 3.3k, Potentiometer_THT:Potentiometer_Bourns_3386C_Horizontal, B.Cu at (86.0, 100.5)
- added ResVol1: 10k, Potentiometer_THT:Potentiometer_Bourns_3386C_Horizontal, B.Cu at (86.0, 56.6)
- added ResVol2: 10k, Potentiometer_THT:Potentiometer_Bourns_3386C_Horizontal, B.Cu at (86.0, 89.5)
- added SW1: Hpass/Lpass Switch, Synth:SW_DPDT_Toggle, F.Cu at (143.0, 44.0)
- added SW2: Bandpass, Synth:SW_Toggle_Blue_wSlots, F.Cu at (118.5, 91.5)
- added SW3: Hpass/Lpass Switch, Synth:SW_DPDT_Toggle, F.Cu at (107.0, 103.0)
- added U1: LM13700, Package_DIP:DIP-16_W7.62mm_Socket, F.Cu at (50.3, 87.2)
- added U2: TL072, Package_DIP:DIP-8_W7.62mm_Socket, F.Cu at (74.2, 61.2)
- added U3: LM13700, Package_DIP:DIP-16_W7.62mm_Socket, F.Cu at (39.2, 101.6)
- added U4: TL072, Package_DIP:DIP-8_W7.62mm_Socket, F.Cu at (78.2, 111.2)
- moved H2 79.5 mm to (228.0, 29.5)
- moved H3 79.5 mm to (228.0, 153.5)
- moved H1 59.5 mm to (186.0, 29.5)
- moved H4 59.5 mm to (186.0, 153.5)
Routing:
- net +12V: track 0.00 -> 225.1 mm
- net -12V: track 0.00 -> 218.2 mm, vias 0 -> 1
- net /Filtre2/Cutoff: track 0.00 -> 92.6 mm
- net /Cutoff: track 0.00 -> 78.6 mm
- net Filter2In: track 0.00 -> 73.2 mm
- net /LPass: track 0.00 -> 70.5 mm
- net /HPass: track 0.00 -> 65.2 mm
- net /FilterIn: track 0.00 -> 60.1 mm
- net /Out1: track 0.00 -> 58.3 mm
- net /ResOut: track 0.00 -> 57.4 mm, vias 0 -> 1
- net Net-(C6-Pad2): track 0.00 -> 56.7 mm
- net /Filtre2/Out1: track 0.00 -> 55.7 mm
- net Net-(C1-Pad2): track 0.00 -> 54.8 mm
- net /Filtre2/HPass: track 0.00 -> 52.5 mm
- net Net-(CUTOFF2-Pad2): track 0.00 -> 47.4 mm
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- added copper zone on B.Cu, net GND
- added copper zone on F.Cu, net GND
Other:
- board size 40 x 133 mm -> 207 x 130 mm
- board text added: "12HP"
- board text added: "Double MS-20 VCF V1.0 BleepSound 2022"
- board text added: "board 1/2"
- board text added: "board 2/2"

Commit message: update front gerber
Parts:
- removed C1, C11, C12, C13, C4, C5: 1nF, Capacitor_THT:C_Disc_D7.0mm_W2.5mm_P5.00mm
- removed C10, C15, C16, C17, C18, C7, C8, C9: 0.1µ, Capacitor_THT:CP_Radial_D5.0mm_P2.00mm
- removed C14, C6: 10µF, Capacitor_THT:CP_Radial_D5.0mm_P2.00mm
- removed C2, C3: 10µ, Capacitor_THT:CP_Radial_D5.0mm_P2.00mm
- removed CUTCV1, CUTCV2, CUTOFF1, CUTOFF2, Res1, Res2: 100k, Potentiometer_THT:Potentiometer_Bourns_PTV09A-1_Single_Vertical
- removed D1: LED-12V, LED_THT:LED_D4.0mm
- removed D10, D11, D12, D13, D2, D3, D4, D5, D6, D7, D8, D9: 1N4148, Diode_THT:D_DO-35_SOD27_P7.62mm_Horizontal
- removed FB1, FB2: 10R, Inductor_THT:L_Axial_L9.5mm_D4.0mm_P12.70mm_Horizontal_Fastron_SMCC
- removed J1, J10, J2, J9: Conn_CircuitBoard, Connector_PinSocket_2.54mm:PinSocket_1x06_P2.54mm_Vertical
- removed J11, J12, J3, J4: Conn_JackBoard, Connector_PinHeader_2.54mm:PinHeader_1x06_P2.54mm_Vertical
- removed J13: FilterCV2, Connector_Audio:Jack_3.5mm_QingPu_WQP-PJ398SM_Vertical_CircularHoles
- removed J14: FilterIn2, Connector_Audio:Jack_3.5mm_QingPu_WQP-PJ398SM_Vertical_CircularHoles
- removed J15: FilterOut2, Connector_Audio:Jack_3.5mm_QingPu_WQP-PJ398SM_Vertical_CircularHoles
- removed J5: Power Input, Connector_PinHeader_2.54mm:PinHeader_2x05_P2.54mm_Vertical
- removed J6: FilterCV1, Connector_Audio:Jack_3.5mm_QingPu_WQP-PJ398SM_Vertical_CircularHoles
- removed J7: FilterIn1, Connector_Audio:Jack_3.5mm_QingPu_WQP-PJ398SM_Vertical_CircularHoles
- removed J8: FilterOut1, Connector_Audio:Jack_3.5mm_QingPu_WQP-PJ398SM_Vertical_CircularHoles
- removed Q1, Q2, Q3, Q4: BC559, Package_TO_SOT_THT:TO-92_Inline
- removed R1, R12, R13, R23, R25, R3, R33, R34: 470, Resistor_THT:R_Axial_DIN0207_L6.3mm_D2.5mm_P10.16mm_Horizontal
- removed R10, R19, R31, R40: 1.8k, Resistor_THT:R_Axial_DIN0207_L6.3mm_D2.5mm_P10.16mm_Horizontal
- removed R11, R15, R16, R2, R24, R27, R28, R32, R36, R37, R6, R7: 100k, Resistor_THT:R_Axial_DIN0207_L6.3mm_D2.5mm_P10.16mm_Horizontal
- removed R14, R35: 82k, Resistor_THT:R_Axial_DIN0207_L6.3mm_D2.5mm_P10.16mm_Horizontal
- removed R17, R38: 33k, Resistor_THT:R_Axial_DIN0207_L6.3mm_D2.5mm_P10.16mm_Horizontal
- removed R18, R39: 56k, Resistor_THT:R_Axial_DIN0207_L6.3mm_D2.5mm_P10.16mm_Horizontal
- removed R20, R26, R30, R4, R41, R5, R9: 2.2k, Resistor_THT:R_Axial_DIN0207_L6.3mm_D2.5mm_P10.16mm_Horizontal
- removed R21, R22, R29, R42, R43, R8: 1k, Resistor_THT:R_Axial_DIN0207_L6.3mm_D2.5mm_P10.16mm_Horizontal
- removed ResLv1, ResLv2: 3.3k, Potentiometer_THT:Potentiometer_Bourns_3386C_Horizontal
- removed ResVol1, ResVol2: 10k, Potentiometer_THT:Potentiometer_Bourns_3386C_Horizontal
- removed SW1, SW3: Hpass/Lpass Switch, Synth:SW_DPDT_Toggle
- removed SW2: Bandpass, Synth:SW_Toggle_Blue_wSlots
- removed U1, U3: LM13700, Package_DIP:DIP-16_W7.62mm_Socket
- removed U2, U4: TL072, Package_DIP:DIP-8_W7.62mm_Socket
Routing:
- net +12V: track 225.1 -> 0.00 mm
- net -12V: track 218.2 -> 0.00 mm, vias 1 -> 0
- net /Filtre2/Cutoff: track 92.6 -> 0.00 mm
- net /Cutoff: track 78.6 -> 0.00 mm
- net Filter2In: track 73.2 -> 0.00 mm
- net /LPass: track 70.5 -> 0.00 mm
- net /HPass: track 65.2 -> 0.00 mm
- net /FilterIn: track 60.1 -> 0.00 mm
- net /Out1: track 58.3 -> 0.00 mm
- net /ResOut: track 57.4 -> 0.00 mm, vias 1 -> 0
- net Net-(C6-Pad2): track 56.7 -> 0.00 mm
- net /Filtre2/Out1: track 55.7 -> 0.00 mm
- net Net-(C1-Pad2): track 54.8 -> 0.00 mm
- net /Filtre2/HPass: track 52.5 -> 0.00 mm
- net Net-(CUTOFF2-Pad2): track 47.4 -> 0.00 mm
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- removed copper zone on B.Cu, net GND
- removed copper zone on F.Cu, net GND
Other:
- board size 207 x 130 mm -> 60 x 130 mm
- board text removed: "12HP"
- board text removed: "Double MS-20 VCF V1.0 BleepSound 2022"
- board text removed: "board 1/2"
- board text removed: "board 2/2"
