File: StupidBox/Panel/StupidBoxPanel.kicad_pcb (KiCad board)
At the start: 2 copper layers, 30 x 133 mm, 2 parts

Commit message: lots
Other:
- board text added: "JLCJLCJLCJLC"
Changed lines of the file:
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@@
   (general
     (thickness 1.6)
-    (drawings 477)
+    (drawings 488)
     (tracks 6)
     (zones 0)
@@
     (pad 1 thru_hole oval (at 0 0) (size 6.7 4.2) (drill oval 5.5 3) (layers *.Cu *.Mask))
   )
+  (gr_line (start 78.2 68.8) (end 78.7 68.3) (layer F.SilkS) (width 0.12))
+  (gr_line (start 76.7 66.8) (end 78.7 68.8) (layer F.SilkS) (width 0.12))
+  (gr_line (start 78.7 68.8) (end 78.7 68.3) (layer F.SilkS) (width 0.12))
+  (gr_line (start 78.7 68.8) (end 78.2 68.8) (layer F.SilkS) (width 0.12))
+  (gr_circle (center 76.2 66.3) (end 75.2 66.8) (layer F.SilkS) (width 0.12))
+  (gr_circle (center 84.3 110.7) (end 84.8 111.7) (layer F.SilkS) (width 0.12))
+  (gr_line (start 84 111.5) (end 83.5 111) (layer F.SilkS) (width 0.12))
+  (gr_line (start 84 111) (end 84 111.5) (layer F.SilkS) (width 0.12))
+  (gr_line (start 84 111) (end 83.5 111) (layer F.SilkS) (width 0.12))
+  (gr_line (start 82 113) (end 84 111) (layer F.SilkS) (width 0.12))
+  (gr_text JLCJLCJLCJLC (at 64 105.5 90) (layer B.SilkS)
+    (effects (font (size 1.5 1.5) (thickness 0.3)) (justify mirror))
+  )
   (dimension 133 (width 0.15) (layer Dwgs.User)

Commit message: update panel for stupid box
Other:
- net class Default removed
- net class Power removed
