File: Drumbox/Drumbox/Drumbox.kicad_pcb (KiCad board)
At the start: 2 copper layers, 186 x 133 mm, 115 parts, among them J1 Conn_01x04_Male, J10 Bass OUT, J11 LBonga OUT, J12 Conn_01x04_Female, J13 Conn_01x04_Male, J14 Conn_01x04_Female, J15 Conn_01x04_Male, J16 HBonga OUT, J17 Clave OUT, J18 Conn_01x03_Female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

Commit message: update drumbox
Parts:
- moved PITCH3 221.6 mm to (126.5, 66.0), turned to 90 degrees
- moved VOL3 217.8 mm to (126.5, 115.0), turned to 90 degrees
- moved J17 217.1 mm to (145.0, 119.5)
- moved J7 206.1 mm to (124.0, 73.2)
- moved J11 201.7 mm to (124.0, 119.5)
- moved VOL4 195.6 mm to (147.5, 115.0), turned to 90 degrees
- moved J9 189.9 mm to (145.0, 73.1)
- moved PITCH4 171.3 mm to (147.5, 66.0), turned to 90 degrees
- moved PITCH2 114.2 mm to (105.5, 66.0), turned to 90 degrees
- moved J8 98.3 mm to (103.0, 73.0)
- moved J16 54.3 mm to (103.0, 119.5)
- moved VOL2 49.0 mm to (105.5, 115.0), turned to 90 degrees
- moved J10 0.71 mm to (82.0, 120.2)
- moved J6 0.55 mm to (82.0, 73.0)
- moved DECAY1 0.50 mm to (84.5, 45.5)
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Routing:
- net GND: vias 2 -> 0
- net (no net): vias 16 -> 14

Commit message: update drumbox (not finished)
Parts:
- removed C21, C22, C25, C26: 10µF, Capacitor_THT:C_Disc_D7.0mm_W2.5mm_P5.00mm
- added C27: 100n, Capacitor_THT:CP_Radial_D5.0mm_P2.00mm, F.Cu at (128.5, 115.5)
- added C28: 100n, Capacitor_THT:CP_Radial_D5.0mm_P2.00mm, F.Cu at (136.5, 115.5)
- D5, J12, J14, J18, J2, J4, J5: moved to B.Cu
- moved C1 410.8 mm to (-16.5, 134.1), turned to -90 degrees
- moved C4 403.3 mm to (-9.50, 134.0), turned to -90 degrees
- moved R11 400.1 mm to (-13.0, 128.9), turned to -90 degrees
- moved C8 398.5 mm to (5.50, 114.1), turned to -90 degrees
- moved C2 387.4 mm to (5.50, 134.1), turned to -90 degrees
- moved R10 380.4 mm to (-2.50, 121.4), turned to -90 degrees
- moved C12 377.0 mm to (-9.50, 114.0), turned to -90 degrees
- moved R12 372.6 mm to (-9.50, 121.4), turned to -90 degrees
- moved R7 372.1 mm to (2.00, 129.0), turned to -90 degrees
- moved C9 370.6 mm to (42.0, 66.5), turned to 90 degrees
- moved C10 369.9 mm to (-2.50, 114.0), turned to -90 degrees
- moved C6 367.7 mm to (-16.5, 114.0), turned to -90 degrees
- moved R5 366.2 mm to (-20.0, 129.0), turned to -90 degrees
- moved C16 363.1 mm to (37.0, 122.5), turned to 180 degrees
- moved C11 359.1 mm to (43.5, 52.0), turned to 180 degrees
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Connections:
- R36 pad 2: Net-(C21-Pad2) -> Net-(U2-Pad1)
- R37 pad 2: Net-(C22-Pad2) -> Net-(U2-Pad6)
- R40 pad 2: Net-(C25-Pad2) -> Net-(U2-Pad8)
- R41 pad 2: Net-(C26-Pad2) -> Net-(U2-Pad13)
- U2 pad 1: Net-(C21-Pad1) -> Net-(U2-Pad1)
- U2 pad 13: Net-(C26-Pad1) -> Net-(U2-Pad13)
- U2 pad 14: Net-(C26-Pad1) -> Net-(U2-Pad13)
- U2 pad 2: Net-(C21-Pad1) -> Net-(U2-Pad1)
- U2 pad 6: Net-(C22-Pad1) -> Net-(U2-Pad6)
- U2 pad 7: Net-(C22-Pad1) -> Net-(U2-Pad6)
- U2 pad 8: Net-(C25-Pad1) -> Net-(U2-Pad8)
- U2 pad 9: Net-(C25-Pad1) -> Net-(U2-Pad8)
Routing:
- net +12V: track 0.00 -> 160.3 mm, vias 0 -> 2
- net O4: track 0.00 -> 119.0 mm
- net O1: track 0.00 -> 101.3 mm
- net In4: track 0.00 -> 91.1 mm
- net PIOut4: track 0.00 -> 81.4 mm
- net O3: track 0.00 -> 80.7 mm
- net O2: track 0.00 -> 78.5 mm
- net In3: track 0.00 -> 63.2 mm
- net -12V: track 0.00 -> 53.6 mm
- net DEIn1: track 0.00 -> 52.3 mm
- net Net-(C19-Pad2): track 0.00 -> 51.8 mm
- net Net-(C20-Pad2): track 0.00 -> 50.6 mm
- net DEIn4: track 0.00 -> 50.6 mm
- net PIOut3: track 0.00 -> 50.4 mm
- net Net-(U2-Pad3): track 0.00 -> 50.2 mm
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- added copper zone on F.Cu, net GND
Other:
- board size 186 x 133 mm -> 253.2 x 133 mm
- board text added: "24HP"
- board text removed: "16HP"

Commit message: update drumbox (not finished 2)
Parts:
- added REF**: Doepfer Mounting hole, Synth:Doepfer Mounting hole, F.Cu at (253.0, 15.5)
- moved C12 93.8 mm to (60.5, 51.5)
- moved R12 93.8 mm to (60.5, 58.9)
- moved C4 93.6 mm to (61.0, 72.5), turned to 0 degrees
- moved C1 92.8 mm to (60.9, 83.0), turned to 0 degrees
- moved C6 91.3 mm to (50.0, 51.5)
- moved R6 91.3 mm to (50.0, 58.9)
- moved R11 90.8 mm to (58.1, 72.5), turned to 180 degrees
- moved R5 90.6 mm to (58.0, 83.0), turned to 180 degrees
- moved C10 86.3 mm to (57.0, 51.5)
- moved R10 86.2 mm to (57.0, 59.0)
- moved C3 86.0 mm to (61.0, 76.0), turned to 0 degrees
- moved R9 83.1 mm to (58.1, 76.0), turned to 180 degrees
- moved C8 78.9 mm to (53.5, 51.5)
- moved R8 78.9 mm to (53.5, 58.9)
- moved C2 77.8 mm to (61.0, 79.5), turned to 0 degrees
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Connections:
- C5 pad 2: PI1Out -> PIOut1
- C6 pad 1: PI1Out -> PIOut1
- D1 pad 1: PI1Out -> PIOut1
Routing:
- net +12V: track 160.3 -> 256.9 mm
- net Net-(C9-Pad1): track 0.00 -> 82.2 mm, vias 0 -> 1
- net Net-(C11-Pad1): track 0.00 -> 76.8 mm, vias 0 -> 3
- net Net-(C5-Pad1): track 0.00 -> 76.1 mm
- net Net-(C7-Pad1): track 0.00 -> 69.8 mm
- net O4: track 119.0 -> 185.6 mm
- net O3: track 80.7 -> 139.9 mm
- net O2: track 78.5 -> 135.7 mm
- net O1: track 101.3 -> 156.9 mm
- net Net-(C16-Pad2): track 0.00 -> 52.9 mm
- net Net-(C13-Pad2): track 0.00 -> 44.5 mm
- net Net-(D4-Pad2): track 0.00 -> 41.0 mm
- net Net-(D3-Pad2): track 0.00 -> 40.2 mm
- net Net-(D2-Pad2): track 0.00 -> 39.3 mm
- net PIOut4: track 81.4 -> 119.4 mm
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Other:
- board size 253.2 x 133 mm -> 286 x 133 mm

Commit message: update drumbox
Parts:
- added ?: , , F.Cu at (208.0, 149.5)
- added ?: , , F.Cu at (304.0, 149.5)
- added REF**: Doepfer Mounting hole, Synth:Doepfer Mounting hole, F.Cu at (304.0, 22.5)
- moved REF** 45.5 mm to (208.0, 22.5)
Routing:
- net (no net): vias 12 -> 20
