File: Basic-mixer/Basic-mixer.kicad_sch (KiCad schematic)
At the start: 41 parts, among them J1 In1, J2 In1, J3 In1, J4 In1, J5 Out, J6 Power Input, SW1 mute1, SW2 mute1, SW3 mute1, SW4 mute1, U1 TL072

Commit message: update basic mixer (schem finish)
Parts:
- removed C2, C3: .1µF, Capacitor_THT:CP_Radial_D5.0mm_P2.00mm, symbol Device:CP
- removed D3: LED-mute, LED_THT:LED_D4.0mm, symbol Device:LED
- removed FB1, FB2: 10R, Inductor_THT:L_Axial_L9.5mm_D4.0mm_P12.70mm_Horizontal_Fastron_SMCC, symbol Device:Ferrite_Bead_Small
- removed J2, J4: In1, Connector_Audio:Jack_3.5mm_QingPu_WQP-PJ398SM_Vertical_CircularHoles, symbol Connector:AudioJack2_Switch
- removed R2, R3: 100k, Resistor_THT:R_Axial_DIN0207_L6.3mm_D2.5mm_P10.16mm_Horizontal, symbol Device:R
- removed R7, R8: 4.7k, Resistor_THT:R_Axial_DIN0207_L6.3mm_D2.5mm_P10.16mm_Horizontal, symbol Device:R
- removed SW1, SW2, SW3, SW4: mute1, symbol Switch:SW_DPST
- added C6, C7: .1µF, Capacitor_THT:CP_Radial_D5.0mm_P2.00mm, symbol Device:CP
- added J5, J6: In, Synth:Thonkiconn, symbol Connector:AudioJack2_Switch
- added R10, R5: 100k, Resistor_THT:R_Axial_DIN0207_L6.3mm_D2.5mm_P10.16mm_Horizontal, symbol Device:R
- added R11: 4.7k, Resistor_THT:R_Axial_DIN0207_L6.3mm_D2.5mm_P10.16mm_Horizontal, symbol Device:R
- added SW1, SW2, SW3, SW4: Mute, Synth:SW_DPDT_Toggle, symbol Switch:SW_Push_DPDT
- D5: value LED-12V -> LED-mute
- J1, J3: value In1 -> In; footprint Connector_Audio:Jack_3.5mm_QingPu_WQP-PJ398SM_Vertical_CircularHoles -> Synth:Thonkiconn
- J4: renamed from J5; footprint Connector_Audio:Jack_3.5mm_QingPu_WQP-PJ398SM_Vertical_CircularHoles -> Synth:Thonkiconn
- R12: value 4.7k -> 100k
- R4: value 100k -> 4.7k
- Vol1, Vol2, Vol3, Vol4: footprint Potentiometer_THT:Potentiometer_Bourns_PTV09A-1_Single_Vertical -> Synth:Pot-bourns-alpha
- renumbered C6 to C2, C7 to C3, J6 to J2, R5 to R1, R1 to R2, R10 to R7, R11 to R8
Connections:
- net +12V: now also J2.1 (Pin_1), J2.2 (Pin_2), R4.1, R11.1; no longer R12.1
- net -12V: now also J2.10 (Pin_10), J2.9 (Pin_9)
- net GND: now also J5.S, J6.S, SW1.1 (A), SW2.1 (A), SW3.1 (A), SW4.1 (A); no longer D5.1 (K)
- net at R2.1, R9.2, U1.6 (-): now also R12.1, R10.1, R5.1; no longer R4.1
- net at D5.2 (A): now also R11.2; no longer R12.2
- net at J1.T: now also SW1.5 (B)
- net at Vol4.1: now also SW4.6 (C)
- net at D4.1 (K): now also SW3.2 (B)
- net at R4.2: now also D2.2 (A); no longer C4.1
- net at Vol3.2: now also C6.2
- net at R6.2: now also D4.2 (A); no longer D2.2 (A)
- net at Vol3.1: now also SW3.6 (C)
- net at Vol2.1: now also SW2.6 (C)
- net at Vol2.2: now also C4.2
- net at D1.1 (K): now also SW1.2 (B)
- net at D2.1 (K): now also SW2.2 (B)
- net at Vol1.1: now also SW1.6 (C)
- net at Vol4.2: now also C7.2; no longer C4.2
- net at J3.T: now also SW2.5 (B)
- new net: J5.T, SW3.5 (B)
- new net: D5.1 (K), SW4.2 (B)
- new net: C7.1, R12.2
- new net: J6.T, SW4.5 (B)
- new net: C6.1, R10.2
- new net: C4.1, R5.2
- no-connect marks 10 -> 18
Other:
- moved on the sheet: C1, C2, C3, C5, D1, J1, J4, R1, R2, R7, R8, R9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
