File: Drumbox/Drumbox.kicad_sch (KiCad schematic)
At the start: 83 parts, among them J1 Conn_01x04_Male, J2 Conn_01x04_Female, J3 Conn_01x04_Male, J4 Conn_01x04_Female, J5 Power Input, Q1 2N3904, Q2 2N3904, Q3 2N3904, Q4 2N3904, U1 4011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

Commit message: update resistor values
Parts:
- R30: value 47k -> 110k
- R31, R32, R33: value 47k -> 100k
Other:
- note removed: "VALEUR Resistance a vérifier!"
Changed lines of the file:
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@@
-    (effects (font (size 1.27 1.27)) (justify left bottom))
-  )
-  (text "VALEUR Resistance a vérifier!" (at 41.91 160.02 0)
     (effects (font (size 1.27 1.27)) (justify left bottom))
   )
@@
       (effects (font (size 1.27 1.27)) (justify right))
     )
-    (property "Value" "47k" (id 1) (at 24.13 175.26 90)
+    (property "Value" "110k" (id 1) (at 24.13 175.26 90)
       (effects (font (size 1.27 1.27)) (justify right))
     )
@@
       (effects (font (size 1.27 1.27)) (justify right))
     )
-    (property "Value" "47k" (id 1) (at 59.69 175.26 90)
+    (property "Value" "100k" (id 1) (at 59.69 175.26 90)
       (effects (font (size 1.27 1.27)) (justify right))
     )
@@
       (effects (font (size 1.27 1.27)) (justify right))
     )
-    (property "Value" "47k" (id 1) (at 95.25 175.26 90)
+    (property "Value" "100k" (id 1) (at 95.25 175.26 90)
       (effects (font (size 1.27 1.27)) (justify right))
     )
@@
       (effects (font (size 1.27 1.27)) (justify right))
     )
-    (property "Value" "47k" (id 1) (at 130.81 175.26 90)
+    (property "Value" "100k" (id 1) (at 130.81 175.26 90)
       (effects (font (size 1.27 1.27)) (justify right))
     )
@@
     )
     (path "/00000000-0000-0000-0000-000061cca9c2"
-      (reference "R30") (unit 1) (value "47k") (footprint "Resistor_THT:R_Axial_DIN0207_L6.3mm_D2.5mm_P10.16mm_Horizontal")
+      (reference "R30") (unit 1) (value "110k") (footprint "Resistor_THT:R_Axial_DIN0207_L6.3mm_D2.5mm_P10.16mm_Horizontal")
     )
     (path "/00000000-0000-0000-0000-000061cca9e9"
-      (reference "R31") (unit 1) (value "47k") (footprint "Resistor_THT:R_Axial_DIN0207_L6.3mm_D2.5mm_P10.16mm_Horizontal")
+      (reference "R31") (unit 1) (value "100k") (footprint "Resistor_THT:R_Axial_DIN0207_L6.3mm_D2.5mm_P10.16mm_Horizontal")
     )
     (path "/00000000-0000-0000-0000-000061ccaa10"
-      (reference "R32") (unit 1) (value "47k") (footprint "Resistor_THT:R_Axial_DIN0207_L6.3mm_D2.5mm_P10.16mm_Horizontal")
+      (reference "R32") (unit 1) (value "100k") (footprint "Resistor_THT:R_Axial_DIN0207_L6.3mm_D2.5mm_P10.16mm_Horizontal")
     )
     (path "/00000000-0000-0000-0000-000061ccaa37"
-      (reference "R33") (unit 1) (value "47k") (footprint "Resistor_THT:R_Axial_DIN0207_L6.3mm_D2.5mm_P10.16mm_Horizontal")
+      (reference "R33") (unit 1) (value "100k") (footprint "Resistor_THT:R_Axial_DIN0207_L6.3mm_D2.5mm_P10.16mm_Horizontal")
     )
     (path "/00000000-0000-0000-0000-00006029ed90/00000000-0000-0000-0000-000060503194"
