File: Drumbox/Jackboard/Drumbox.kicad_pcb (KiCad board)
At the start: 2 copper layers, 286 x 133 mm, 117 parts, among them J1 Conn_01x04_Male, J10 Bass OUT, J11 LBonga OUT, J12 Conn_01x04_Female, J13 Conn_01x04_Male, J14 Conn_01x04_Female, J15 Conn_01x04_Male, J16 HBonga OUT, J17 Clave OUT, J18 Conn_01x03_Female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

Commit message: create gerber for drumbox
Parts:
- removed ? (x2): , 
- removed C1, C13: 150nF, Capacitor_THT:C_Disc_D7.0mm_W2.5mm_P5.00mm
- removed C10, C9: 12nF, Capacitor_THT:C_Disc_D7.0mm_W2.5mm_P5.00mm
- removed C11, C12: 1.5nF, Capacitor_THT:C_Disc_D7.0mm_W2.5mm_P5.00mm
- removed C14, C2: 33nF, Capacitor_THT:C_Disc_D7.0mm_W2.5mm_P5.00mm
- removed C15, C3: 39nF, Capacitor_THT:C_Disc_D7.0mm_W2.5mm_P5.00mm
- removed C16: 4.7nF, Capacitor_THT:C_Disc_D7.0mm_W2.5mm_P5.00mm
- removed C17, C18: 10µ, Capacitor_THT:CP_Radial_D5.0mm_P2.00mm
- removed C4: 56nF, Capacitor_THT:C_Disc_D7.0mm_W2.5mm_P5.00mm
- removed C5, C6: 47nF, Capacitor_THT:C_Disc_D7.0mm_W2.5mm_P5.00mm
- removed C7, C8: 10nF, Capacitor_THT:C_Disc_D7.0mm_W2.5mm_P5.00mm
- removed D1, D2, D3, D4: 1N4148, Diode_THT:D_DO-35_SOD27_P7.62mm_Horizontal
- removed D5: LED-12V, LED_THT:LED_D4.0mm
- removed FB1, FB2: 10R, Inductor_THT:L_Axial_L9.5mm_D4.0mm_P12.70mm_Horizontal_Fastron_SMCC
- removed J1, J13, J15, J3: Conn_01x04_Male, Connector_PinHeader_2.54mm:PinHeader_1x04_P2.54mm_Vertical
- removed J19: Conn_01x03_Male, Connector_PinHeader_2.54mm:PinHeader_1x03_P2.54mm_Vertical
- removed J5: Power Input, Connector_PinHeader_2.54mm:PinHeader_2x05_P2.54mm_Vertical
- removed R1, R2, R3, R4: 150k, Resistor_THT:R_Axial_DIN0207_L6.3mm_D2.5mm_P10.16mm_Horizontal
- removed R10, R11, R12, R5, R6, R7, R8, R9: 68k, Resistor_THT:R_Axial_DIN0207_L6.3mm_D2.5mm_P10.16mm_Horizontal
- removed R13, R14, R15, R16: 27k, Resistor_THT:R_Axial_DIN0207_L6.3mm_D2.5mm_P10.16mm_Horizontal
- removed R17, R19, R21, R23: 12k, Resistor_THT:R_Axial_DIN0207_L6.3mm_D2.5mm_P10.16mm_Horizontal
- removed R18, R20, R22, R24: 47k, Resistor_THT:R_Axial_DIN0207_L6.3mm_D2.5mm_P10.16mm_Horizontal
- removed R25: 2.2k, Resistor_THT:R_Axial_DIN0207_L6.3mm_D2.5mm_P10.16mm_Horizontal
- removed REF** (x2): Doepfer Mounting hole, Synth:Doepfer Mounting hole
- removed U1: 4011, Package_DIP:DIP-14_W7.62mm_Socket
Routing:
- net +12V: track 256.9 -> 161.3 mm
- net Net-(C9-Pad1): track 82.2 -> 0.00 mm, vias 1 -> 0
- net Net-(C11-Pad1): track 76.8 -> 0.00 mm, vias 3 -> 0
- net Net-(C5-Pad1): track 76.1 -> 0.00 mm
- net Net-(C7-Pad1): track 69.8 -> 0.00 mm
- net O4: track 185.6 -> 119.0 mm
- net O3: track 139.9 -> 80.7 mm
- net O2: track 135.7 -> 78.5 mm
- net O1: track 156.9 -> 101.3 mm
- net Net-(C16-Pad2): track 52.9 -> 0.00 mm
- net Net-(C13-Pad2): track 44.5 -> 0.00 mm
- net Net-(D4-Pad2): track 41.0 -> 0.00 mm
- net Net-(D3-Pad2): track 40.2 -> 0.00 mm
- net Net-(D2-Pad2): track 39.3 -> 0.00 mm
- net PIOut4: track 119.4 -> 81.4 mm
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Other:
- board size 286 x 133 mm -> 120 x 110 mm
- board text removed: "8HP"
- board text removed: "board 1/2"
