File: Mixers/Basic-mixer/jackboard/Basic-mixer.kicad_pcb (KiCad board)
At the start: 2 copper layers, 40 x 110 mm, 37 parts, among them J1 In, J2 Power Input, J3 In, J4 Out, J5 In, J6 In, SW1 Mute, SW2 Mute, SW3 Mute, SW4 Mute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

Commit message: Fix GND link to inv Opamp 1
Other:
- board text removed: "8HP"
Changed lines of the file:
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@@
       (svguseinch false)
       (svgprecision 6)
-      (excludeedgelayer true)
+      (excludeedgelayer false)
       (plotframeref false)
       (viasonmask false)
@@
     (fp_line (start 2.721 1.04) (end 2.721 1.937) (layer "F.SilkS") (width 0.12))
     (fp_line (start 1.721 1.04) (end 1.721 2.48) (layer "F.SilkS") (width 0.12))
-    (fp_line (start 2.521 1.04) (end 2.521 2.095) (layer "F.SilkS") (width 0.12))
     (fp_line (start 1.721 -2.48) (end 1.721 -1.04) (layer "F.SilkS") (width 0.12))
     (fp_line (start 1.961 -2.398) (end 1.961 -1.04) (layer "F.SilkS") (width 0.12))
@@
     (fp_line (start 2.601 1.04) (end 2.601 2.035) (layer "F.SilkS") (width 0.12))
     (fp_line (start 2.801 -1.864) (end 2.801 -1.04) (layer "F.SilkS") (width 0.12))
+    (fp_line (start 2.521 -2.095) (end 2.521 -1.04) (layer "F.SilkS") (width 0.12))
     (fp_line (start 1.921 -2.414) (end 1.921 -1.04) (layer "F.SilkS") (width 0.12))
     (fp_line (start 2.561 1.04) (end 2.561 2.065) (layer "F.SilkS") (width 0.12))
-    (fp_line (start 2.521 -2.095) (end 2.521 -1.04) (layer "F.SilkS") (width 0.12))
+    (fp_line (start 2.561 -2.065) (end 2.561 -1.04) (layer "F.SilkS") (width 0.12))
     (fp_line (start 1.921 1.04) (end 1.921 2.414) (layer "F.SilkS") (width 0.12))
     (fp_line (start 1.2 -2.573) (end 1.2 -1.04) (layer "F.SilkS") (width 0.12))
@@
     (fp_line (start 1.24 -2.569) (end 1.24 -1.04) (layer "F.SilkS") (width 0.12))
     (fp_line (start 1.68 -2.491) (end 1.68 -1.04) (layer "F.SilkS") (width 0.12))
-    (fp_line (start 2.561 -2.065) (end 2.561 -1.04) (layer "F.SilkS") (width 0.12))
+    (fp_line (start 2.521 1.04) (end 2.521 2.095) (layer "F.SilkS") (width 0.12))
     (fp_line (start 2.441 1.04) (end 2.441 2.149) (layer "F.SilkS") (width 0.12))
     (fp_line (start 1.801 1.04) (end 1.801 2.455) (layer "F.SilkS") (width 0.12))
@@
     (fp_line (start 2.321 1.04) (end 2.321 2.224) (layer "F.SilkS") (width 0.12))
     (fp_line (start 1.16 1.04) (end 1.16 2.576) (layer "F.SilkS") (width 0.12))
-    (fp_line (start 3.561 -0.518) (end 3.561 0.518) (layer "F.SilkS") (width 0.12))
+    (fp_line (start 3.601 -0.284) (end 3.601 0.284) (layer "F.SilkS") (width 0.12))
     (fp_line (start 2.881 1.04) (end 2.881 1.785) (layer "F.SilkS") (width 0.12))
     (fp_line (start 1.841 1.04) (end 1.841 2.442) (layer "F.SilkS") (width 0.12))
@@
     (fp_line (start 2.641 1.04) (end 2.641 2.004) (layer "F.SilkS") (width 0.12))
     (fp_line (start 1.32 1.04) (end 1.32 2.561) (layer "F.SilkS") (width 0.12))
+    (fp_line (start 3.561 -0.518) (end 3.561 0.518) (layer "F.SilkS") (width 0.12))
     (fp_line (start 3.041 -1.605) (end 3.041 1.605) (layer "F.SilkS") (width 0.12))
     (fp_line (start 1 1.04) (end 1 2.58) (layer "F.SilkS") (width 0.12))
@@
     (fp_line (start 1.64 -2.501) (end 1.64 -1.04) (layer "F.SilkS") (width 0.12))
     (fp_line (start 1.56 1.04) (end 1.56 2.52) (layer "F.SilkS") (width 0.12))
-    (fp_line (start 3.521 -0.677) (end 3.521 0.677) (layer "F.SilkS") (width 0.12))
     (fp_line (start 3.081 -1.554) (end 3.081 1.554) (layer "F.SilkS") (width 0.12))
     (fp_line (start 1.28 -2.565) (end 1.28 -1.04) (layer "F.SilkS") (width 0.12))
@@
     (fp_line (start 2.921 1.04) (end 2.921 1.743) (layer "F.SilkS") (width 0.12))
     (fp_line (start 2.401 -2.175) (end 2.401 -1.04) (layer "F.SilkS") (width 0.12))
-    (fp_line (start 3.601 -0.284) (end 3.601 0.284) (layer "F.SilkS") (width 0.12))
+    (fp_line (start 3.521 -0.677) (end 3.521 0.677) (layer "F.SilkS") (width 0.12))
     (fp_line (start 2.241 1.04) (end 2.241 2.268) (layer "F.SilkS") (width 0.12))
     (fp_line (start 2.241 -2.268) (end 2.241 -1.04) (layer "F.SilkS") (width 0.12))
@@
     (effects (font (size 1 1) (thickness 0.15)))
   )
-  (gr_text "8HP\n" (at 49 23) (layer "Dwgs.User")
-    (effects (font (size 1 1) (thickness 0.15)))
-  )
-  (dimension (type aligned) (layer "Dwgs.User")
-    (pts (xy 30 141) (xy 30 31))
-    (height -4.999999)
-    (gr_text "110.0000 mm" (at 23.850001 86 90) (layer "Dwgs.User")
-      (effects (font (size 1 1) (thickness 0.15)))
-    )
-    (format (units 2) (units_format 1) (precision 4))
-    (style (thickness 0.15) (arrow_length 1.27) (text_position_mode 0) (extension_height 0.58642) (extension_offset 0) keep_text_aligned)
-  )
-  (dimension (type aligned) (layer "Dwgs.User")
-    (pts (xy 70 25) (xy 30 25))
-    (height 5)
-    (gr_text "40.0000 mm" (at 50 18.85) (layer "Dwgs.User")
-      (effects (font (size 1 1) (thickness 0.15)))
-    )
-    (format (units 2) (units_format 1) (precision 4))
-    (style (thickness 0.15) (arrow_length 1.27) (text_position_mode 0) (extension_height 0.58642) (extension_offset 0) keep_text_aligned)
-  )
-  (dimension (type aligned) (layer "Dwgs.User")
-    (pts (xy 30 62.5) (xy 30 85))
-    (height 9.499999)
-    (gr_text "22.5000 mm" (at 19.350001 73.75 90) (layer "Dwgs.User")
-      (effects (font (size 1 1) (thickness 0.15)))
-    )
-    (format (units 3) (units_format 1) (precision 4))
-    (style (thickness 0.15) (arrow_length 1.27) (text_position_mode 0) (extension_height 0.58642) (extension_offset 0.5) keep_text_aligned)
-  )
-  (dimension (type aligned) (layer "Dwgs.User")
-    (pts (xy 30 40) (xy 30 62.5))
-    (height 9.499999)
-    (gr_text "22.5000 mm" (at 19.350001 51.25 90) (layer "Dwgs.User")
-      (effects (font (size 1 1) (thickness 0.15)))
-    )
-    (format (units 3) (units_format 1) (precision 4))
-    (style (thickness 0.15) (arrow_length 1.27) (text_position_mode 0) (extension_height 0.58642) (extension_offset 0.5) keep_text_aligned)
-  )
-  (dimension (type aligned) (layer "Dwgs.User")
-    (pts (xy 33 31) (xy 33 25))
-    (height -6)
-    (gr_text "6.0000 mm" (at 25.85 28 90) (layer "Dwgs.User")
-      (effects (font (size 1 1) (thickness 0.15)))
-    )
-    (format (units 2) (units_format 1) (precision 4))
-    (style (thickness 0.15) (arrow_length 1.27) (text_position_mode 0) (extension_height 0.58642) (extension_offset 0) keep_text_aligned)
-  )
-  (dimension (type aligned) (layer "Dwgs.User")
-    (pts (xy 29.999999 85) (xy 29.999999 107.5))
-    (height 9.499999)
-    (gr_text "22.5000 mm" (at 19.35 96.25 90) (layer "Dwgs.User")
-      (effects (font (size 1 1) (thickness 0.15)))
-    )
-    (format (units 3) (units_format 1) (precision 4))
-    (style (thickness 0.15) (arrow_length 1.27) (text_position_mode 0) (extension_height 0.58642) (extension_offset 0.5) keep_text_aligned)
-  )
   (segment (start 43.925 135.725) (end 43.925 138.265) (width 0.25) (layer "F.Cu") (net 2))
