File: Mixers/Basic-AC-mixer/Basic-mixer.kicad_pcb (KiCad board)
At the start: 2 copper layers, 82 x 128 mm, 37 parts, among them J1 In, J2 Power Input, J3 In, J4 Out, J5 In, J6 In, SW1 Mute, SW2 Mute, SW3 Mute, SW4 Mute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

Commit message: output gerber for jackboard
Connections:
- U1 pad 5: /Vgnd -> GND
Changed lines of the file:
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@@
   (net 44 "unconnected-(SW4-Pad4)")
   (net 45 "Net-(SW4-Pad6)")
-  (net 46 "/Vgnd")
   (footprint "Synth:Pot-bourns-alpha" (layer "F.Cu")
     (at 63.5 92.55 90)
@@
       (net 3 "-12V") (pinfunction "V-") (pintype "power_in"))
     (pad "5" thru_hole oval locked (at 7.62 7.62 90) (size 1.6 1.6) (drill 0.8) (layers *.Cu *.Mask)
-      (net 46 "/Vgnd") (pinfunction "+") (pintype "input"))
+      (net 1 "GND") (pinfunction "+") (pintype "input"))
     (pad "6" thru_hole oval locked (at 7.62 5.08 90) (size 1.6 1.6) (drill 0.8) (layers *.Cu *.Mask)
       (net 29 "Net-(R10-Pad1)") (pinfunction "-") (pintype "input"))
