File: PSU/PSU/PSU.kicad_sch (KiCad schematic)
At the start: 27 parts, among them J1 Power_Input, J2 Power connector, U1 L7812, U2 L7912

Commit message: update PSU gerber (with 3 pole terminal block output) + BOM
Detailled BOM in .xls with total component price for one system
Parts:
- removed J2: Power connector, Connector_PinHeader_2.54mm:PinHeader_2x05_P2.54mm_Vertical, symbol Connector:Conn_01x10_Male
- added J2: Power output, TerminalBlock:TerminalBlock_bornier-3_P5.08mm, symbol Connector:Screw_Terminal_01x03
- renumbered C5 to C2, C2 to C3, C6 to C4, C3 to C5, C7 to C6, C4 to C7, D2 to D1, D1 to D2, D6 to D5, D5 to D6, R2 to R1, R1 to R2
Connections:
- net GND: now also J2.2 (Pin_2)
- net at C9.1, D3.2 (A), D5.1 (K)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: now also J2.1 (Pin_1)
- net at C10.2, D4.1 (K), D6.2 (A)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: now also J2.3 (Pin_3)
Other:
- moved on the sheet: J1
