File: MS20-VCF/Simple/MS20-VCF.kicad_pcb (KiCad board)
At the start: 2 copper layers, 207 x 128 mm, 110 parts, among them J1 Conn_CircuitBoard, J10 Conn_CircuitBoard, J11 Conn_JackBoard, J12 Conn_JackBoard, J13 FilterCV2, J14 FilterIn2, J15 FilterOut2, J2 Conn_CircuitBoard, J3 Conn_JackBoard, J4 Conn_JackBoard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

Commit message: initial layout
Parts:
- removed C11, C12, C13: 1nF, Capacitor_THT:C_Disc_D7.0mm_W2.5mm_P5.00mm
- removed C14: 10µF, Capacitor_THT:CP_Radial_D5.0mm_P2.00mm
- removed CUTCV2, CUTOFF2, Res2: 100k, Potentiometer_THT:Potentiometer_Bourns_PTV09A-1_Single_Vertical
- removed D10, D11, D12, D13, D8, D9: 1N4148, Diode_THT:D_DO-35_SOD27_P7.62mm_Horizontal
- removed J1, J10, J2, J9: Conn_CircuitBoard, Connector_PinSocket_2.54mm:PinSocket_1x06_P2.54mm_Vertical
- removed J11, J12, J3, J4: Conn_JackBoard, Connector_PinHeader_2.54mm:PinHeader_1x06_P2.54mm_Vertical
- removed J13: FilterCV2, Connector_Audio:Jack_3.5mm_QingPu_WQP-PJ398SM_Vertical_CircularHoles
- removed J14: FilterIn2, Connector_Audio:Jack_3.5mm_QingPu_WQP-PJ398SM_Vertical_CircularHoles
- removed J15: FilterOut2, Connector_Audio:Jack_3.5mm_QingPu_WQP-PJ398SM_Vertical_CircularHoles
- removed Q3, Q4: BC559, Package_TO_SOT_THT:TO-92_Inline
- removed R23, R25, R33, R34: 470, Resistor_THT:R_Axial_DIN0207_L6.3mm_D2.5mm_P10.16mm_Horizontal
- removed R24, R27, R28, R32, R36, R37: 100k, Resistor_THT:R_Axial_DIN0207_L6.3mm_D2.5mm_P10.16mm_Horizontal
- removed R26, R30, R41: 2.2k, Resistor_THT:R_Axial_DIN0207_L6.3mm_D2.5mm_P10.16mm_Horizontal
- removed R29, R42, R43: 1k, Resistor_THT:R_Axial_DIN0207_L6.3mm_D2.5mm_P10.16mm_Horizontal
- removed R31, R40: 1.8k, Resistor_THT:R_Axial_DIN0207_L6.3mm_D2.5mm_P10.16mm_Horizontal
- removed R35: 82k, Resistor_THT:R_Axial_DIN0207_L6.3mm_D2.5mm_P10.16mm_Horizontal
- removed R38: 33k, Resistor_THT:R_Axial_DIN0207_L6.3mm_D2.5mm_P10.16mm_Horizontal
- removed R39: 56k, Resistor_THT:R_Axial_DIN0207_L6.3mm_D2.5mm_P10.16mm_Horizontal
- removed ResLv2: 3.3k, Potentiometer_THT:Potentiometer_Bourns_3386C_Horizontal
- removed ResVol2: 10k, Potentiometer_THT:Potentiometer_Bourns_3386C_Horizontal
- removed SW2: Bandpass, Synth:SW_Toggle_Blue_wSlots
- removed SW3: Hpass/Lpass Switch, Synth:SW_DPDT_Toggle
- removed U3: LM13700, Package_DIP:DIP-16_W7.62mm_Socket
- removed U4: TL072, Package_DIP:DIP-8_W7.62mm_Socket
- moved SW1 98.2 mm to (82.0, 121.0)
- moved J6 94.6 mm to (38.5, 129.7)
- moved J7 91.4 mm to (36.0, 94.7)
- moved CUTCV1 90.0 mm to (41.0, 123.0)
- moved Res1 83.3 mm to (62.0, 99.0)
- moved J8 55.2 mm to (84.0, 95.2)
- moved CUTOFF1 49.8 mm to (63.0, 56.0)
- moved FB1 45.0 mm to (73.5, 130.7)
- moved FB2 45.0 mm to (68.5, 143.3)
- moved J5 42.1 mm to (53.4, 133.7)
- moved C7 37.2 mm to (59.5, 121.0)
- moved C8 37.2 mm to (58.0, 127.5)
- moved C2 25.0 mm to (65.0, 114.0)
- moved C3 25.0 mm to (67.0, 120.5)
Connections:
- R22 pad 1: /FilterOut -> /JackOut
Routing:
- net +12V: track 281.3 -> 0.00 mm, vias 1 -> 0
- net -12V: track 267.1 -> 0.00 mm, vias 2 -> 0
- net /Filtre2/Cutoff: track 92.6 -> 0.00 mm
- net /Cutoff: track 78.6 -> 0.00 mm
- net /LPass: track 70.5 -> 0.00 mm
- net Filter2In: track 69.0 -> 0.00 mm
- net /HPass: track 65.2 -> 0.00 mm
- net /FilterIn: track 60.5 -> 0.00 mm
- net /Filtre2/ResOut: track 58.4 -> 0.00 mm
- net /Out1: track 58.3 -> 0.00 mm
- net Net-(C6-Pad2): track 56.7 -> 0.00 mm
- net Net-(CUTCV2-Pad2): track 55.4 -> 0.00 mm
- net Net-(C1-Pad2): track 54.8 -> 0.00 mm
- net /Filtre2/HPass: track 52.5 -> 0.00 mm
- net Net-(CUTOFF2-Pad2): track 48.1 -> 0.00 mm
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Other:
- board text added: "MS-20 VCF V1.0 BleepSound 2022"
- board text removed: "Double MS-20 VCF V1.1 BleepSound 2022"
- board text removed: "board 1/2"
