File: MS20-VCF/Simple/MS20-VCF.kicad_sch (KiCad schematic)
At the start: 62 parts, among them J1 Conn_CircuitBoard, J2 Conn_CircuitBoard, J3 Conn_JackBoard, J4 Conn_JackBoard, J5 Power Input, J6 FilterCV1, J7 FilterIn1, J8 FilterOut1, Q1 BC559, Q2 BC559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

Commit message: initial layout
Parts:
- removed J1, J2: Conn_CircuitBoard, Connector_PinSocket_2.54mm:PinSocket_1x06_P2.54mm_Vertical, symbol Connector:Conn_01x06_Female
- removed J3, J4: Conn_JackBoard, Connector_PinHeader_2.54mm:PinHeader_1x06_P2.54mm_Vertical, symbol Connector:Conn_01x06_Male
- removed SW2: Bandpass, Synth:SW_Toggle_Blue_wSlots, symbol Switch:SW_SPDT
Connections:
- net FilterOut is gone; now on net JackOut: R22.1
- no-connect marks 15 -> 9
Other:
- removed sheet Filtre2
