File: Drumbox/V1.1/Drumbox.kicad_pcb (KiCad board)
At the start: 2 copper layers, 286 x 128 mm, 117 parts, among them J1 Conn_01x04_Male, J10 Bass OUT, J11 LBonga OUT, J12 Conn_01x04_Female, J13 Conn_01x04_Male, J14 Conn_01x04_Female, J15 Conn_01x04_Male, J16 HBonga OUT, J17 Clave OUT, J18 Conn_01x03_Female, J19 Conn_01x03_Male, J2 Conn_01x04_Female, J3 Conn_01x04_Male, J4 Conn_01x04_Female, J5 Power Input, J6 Bass IN, J7 LBonga IN, J8 HBonga IN, J9 Clave IN, Q1 2N3904, Q2 2N3904, Q3 2N3904, Q4 2N3904, U1 4011, U2 TL074

Commit message: update drumbox
delete chanel output for single output + add button to trigger each sound
Parts:
- removed ? (x2): , 
- removed D6: LED1, LED_THT:LED_D4.0mm
- removed D7: LED2, LED_THT:LED_D4.0mm
- removed D8: LED3, LED_THT:LED_D4.0mm
- removed D9: LED4, LED_THT:LED_D4.0mm
- removed the J11 at (148.5, 120.2)
- removed the J16 at (118.5, 120.2)
- removed J17: Clave OUT, Connector_Audio:Jack_3.5mm_QingPu_WQP-PJ398SM_Vertical_CircularHoles
- removed the R26 at (84.0, 98.5)
- removed the R27 at (114.0, 98.6)
- removed the R28 at (144.0, 98.6)
- removed the R29 at (174.0, 98.5)
- removed the R30 at (93.0, 88.3)
- removed the R31 at (123.0, 88.4)
- removed the R37 at (113.4, 135.0)
- removed the R40 at (153.6, 135.0)
- removed R41: 1k, Resistor_THT:R_Axial_DIN0207_L6.3mm_D2.5mm_P10.16mm_Horizontal
- removed REF** (x2): Doepfer Mounting hole, Synth:Doepfer Mounting hole
- added H1: MountingHole, Synth:Doepfer Mounting hole, F.Cu at (203.5, 25.0)
- added H2: MountingHole, Synth:Doepfer Mounting hole, F.Cu at (308.5, 25.0)
- added H3: MountingHole, Synth:Doepfer Mounting hole, F.Cu at (203.5, 147.0)
- added H4: MountingHole, Synth:Doepfer Mounting hole, F.Cu at (308.5, 147.0)
- added H5: SpacerHoles, MountingHole:MountingHole_3.2mm_M3, F.Cu at (207.0, 135.0)
- added H6: SpacerHoles, MountingHole:MountingHole_3.2mm_M3, F.Cu at (84.5, 135.0)
- added H7: SpacerHoles, MountingHole:MountingHole_3.2mm_M3, F.Cu at (133.5, 44.5)
- added H8: SpacerHoles, MountingHole:MountingHole_3.2mm_M3, F.Cu at (256.0, 44.5)
- added R16: 1k, Resistor_THT:R_Axial_DIN0207_L6.3mm_D2.5mm_P10.16mm_Horizontal, F.Cu at (123.5, 100.5)
- added R18: 100k, Resistor_THT:R_Axial_DIN0207_L6.3mm_D2.5mm_P10.16mm_Horizontal, F.Cu at (123.5, 89.5)
- added R23: 47k, Resistor_THT:R_Axial_DIN0207_L6.3mm_D2.5mm_P10.16mm_Horizontal, F.Cu at (131.5, 85.9)
- added R24: 33k, Resistor_THT:R_Axial_DIN0207_L6.3mm_D2.5mm_P10.16mm_Horizontal, F.Cu at (135.0, 96.1)
- added R34: 1k, Resistor_THT:R_Axial_DIN0207_L6.3mm_D2.5mm_P10.16mm_Horizontal, F.Cu at (183.5, 89.5)
- added R35: 100k, Resistor_THT:R_Axial_DIN0207_L6.3mm_D2.5mm_P10.16mm_Horizontal, F.Cu at (183.5, 100.5)
- added R7: 1k, Resistor_THT:R_Axial_DIN0207_L6.3mm_D2.5mm_P10.16mm_Horizontal, F.Cu at (93.5, 100.5)
- added R8: 100k, Resistor_THT:R_Axial_DIN0207_L6.3mm_D2.5mm_P10.16mm_Horizontal, F.Cu at (93.5, 89.5)
- added SW1: SW_MEC_LOW_PROF_LED, Synth:PB01-109TL, F.Cu at (88.5, 95.0)
- added SW2: SW_MEC_LOW_PROF_LED, Synth:PB01-109TL, F.Cu at (118.5, 95.0)
- added SW3: SW_MEC_LOW_PROF_LED, Synth:PB01-109TL, F.Cu at (148.5, 95.0)
- added SW4: SW_MEC_LOW_PROF_LED, Synth:PB01-109TL, F.Cu at (178.5, 95.0)
- J10: value Bass OUT -> Main OUT
- R32: value 47k -> 1k
- R33: value 47k -> 100k
- moved R36 104.4 mm to (187.6, 128.0), turned to 180 degrees
- moved J10 88.8 mm to (176.0, 135.0), turned to 90 degrees
- moved R33 29.4 mm to (153.6, 89.5), turned to 180 degrees
- moved R40 16.6 mm to (188.0, 120.0), turned to 90 degrees
- moved R32 12.1 mm to (153.5, 100.5), turned to 180 degrees
- moved Q4 8.54 mm to (171.5, 94.0), turned to -90 degrees
- moved Q3 8.48 mm to (141.6, 93.7), turned to -90 degrees
- moved Q1 8.44 mm to (81.6, 93.7), turned to -90 degrees
- moved Q2 8.44 mm to (111.6, 93.7), turned to -90 degrees
- moved VOL1 5.00 mm to (91.0, 120.0)
- moved VOL2 5.00 mm to (151.0, 120.0)
- moved VOL3 5.00 mm to (121.0, 120.0)
- moved VOL4 5.00 mm to (181.0, 120.0)
- moved R37 2.63 mm to (97.0, 120.1), turned to 90 degrees
- moved R38 2.63 mm to (157.0, 120.1), turned to 90 degrees
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- renumbered C13 to C1, C7 to C10, C2 to C11, C8 to C12, C15 to C13, C9 to C14, C3 to C15, C10 to C16, C16 to C17, C11 to C18, C4 to C19, C5 to C2, C12 to C20, C19 to C21, C23 to C22, C20 to C23, C1 to C3, C17 to C4, C18 to C5, C27 to C7, C28 to C8, C14 to C9, D5 to D3, D3 to D4, D4 to D5, J5 to J1, J12 to J11, J13 to J12, J18 to J13, J19 to J14, J14 to J15, J15 to J16, J3 to J2, J1 to J3, J2 to J5, J8 to J7, J7 to J8, R17 to R1, R2 to R10, R7 to R11, R20 to R12, R14 to R13, R8 to R14, R25 to R15, R21 to R17, R3 to R19, R1 to R2, R9 to R20, R22 to R21, R15 to R22, R10 to R25, R23 to R26, R4 to R27, R11 to R28, R24 to R29, R5 to R3, R16 to R30, R12 to R31, R34 to R37, R35 to R39, R18 to R4, R39 to R40, R13 to R5, R19 to R9, VOL3 to VOL2, VOL2 to VOL3
Connections:
- J10 pad T: Out1 -> Net-(J10-PadT)
- R32 pad 1: In3 -> +5V
- R32 pad 2: Net-(Q3-Pad2) -> Net-(Q3-Pad3)
- R33 pad 1: In4 -> In3
- R33 pad 2: Net-(Q4-Pad2) -> Net-(Q3-Pad2)
- R36 pad 1: Out1 -> Net-(J10-PadT)
- R36 pad 2: Net-(R36-Pad2) -> Out1
- U2 pad 1: Net-(R36-Pad2) -> Out1
- U2 pad 13: Net-(R41-Pad2) -> Out1
- U2 pad 14: Net-(R41-Pad2) -> Out1
- U2 pad 2: Net-(R36-Pad2) -> Out1
- U2 pad 6: Net-(R37-Pad2) -> Out1
- U2 pad 7: Net-(R37-Pad2) -> Out1
- U2 pad 8: Net-(R40-Pad2) -> Out1
- U2 pad 9: Net-(R40-Pad2) -> Out1
Routing:
- net +5V: track 0.00 -> 120.1 mm, vias 0 -> 1
- net +12V: track 257.9 -> 168.9 mm, vias 2 -> 0
- net Out1: track 6.48 -> 69.3 mm
- net Net-(R36-Pad2): track 44.0 -> 0.00 mm
- net Net-(R41-Pad2): track 44.0 -> 0.00 mm
- net In4: track 108.2 -> 150.0 mm, vias 0 -> 1
- net In3: track 79.7 -> 96.0 mm, vias 0 -> 1
- net O4: track 185.6 -> 174.7 mm
- net In2: track 49.7 -> 59.6 mm, vias 0 -> 1
- net Net-(R37-Pad2): track 8.84 -> 0.00 mm
- net Net-(R40-Pad2): track 8.82 -> 0.00 mm
- net Net-(J10-PadT): track 0.00 -> 7.07 mm
- net Out4: track 6.48 -> 0.00 mm
- net Out3: track 6.48 -> 0.00 mm
- net Out2: track 6.48 -> 0.00 mm
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
Commit message: Update gerbers for V1.1 of drumbox
Routing:
- net Out1: track 69.3 -> 80.4 mm
Changed lines of the file:
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@@
     (fp_line (start 4 -2.75) (end 4 2.75) (layer "B.CrtYd") (width 0.05))
     (fp_line (start -0.73 1.32665) (end -0.73 -1.32665) (layer "B.Fab") (width 0.1))
-    (fp_arc (start -0.730339 -1.32614) (mid 3.670001 -0.000306) (end -0.73 1.32665) (layer "B.Fab") (width 0.1))
+    (fp_arc (start -0.730339 -1.32614) (mid 3.67 -0.000308) (end -0.73 1.32665) (layer "B.Fab") (width 0.1))
     (fp_circle (center 1.27 0) (end 3.27 0) (layer "B.Fab") (width 0.1) (fill none))
     (pad "1" thru_hole rect (at 0 0 180) (size 1.8 1.8) (drill 0.9) (layers *.Cu *.Mask)
@@
   (segment (start 168.305 137.115) (end 177.42 128) (width 0.3) (layer "F.Cu") (net 38))
   (segment (start 129.7 134.575) (end 129.7 137.115) (width 0.3) (layer "F.Cu") (net 38))
+  (segment (start 136.170489 133.425489) (end 137.32 134.575) (width 0.3) (layer "B.Cu") (net 38))
+  (segment (start 136.170489 125.564511) (end 136.170489 133.425489) (width 0.3) (layer "B.Cu") (net 38))
+  (segment (start 137.32 124.415) (end 136.170489 125.564511) (width 0.3) (layer "B.Cu") (net 38))
   (segment (start 81 95) (end 81.64 95) (width 0.3) (layer "F.Cu") (net 39))
   (segment (start 80.5 92.34) (end 80.5 94.5) (width 0.3) (layer "F.Cu") (net 39))
