File: Mixers/Output-mixer/Stereo input/StereoInputs.kicad_sch (KiCad schematic)
At the start: 0 parts

Commit message: update stereo output mixer
Parts:
- added C? (x6): .1µF, Capacitor_THT:CP_Radial_D5.0mm_P2.00mm, symbol Device:CP
- added R? (x6): 1k, Resistor_THT:R_Axial_DIN0207_L6.3mm_D2.5mm_P10.16mm_Horizontal, symbol Device:R
- added R? (x6): 10k, Resistor_THT:R_Axial_DIN0207_L6.3mm_D2.5mm_P10.16mm_Horizontal, symbol Device:R
- added RV2, RV3, RV4, RV5, RV6, RV7: 50k, Synth:PTV1124420AA503, symbol Device:R_Potentiometer_Dual_Separate
- added U1, U2, U3, U6, U7, U8: TL072, Package_DIP:DIP-8_W7.62mm_Socket, symbol Amplifier_Operational:TL072
Connections:
- new net: C?.1, R?.2 (x6)
- new net: R?.1, R?.2, U7.6 (-)
- new net: R?.1, RV4.6
- new net: R?.1, RV6.6
- new net: R?.1, R?.2, U6.6 (-)
- new net: R?.1, RV2.6
- new net: R?.1, RV5.6
- new net: R?.1, R?.2, U3.6 (-)
- new net: R?.1, R?.2, U2.6 (-)
- new net: R?.1, R?.2, U1.6 (-)
- new net: R?.1, R?.2, U8.6 (-)
- new net: R?.1, RV7.6
- new net: R?.1, RV3.6
- new net GND: U1.5 (+), U2.5 (+), U3.5 (+), U6.5 (+), U7.5 (+), U8.5 (+)
- new net Left1_In: C?.2
- new net Left1_Out: RV2.4, RV2.5, U1.7
- new net Left2_In: C?.2
- new net Left2_Out: RV3.4, RV3.5, U2.7
- new net Left3_In: C?.2
- new net Left3_Out: RV4.4, RV4.5, U3.7
- new net Left4_In: C?.2
- new net Left4_Out: RV5.4, RV5.5, U6.7
- new net Left5_In: C?.2
- new net Left5_Out: RV6.4, RV6.5, U7.7
- new net Left6_In: C?.2
- new net Left6_Out: RV7.4, RV7.5, U8.7

Commit message: finish schem update
Parts:
- added C37, C38, C39, C40, C41, C42: 100nF, Capacitor_THT:C_Disc_D7.0mm_W2.5mm_P5.00mm, symbol Device:C_Small
- added unit 3 of U6
- added unit 3 of U7
- added unit 3 of U8
- gave numbers to parts that had none: 18
- renumbered RV2 to RV8
Connections:
- net GND: now also C37.2, C38.2, C39.2, C40.2, C41.2, C42.2
- new net +12V: C37.1, C39.1, C41.1, U6.8 (V+), U7.8 (V+), U8.8 (V+)
- new net -12V: C38.1, C40.1, C42.1, U6.4 (V-), U7.4 (V-), U8.4 (V-)

Commit message: update schem (not finished)
Parts:
- removed RV8: 50k, Synth:PTV1124420AA503, symbol Device:R_Potentiometer_Dual_Separate
Connections:
- net Left1_Out: no longer U1.7

Commit message: finish update schem
Parts:
- added J27, J28, J29, J30, J35, J36: Conn_01x06_Female, Connector_PinSocket_2.54mm:PinSocket_1x06_P2.54mm_Vertical, symbol Connector:Conn_01x06_Female
- added J31, J32, J33, J34, J37, J38: Conn_01x06_Male, Connector_PinHeader_2.54mm:PinHeader_1x06_P2.54mm_Vertical, symbol Connector:Conn_01x06_Male
- added RV9: 50k, Synth:PTV1124420AA503, symbol Device:R_Potentiometer_Dual_Separate
Connections:
- net Left1_In: now also J27.1 (Pin_1), J31.1 (Pin_1)
- net Left1_Out: now also U1.7, J27.2 (Pin_2), J31.2 (Pin_2), RV9.4, RV9.5
- net Left2_In: now also J28.1 (Pin_1), J32.1 (Pin_1)
- net Left2_Out: now also J28.2 (Pin_2), J32.2 (Pin_2)
- net Left3_In: now also J29.1 (Pin_1), J33.1 (Pin_1)
- net Left3_Out: now also J29.2 (Pin_2), J33.2 (Pin_2)
- net Left4_In: now also J30.1 (Pin_1), J34.1 (Pin_1)
- net Left4_Out: now also J30.2 (Pin_2), J34.2 (Pin_2)
- net Left5_In: now also J35.1 (Pin_1), J37.1 (Pin_1)
- net Left5_Out: now also J35.2 (Pin_2), J37.2 (Pin_2)
- net Left6_In: now also J36.1 (Pin_1), J38.1 (Pin_1)
- net Left6_Out: now also J36.2 (Pin_2), J38.2 (Pin_2)
- net Left3_GOut: now reaches R73.1, RV4.6
- net Left3_GOut: now also J29.3 (Pin_3), J33.3 (Pin_3)
- net Left5_GOut: now reaches R75.1, RV6.6
- net Left5_GOut: now also J35.3 (Pin_3), J37.3 (Pin_3)
- net Left4_GOut: now reaches R74.1, RV5.6
- net Left4_GOut: now also J30.3 (Pin_3), J34.3 (Pin_3)
- net Left6_GOut: now reaches R76.1, RV7.6
- net Left6_GOut: now also J36.3 (Pin_3), J38.3 (Pin_3)
- net Left2_GOut: now reaches R72.1, RV3.6
- net Left2_GOut: now also J28.3 (Pin_3), J32.3 (Pin_3)
- net Left1_GOut: now reaches R71.1
- net Left1_GOut: now also J27.3 (Pin_3), J31.3 (Pin_3), RV9.6
- new net Right1_GOut: J27.6 (Pin_6), J31.6 (Pin_6)
- new net Right1_In: J27.4 (Pin_4), J31.4 (Pin_4)
- new net Right1_Out: J27.5 (Pin_5), J31.5 (Pin_5)
- new net Right2_GOut: J28.6 (Pin_6), J32.6 (Pin_6)
- new net Right2_In: J28.4 (Pin_4), J32.4 (Pin_4)
- new net Right2_Out: J28.5 (Pin_5), J32.5 (Pin_5)
- new net Right3_GOut: J29.6 (Pin_6), J33.6 (Pin_6)
- new net Right3_In: J29.4 (Pin_4), J33.4 (Pin_4)
- new net Right3_Out: J29.5 (Pin_5), J33.5 (Pin_5)
- new net Right4_GOut: J30.6 (Pin_6), J34.6 (Pin_6)
- new net Right4_In: J30.4 (Pin_4), J34.4 (Pin_4)
- new net Right4_Out: J30.5 (Pin_5), J34.5 (Pin_5)
- new net Right5_GOut: J35.6 (Pin_6), J37.6 (Pin_6)
- new net Right5_In: J35.4 (Pin_4), J37.4 (Pin_4)
- new net Right5_Out: J35.5 (Pin_5), J37.5 (Pin_5)
- new net Right6_GOut: J36.6 (Pin_6), J38.6 (Pin_6)
- new net Right6_In: J36.4 (Pin_4), J38.4 (Pin_4)
- new net Right6_Out: J36.5 (Pin_5), J38.5 (Pin_5)

Commit message: early board update
Parts:
- added J39: Conn_01x04_Male, Connector_PinHeader_2.54mm:PinHeader_1x04_P2.54mm_Vertical, symbol Connector:Conn_01x04_Male
- added J40: Conn_01x04_Female, Connector_PinSocket_2.54mm:PinSocket_1x04_P2.54mm_Vertical, symbol Connector:Conn_01x04_Female
- renumbered R1 to R65, R2 to R66, R3 to R67, R4 to R68, R5 to R69, R6 to R70, RV9 to RV1, RV3 to RV2, RV4 to RV3, RV5 to RV4, RV6 to RV5, RV7 to RV6, U6 to U4, U7 to U5, U8 to U6
Connections:
- net +12V: now also J39.1 (Pin_1), J40.1 (Pin_1)
- net -12V: now also J39.4 (Pin_4), J40.4 (Pin_4)
- net GND: now also J39.2 (Pin_2), J39.3 (Pin_3), J40.2 (Pin_2), J40.3 (Pin_3)
