File: HiHat + Snare/V1.1/JackBoard/Snare+Hihat.kicad_pcb (KiCad board)
At the start: 2 copper layers, 40 x 110 mm, 36 parts, among them J1 Snare IN, J10 Conn_01x03_Female, J3 HiHat IN, J4 Snare OUT, J6 Conn_01x08_Female, J8 Conn_01x08_Female, J9 HiHat OUT, Q4 2N3904, Q8 2N3904, U1 TL072

Commit message: add gerber files
Parts:
- added C10: .1µF, Capacitor_THT:C_Disc_D7.0mm_W2.5mm_P5.00mm, F.Cu at (54.5, 111.2)
- added C15: 10µF, Capacitor_THT:CP_Radial_D5.0mm_P2.00mm, B.Cu at (34.0, 74.5)
- added C16: 10µF, Capacitor_THT:CP_Radial_D5.0mm_P2.00mm, B.Cu at (39.5, 61.0)
- added C17: 1µF, Capacitor_THT:C_Disc_D7.0mm_W2.5mm_P5.00mm, F.Cu at (45.0, 92.6)
- added C18: 10nF, Capacitor_THT:C_Disc_D7.0mm_W2.5mm_P5.00mm, F.Cu at (45.0, 95.6)
- added C19: 680pF, Capacitor_THT:C_Disc_D7.0mm_W2.5mm_P5.00mm, F.Cu at (39.0, 111.2)
- added C20: .1µF, Capacitor_THT:C_Disc_D7.0mm_W2.5mm_P5.00mm, F.Cu at (44.0, 108.0)
- added C22: 100µ, Capacitor_THT:CP_Radial_D5.0mm_P2.00mm, B.Cu at (47.2, 99.2)
- added C23: 100µ, Capacitor_THT:CP_Radial_D5.0mm_P2.00mm, B.Cu at (53.0, 99.2)
- added C24: 22pF, Capacitor_THT:C_Disc_D7.0mm_W2.5mm_P5.00mm, F.Cu at (94.9, 107.1)
- added C25: 22pF, Capacitor_THT:C_Disc_D7.0mm_W2.5mm_P5.00mm, F.Cu at (91.1, 107.1)
- added C4: 10µF, Capacitor_THT:CP_Radial_D5.0mm_P2.00mm, B.Cu at (60.8, 75.0)
- added C7: 10µF, Capacitor_THT:CP_Radial_D5.0mm_P2.00mm, B.Cu at (66.2, 61.5)
- added C8: 1µF, Capacitor_THT:C_Disc_D7.0mm_W2.5mm_P5.00mm, F.Cu at (55.0, 92.6)
- added C9: 0.1µF, Capacitor_THT:C_Disc_D7.0mm_W2.5mm_P5.00mm, F.Cu at (55.0, 95.6)
- added D1: 1N4148, Diode_THT:D_DO-35_SOD27_P7.62mm_Horizontal, F.Cu at (58.8, 70.0)
- added D2: 1N4148, Diode_THT:D_DO-35_SOD27_P7.62mm_Horizontal, F.Cu at (61.8, 62.4)
- added D3: 1N4148, Diode_THT:D_DO-35_SOD27_P7.62mm_Horizontal, F.Cu at (55.0, 88.2)
- added D4: LED-12V, LED_THT:LED_D4.0mm, B.Cu at (59.0, 120.5)
- added D6: 1N4148, Diode_THT:D_DO-35_SOD27_P7.62mm_Horizontal, F.Cu at (32.5, 69.5)
- added D7: 1N4148, Diode_THT:D_DO-35_SOD27_P7.62mm_Horizontal, F.Cu at (35.0, 61.9)
- added D8: 1N4148, Diode_THT:D_DO-35_SOD27_P7.62mm_Horizontal, F.Cu at (45.0, 88.2)
- added FB1: 10R, Inductor_THT:L_Axial_L9.5mm_D4.0mm_P12.70mm_Horizontal_Fastron_SMCC, B.Cu at (63.0, 125.2)
- added FB2: 10R, Inductor_THT:L_Axial_L9.5mm_D4.0mm_P12.70mm_Horizontal_Fastron_SMCC, B.Cu at (37.0, 125.2)
- added J11: Conn_01x03_Male, Connector_PinHeader_2.54mm:PinHeader_1x03_P2.54mm_Vertical, F.Cu at (52.5, 137.5)
- added J2: Power Input, Connector_IDC:IDC-Header_2x05_P2.54mm_Vertical, B.Cu at (44.9, 130.0)
- added J5: Conn_01x08_Male, Connector_PinHeader_2.54mm:PinHeader_1x08_P2.54mm_Vertical, F.Cu at (68.0, 98.5)
- added J7: Conn_01x08_Male, Connector_PinHeader_2.54mm:PinHeader_1x08_P2.54mm_Vertical, F.Cu at (32.0, 98.5)
- added Q1: BC546, Package_TO_SOT_THT:TO-92_Inline, F.Cu at (64.0, 83.6)
- added Q2: BC546, Package_TO_SOT_THT:TO-92_Inline, F.Cu at (59.0, 83.6)
- added Q3: BC546, Package_TO_SOT_THT:TO-92_Inline, F.Cu at (59.0, 89.1)
- added Q5: BC546, Package_TO_SOT_THT:TO-92_Inline, F.Cu at (36.5, 83.1)
- added Q6: BC546, Package_TO_SOT_THT:TO-92_Inline, F.Cu at (41.5, 83.1)
- added Q7: BC546, Package_TO_SOT_THT:TO-92_Inline, F.Cu at (41.5, 88.6)
- added R1: 4k7, Resistor_THT:R_Axial_DIN0207_L6.3mm_D2.5mm_P10.16mm_Horizontal, F.Cu at (65.2, 75.0)
- added R10: 0R, Resistor_THT:R_Axial_DIN0207_L6.3mm_D2.5mm_P10.16mm_Horizontal, F.Cu at (61.5, 114.5)
- added R12: 4k7, Resistor_THT:R_Axial_DIN0207_L6.3mm_D2.5mm_P10.16mm_Horizontal, F.Cu at (38.5, 74.5)
- added R13: 47k, Resistor_THT:R_Axial_DIN0207_L6.3mm_D2.5mm_P10.16mm_Horizontal, F.Cu at (36.5, 86.1)
- added R14: 4k7, Resistor_THT:R_Axial_DIN0207_L6.3mm_D2.5mm_P10.16mm_Horizontal, F.Cu at (48.0, 80.6)
- added R15: 1M, Resistor_THT:R_Axial_DIN0207_L6.3mm_D2.5mm_P10.16mm_Horizontal, F.Cu at (35.8, 117.3)
- added R17: 1M, Resistor_THT:R_Axial_DIN0207_L6.3mm_D2.5mm_P10.16mm_Horizontal, F.Cu at (35.2, 104.5)
- added R18: 10k, Resistor_THT:R_Axial_DIN0207_L6.3mm_D2.5mm_P2.54mm_Vertical, F.Cu at (97.4, 115.5)
- added R2: 47k, Resistor_THT:R_Axial_DIN0207_L6.3mm_D2.5mm_P10.16mm_Horizontal, F.Cu at (64.0, 86.6)
- added R20: 330k, Resistor_THT:R_Axial_DIN0207_L6.3mm_D2.5mm_P2.54mm_Vertical, F.Cu at (99.6, 110.3)
- added R22: 10k, Resistor_THT:R_Axial_DIN0207_L6.3mm_D2.5mm_P2.54mm_Vertical, F.Cu at (88.6, 115.5)
- added R23: 330k, Resistor_THT:R_Axial_DIN0207_L6.3mm_D2.5mm_P2.54mm_Vertical, F.Cu at (86.3, 110.3)
- added R3: 4k7, Resistor_THT:R_Axial_DIN0207_L6.3mm_D2.5mm_P10.16mm_Horizontal, F.Cu at (52.0, 80.6)
- added R4: 1M, Resistor_THT:R_Axial_DIN0207_L6.3mm_D2.5mm_P10.16mm_Horizontal, F.Cu at (64.2, 117.0)
- added R6: 2.2k, Resistor_THT:R_Axial_DIN0207_L6.3mm_D2.5mm_P10.16mm_Horizontal, F.Cu at (43.4, 120.5)
- added R7: 1M, Resistor_THT:R_Axial_DIN0207_L6.3mm_D2.5mm_P10.16mm_Horizontal, F.Cu at (61.6, 108.0)
- added R8: 0R, Resistor_THT:R_Axial_DIN0207_L6.3mm_D2.5mm_P10.16mm_Horizontal, F.Cu at (38.8, 114.5)
- DECAY1, DECAY2, Strike1, Strike2, VOL1, VOL2: footprint Potentiometer_THT:Potentiometer_Bourns_PTV09A-1_Single_Vertical -> Synth:Pot-bourns-alpha
- J1, J3, J4, J9: footprint Connector_Audio:Jack_3.5mm_QingPu_WQP-PJ398SM_Vertical_CircularHoles -> Synth:Thonkiconn
- R16, R19, R5, R9: footprint Resistor_THT:R_Axial_DIN0207_L6.3mm_D2.5mm_P10.16mm_Horizontal -> Resistor_THT:R_Axial_DIN0207_L6.3mm_D2.5mm_P2.54mm_Vertical
- moved R9 23.9 mm to (96.0, 99.6), turned to 90 degrees
- moved C14 23.1 mm to (91.1, 88.9)
- moved R5 22.2 mm to (97.6, 102.8), turned to 0 degrees
- moved Q8 22.1 mm to (80.7, 103.9)
- moved C1 22.1 mm to (102.5, 70.0)
- moved C11 22.1 mm to (80.5, 70.0)
- moved C12 22.1 mm to (111.0, 121.0)
- moved C13 22.1 mm to (83.5, 70.0)
- moved C2 22.1 mm to (105.0, 70.0)
- moved C21 22.1 mm to (75.0, 121.0)
- moved C5 22.1 mm to (95.0, 132.5)
- moved C6 22.1 mm to (91.0, 132.5)
- moved D5 22.1 mm to (102.7, 109.0)
- moved DECAY1 22.1 mm to (106.5, 44.5)
- moved DECAY2 22.1 mm to (84.5, 44.5)
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Connections:
- C12 pad 1: Net-(U1-Pad2) -> Net-(C12-Pad1)
- U1 pad 1: Net-(U1-Pad2) -> Net-(C12-Pad1)
- U1 pad 6: Net-(C21-Pad1) -> Net-(U1-Pad6)
Routing:
- net +12V: track 39.2 -> 170.1 mm
- net /So: track 54.1 -> 105.8 mm
- net /SnH: track 84.2 -> 134.3 mm
- net /HiH: track 78.8 -> 128.3 mm
- net /Ho: track 52.1 -> 93.5 mm
- net /DeH: track 79.0 -> 117.1 mm
- net /HiDH: track 71.9 -> 108.3 mm
- net /HiI: track 24.3 -> 59.7 mm
- net /SnI: track 24.3 -> 58.5 mm
- net Net-(C12-Pad1): track 0.00 -> 32.6 mm
- net -12V: track 27.2 -> 56.5 mm
- net Net-(C8-Pad1): track 0.00 -> 25.5 mm
- net Net-(C17-Pad1): track 0.00 -> 25.4 mm
- net Net-(C17-Pad2): track 0.00 -> 22.8 mm
- net Net-(C8-Pad2): track 0.00 -> 22.3 mm
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Other:
- board size 40 x 110 mm -> 127.5 x 128 mm
- board text added: "8HP"
- board text added: "Board 1/2"
- board text added: "Snare + HiHat V1.1 BleepSound 2022"
- board text removed: "Snare + HiHat V1.0 BleepSound 2022"

Commit message: gerber creation
Parts:
- removed C10, C20: .1µF, Capacitor_THT:C_Disc_D7.0mm_W2.5mm_P5.00mm
- removed C15, C16, C4, C7: 10µF, Capacitor_THT:CP_Radial_D5.0mm_P2.00mm
- removed C17, C8: 1µF, Capacitor_THT:C_Disc_D7.0mm_W2.5mm_P5.00mm
- removed C18: 10nF, Capacitor_THT:C_Disc_D7.0mm_W2.5mm_P5.00mm
- removed C19: 680pF, Capacitor_THT:C_Disc_D7.0mm_W2.5mm_P5.00mm
- removed C22, C23: 100µ, Capacitor_THT:CP_Radial_D5.0mm_P2.00mm
- removed C9: 0.1µF, Capacitor_THT:C_Disc_D7.0mm_W2.5mm_P5.00mm
- removed D1, D2, D3, D6, D7, D8: 1N4148, Diode_THT:D_DO-35_SOD27_P7.62mm_Horizontal
- removed D4: LED-12V, LED_THT:LED_D4.0mm
- removed FB1, FB2: 10R, Inductor_THT:L_Axial_L9.5mm_D4.0mm_P12.70mm_Horizontal_Fastron_SMCC
- removed J11: Conn_01x03_Male, Connector_PinHeader_2.54mm:PinHeader_1x03_P2.54mm_Vertical
- removed J2: Power Input, Connector_IDC:IDC-Header_2x05_P2.54mm_Vertical
- removed J5, J7: Conn_01x08_Male, Connector_PinHeader_2.54mm:PinHeader_1x08_P2.54mm_Vertical
- removed Q1, Q2, Q3, Q5, Q6, Q7: BC546, Package_TO_SOT_THT:TO-92_Inline
- removed R1, R12, R14, R3: 4k7, Resistor_THT:R_Axial_DIN0207_L6.3mm_D2.5mm_P10.16mm_Horizontal
- removed R10, R8: 0R, Resistor_THT:R_Axial_DIN0207_L6.3mm_D2.5mm_P10.16mm_Horizontal
- removed R13, R2: 47k, Resistor_THT:R_Axial_DIN0207_L6.3mm_D2.5mm_P10.16mm_Horizontal
- removed R15, R17, R4, R7: 1M, Resistor_THT:R_Axial_DIN0207_L6.3mm_D2.5mm_P10.16mm_Horizontal
- removed R6: 2.2k, Resistor_THT:R_Axial_DIN0207_L6.3mm_D2.5mm_P10.16mm_Horizontal
Routing:
- net +12V: track 170.1 -> 49.2 mm
- net /So: track 105.8 -> 54.1 mm
- net /HiH: track 128.3 -> 77.0 mm
- net /SnH: track 134.3 -> 83.1 mm
- net /Ho: track 93.5 -> 52.1 mm
- net /DeH: track 117.1 -> 79.2 mm
- net /HiDH: track 108.3 -> 72.3 mm
- net /HiI: track 59.7 -> 24.3 mm
- net /SnI: track 58.5 -> 24.3 mm
- net -12V: track 56.5 -> 26.9 mm
- net Net-(C8-Pad1): track 25.5 -> 0.00 mm
- net Net-(C17-Pad1): track 25.4 -> 0.00 mm
- net Net-(C17-Pad2): track 22.8 -> 0.00 mm
- net Net-(C8-Pad2): track 22.3 -> 0.00 mm
- net /HiO: track 55.9 -> 35.1 mm
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Other:
- board size 127.5 x 128 mm -> 40 x 110 mm
- board text removed: "8HP"
- board text removed: "Board 1/2"
