File: HiHat + Snare/V1.1/Kicad/Snare+Hihat.kicad_pcb (KiCad board)
At the start: 2 copper layers, 127.5 x 128 mm, 87 parts, among them J1 Snare IN, J10 Conn_01x03_Female, J11 Conn_01x03_Male, J2 Power Input, J3 HiHat IN, J4 Snare OUT, J5 Conn_01x08_Male, J6 Conn_01x08_Female, J7 Conn_01x08_Male, J8 Conn_01x08_Female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

Commit message: update hihat + snare (functionnal) no gerber update yet
Parts:
- C15, C16, C22, C23, C4, C7, FB1, FB2: moved to B.Cu
- DECAY1, DECAY2, Strike1, Strike2, VOL1, VOL2: footprint Potentiometer_THT:Potentiometer_Bourns_PTV09A-1_Single_Vertical -> Synth:Pot-bourns-alpha
- J1, J3, J4, J9: footprint Connector_Audio:Jack_3.5mm_QingPu_WQP-PJ398SM_Vertical_CircularHoles -> Synth:Thonkiconn
- J2: footprint Connector_PinHeader_2.54mm:PinHeader_2x05_P2.54mm_Vertical -> Connector_IDC:IDC-Header_2x05_P2.54mm_Vertical
- R16, R18, R19, R20, R22, R23, R5, R9: footprint Resistor_THT:R_Axial_DIN0207_L6.3mm_D2.5mm_P10.16mm_Horizontal -> Resistor_THT:R_Axial_DIN0207_L6.3mm_D2.5mm_P2.54mm_Vertical
- moved C25 50.2 mm to (91.1, 107.1), turned to 180 degrees
- moved R20 49.8 mm to (99.6, 110.3), turned to 180 degrees
- moved C24 48.4 mm to (94.9, 107.1)
- moved R23 42.4 mm to (86.3, 110.3)
- moved R22 33.6 mm to (88.6, 115.5), turned to 90 degrees
- moved R18 33.5 mm to (97.4, 115.5), turned to 90 degrees
- moved D4 29.2 mm to (59.0, 120.5), turned to 180 degrees
- moved FB1 24.1 mm to (63.0, 125.2)
- moved FB2 24.1 mm to (37.0, 125.2)
- moved R6 9.42 mm to (43.4, 120.5), turned to 0 degrees
- moved R19 6.42 mm to (90.0, 99.6), turned to 90 degrees
- moved R9 6.37 mm to (96.0, 99.6), turned to 90 degrees
- moved R16 3.04 mm to (88.4, 102.8), turned to 180 degrees
- moved R5 3.04 mm to (97.6, 102.8), turned to 0 degrees
- moved C14 1.10 mm to (91.1, 88.9)
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Connections:
- J2 pad 1: Net-(FB1-Pad2) -> Net-(FB2-Pad2)
- J2 pad 10: Net-(FB2-Pad2) -> Net-(FB1-Pad2)
- J2 pad 2: Net-(FB1-Pad2) -> Net-(FB2-Pad2)
- J2 pad 9: Net-(FB2-Pad2) -> Net-(FB1-Pad2)
Routing:
- net Net-(U1-Pad2): track 0.00 -> 19.6 mm
- net +12V: track 151.2 -> 170.1 mm
- net Net-(U1-Pad6): track 0.00 -> 16.8 mm
- net Net-(C12-Pad1): track 17.9 -> 32.6 mm
- net Net-(C21-Pad1): track 17.9 -> 32.2 mm
- net Net-(Q4-Pad2): track 16.1 -> 5.26 mm
- net Net-(Q8-Pad2): track 15.7 -> 5.32 mm
- net Net-(Q4-Pad3): track 16.3 -> 9.28 mm
- net Net-(Q8-Pad3): track 15.5 -> 9.68 mm
- net Net-(FB2-Pad2): track 8.03 -> 12.7 mm
- net Net-(FB1-Pad2): track 8.03 -> 12.7 mm
- net -12V: track 59.6 -> 56.8 mm
- net Net-(U1-Pad5): track 40.9 -> 42.6 mm
- net Net-(C14-Pad2): track 7.75 -> 9.30 mm
- net /HiH: track 130.1 -> 128.6 mm
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
Commit message: add gerber files
Routing:
- net Net-(U1-Pad3): track 44.2 -> 43.6 mm
Other:
- board text added: "Front panel"
Changed lines of the file:
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@@
     (property "Sheetname" "")
     (attr through_hole)
-    (fp_text reference "J1" (at -4.03 1.08 180) (layer "F.SilkS")
+    (fp_text reference "J1" (at 3.8 1.08 180) (layer "F.SilkS")
       (effects (font (size 1 1) (thickness 0.15)))
     )
@@
   (gr_line (start 30 31) (end 69.999999 31) (layer "Edge.Cuts") (width 0.05))
   (gr_line (start 30 141) (end 70 141) (layer "Edge.Cuts") (width 0.05))
+  (gr_text "Snare + HiHat\nV1.1 BleepSound\n2022" (at 137.5 66.9) (layer "B.SilkS")
+    (effects (font (size 1 1) (thickness 0.15)) (justify mirror))
+  )
   (gr_text "JLCJLCJLCJLC\n" (at 79 32.5) (layer "B.SilkS")
     (effects (font (size 1 1) (thickness 0.15)) (justify mirror))
@@
     (effects (font (size 1 1) (thickness 0.15)) (justify mirror))
   )
+  (gr_text "Front panel" (at 137.5 70.5) (layer "B.SilkS")
+    (effects (font (size 1 1) (thickness 0.15)) (justify mirror))
+  )
   (gr_text "JLCJLCJLCJLC\n" (at 36 139.5) (layer "F.SilkS")
     (effects (font (size 1 1) (thickness 0.15)))
@@
   (segment (start 35 140) (end 34.5 139.5) (width 0.3) (layer "F.Cu") (net 3))
   (segment (start 47.445 137.5) (end 40 137.5) (width 0.3) (layer "F.Cu") (net 3))
-  (segment (start 89.2 132.3) (end 89 132.5) (width 0.3) (layer "F.Cu") (net 3))
   (segment (start 96.5 129.5) (end 90.86863 129.5) (width 0.3) (layer "B.Cu") (net 3))
   (segment (start 90.86863 129.5) (end 89 131.36863) (width 0.3) (layer "B.Cu") (net 3))
@@
   (segment (start 111 128.34) (end 111 126) (width 0.3) (layer "F.Cu") (net 9))
   (segment (start 89.7 93.9) (end 84.4 99.2) (width 0.3) (layer "B.Cu") (net 10))
-  (segment (start 84.8 99.2) (end 84.4 99.2) (width 0.3) (layer "B.Cu") (net 10))
   (segment (start 91.1 93.9) (end 89.7 93.9) (width 0.3) (layer "B.Cu") (net 10))
   (segment (start 105.27 103.14) (end 105.27 108.995) (width 0.3) (layer "B.Cu") (net 11))
@@
   (segment (start 77 119.9) (end 82 124.9) (width 0.3) (layer "B.Cu") (net 25))
   (segment (start 75 103.54) (end 77 105.54) (width 0.3) (layer "B.Cu") (net 25))
-  (segment (start 75.24 105.84) (end 75 106.08) (width 0.3) (layer "F.Cu") (net 26))
   (segment (start 83.6 45.4) (end 83.6 64.15) (width 0.3) (layer "F.Cu") (net 26))
   (segment (start 39.5 61) (end 35.88 61) (width 0.3) (layer "F.Cu") (net 26))
@@
   (segment (start 83.634999 102.000001) (end 82 103.635) (width 0.3) (layer "F.Cu") (net 52))
   (segment (start 85.060001 102.000001) (end 83.634999 102.000001) (width 0.3) (layer "F.Cu") (net 52))
-  (segment (start 82 103.86) (end 82 104.085) (width 0.3) (layer "B.Cu") (net 52))
   (segment (start 82 139.4) (end 75.82 139.4) (width 0.3) (layer "F.Cu") (net 53))
   (segment (start 75.82 139.4) (end 75 138.58) (width 0.3) (layer "F.Cu") (net 53))
@@
   (segment (start 84.4 94.5) (end 84.3 94.5) (width 0.3) (layer "F.Cu") (net 55))
   (segment (start 93.350489 93.043165) (end 98.893654 87.5) (width 0.3) (layer "B.Cu") (net 56))
-  (segment (start 104 85) (end 103.374345 85) (width 0.3) (layer "B.Cu") (net 56))
   (segment (start 96.8 121.22) (end 93.350489 117.770489) (width 0.3) (layer "B.Cu") (net 56))
   (segment (start 93.350489 117.770489) (end 93.350489 93.043165) (width 0.3) (layer "B.Cu") (net 56))

Commit message: gerber creation
Routing:
- net GND: vias 6 -> 14
Changed lines of the file:
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@@
   (via (at 126.5 57.55) (size 6.8) (drill 6) (layers "F.Cu" "B.Cu") (net 0))
   (via (at 50 45.5) (size 3.6) (drill 3.1) (layers "F.Cu" "B.Cu") (net 1))
+  (via (at 111 90) (size 0.8) (drill 0.4) (layers "F.Cu" "B.Cu") (free) (net 1))
+  (via (at 111 91) (size 0.8) (drill 0.4) (layers "F.Cu" "B.Cu") (free) (net 1))
+  (via (at 111 89) (size 0.8) (drill 0.4) (layers "F.Cu" "B.Cu") (free) (net 1))
+  (via (at 111 88) (size 0.8) (drill 0.4) (layers "F.Cu" "B.Cu") (free) (net 1))
   (via (at 84 67.5) (size 0.8) (drill 0.4) (layers "F.Cu" "B.Cu") (free) (net 1))
+  (via (at 107.5 110.5) (size 0.8) (drill 0.4) (layers "F.Cu" "B.Cu") (free) (net 1))
   (via (at 93 45.5) (size 3.6) (drill 3.1) (layers "F.Cu" "B.Cu") (net 1))
+  (via (at 107.5 111.5) (size 0.8) (drill 0.4) (layers "F.Cu" "B.Cu") (free) (net 1))
   (via (at 85 67.5) (size 0.8) (drill 0.4) (layers "F.Cu" "B.Cu") (free) (net 1))
   (via (at 79.5 67.5) (size 0.8) (drill 0.4) (layers "F.Cu" "B.Cu") (free) (net 1))
   (via (at 78.5 67.5) (size 0.8) (drill 0.4) (layers "F.Cu" "B.Cu") (free) (net 1))
+  (via (at 107.5 104.3) (size 0.8) (drill 0.4) (layers "F.Cu" "B.Cu") (free) (net 1))
+  (via (at 107.5 102) (size 0.8) (drill 0.4) (layers "F.Cu" "B.Cu") (free) (net 1))
   (segment (start 43.42 120.5) (end 46.92 117) (width 0.3) (layer "F.Cu") (net 2))
   (segment (start 89.18 126.3) (end 93.1 122.38) (width 0.3) (layer "F.Cu") (net 2))
@@
   (segment (start 111 108.62) (end 109.12 108.62) (width 0.3) (layer "F.Cu") (net 42))
   (via (at 108 107.5) (size 0.8) (drill 0.4) (layers "F.Cu" "B.Cu") (net 42))
+  (segment (start 109 100.5) (end 109 87.5) (width 0.3) (layer "B.Cu") (net 42))
   (segment (start 63.25 109.75) (end 61 109.75) (width 0.3) (layer "B.Cu") (net 42))
-  (segment (start 109 100) (end 109 87.5) (width 0.3) (layer "B.Cu") (net 42))
+  (segment (start 61 109.75) (end 59.5 111.25) (width 0.3) (layer "B.Cu") (net 42))
+  (segment (start 108.6 105.232893) (end 108.6 100.9) (width 0.3) (layer "B.Cu") (net 42))
+  (segment (start 108.6 100.9) (end 109 100.5) (width 0.3) (layer "B.Cu") (net 42))
   (segment (start 109 87.5) (end 106.5 85) (width 0.3) (layer "B.Cu") (net 42))
-  (segment (start 61 109.75) (end 59.5 111.25) (width 0.3) (layer "B.Cu") (net 42))
-  (segment (start 108 101) (end 109 100) (width 0.3) (layer "B.Cu") (net 42))
   (segment (start 64.34 108.66) (end 63.25 109.75) (width 0.3) (layer "B.Cu") (net 42))
+  (segment (start 108.5 105.332893) (end 108.6 105.232893) (width 0.3) (layer "B.Cu") (net 42))
+  (segment (start 108.5 107) (end 108.5 105.332893) (width 0.3) (layer "B.Cu") (net 42))
+  (segment (start 108 107.5) (end 108.5 107) (width 0.3) (layer "B.Cu") (net 42))
   (segment (start 68 108.66) (end 64.34 108.66) (width 0.3) (layer "B.Cu") (net 42))
-  (segment (start 108 107.5) (end 108 101) (width 0.3) (layer "B.Cu") (net 42))
   (segment (start 35.17 104.5) (end 36.75 104.5) (width 0.3) (layer "F.Cu") (net 43))
   (segment (start 38.34 108.66) (end 32 108.66) (width 0.3) (layer "F.Cu") (net 43))
