File: ms20_vcf/simple/Front/MS20-VCF.kicad_pcb (KiCad board)
At the start: 2 copper layers, 50 x 128 mm, 4 parts

Commit message: fix issues on ms20 vcf
Parts:
- moved H1 0.50 mm to (111.0, 30.0)
- moved H2 0.50 mm to (145.0, 30.0)
Other:
- board size 50 x 128 mm -> 50 x 128.5 mm
- board text added: "MS-20 VCF Face plate V1.1 BleepSound 2022"
- board text removed: "MS-20 VCF Face plate V1.0 BleepSound 2022"
