File: ms20_vcf/simple/JackBoard/MS20-VCF.kicad_pcb (KiCad board)
At the start: 2 copper layers, 50 x 110 mm, 55 parts, among them J5 Power Input, J6 FilterCV1, J7 FilterIn1, J8 FilterOut1, Q1 BC559, Q2 BC559, SW1 Hpass/Lpass Switch, U1 LM13700, U2 TL072

Commit message: fix issues on ms20 vcf
Connections:
- CUTCV1 pad 1: GND -> /CVIn
- CUTCV1 pad 3: /CVIn -> GND
- CUTOFF1 pad 3: Net-(CUTOFF1-Pad3) -> Net-(R18-Pad2)
- R17 pad 1: Net-(CUTOFF1-Pad3) -> Net-(CUTOFF1-Pad1)
- R18 pad 2: Net-(CUTOFF1-Pad1) -> Net-(R18-Pad2)
- Res1 pad 1: GND -> Net-(R21-Pad1)
- Res1 pad 3: Net-(R21-Pad1) -> GND
Routing:
- net Net-(R18-Pad2): track 0.00 -> 14.6 mm
- net Net-(CUTOFF1-Pad3): track 11.5 -> 0.00 mm
- net Net-(CUTOFF1-Pad1): track 18.9 -> 15.9 mm
- net Net-(R21-Pad1): track 9.59 -> 7.51 mm
- net /CVIn: track 21.0 -> 18.9 mm
Other:
- board text added: "12HP"
- board text added: "MS-20 VCF V1.1 BleepSound 2022"
- board text removed: "MS-20 VCF V1.0 BleepSound 2022"
Changed lines of the file:
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@@
       (svguseinch false)
       (svgprecision 6)
-      (excludeedgelayer false)
+      (excludeedgelayer true)
       (plotframeref false)
       (viasonmask false)
@@
   (net 12 "/HPass")
   (net 13 "/Out1")
-  (net 14 "Net-(CUTCV1-Pad2)")
+  (net 14 "Net-(R14-Pad2)")
   (net 15 "/CVIn")
   (net 16 "Net-(CUTOFF1-Pad1)")
-  (net 17 "Net-(CUTOFF1-Pad2)")
-  (net 18 "Net-(CUTOFF1-Pad3)")
+  (net 17 "Net-(R15-Pad2)")
+  (net 18 "Net-(R18-Pad2)")
   (net 19 "Net-(D1-Pad2)")
   (net 20 "Net-(D2-Pad2)")
@@
     (pad "" np_thru_hole circle (at 7 -6.9 90) (size 4 4) (drill 2) (layers *.Cu *.Mask))
     (pad "1" thru_hole circle (at 0 0 90) (size 1.8 1.8) (drill 1) (layers *.Cu *.Mask)
-      (net 1 "GND") (pinfunction "1") (pintype "passive"))
+      (net 15 "/CVIn") (pinfunction "1") (pintype "passive"))
     (pad "2" thru_hole circle (at 0 -2.5 90) (size 1.8 1.8) (drill 1) (layers *.Cu *.Mask)
-      (net 14 "Net-(CUTCV1-Pad2)") (pinfunction "2") (pintype "passive"))
+      (net 14 "Net-(R14-Pad2)") (pinfunction "2") (pintype "passive"))
     (pad "3" thru_hole circle (at 0 -5 90) (size 1.8 1.8) (drill 1) (layers *.Cu *.Mask)
-      (net 15 "/CVIn") (pinfunction "3") (pintype "passive"))
+      (net 1 "GND") (pinfunction "3") (pintype "passive"))
     (model "${KICAD6_3DMODEL_DIR}/Potentiometer_THT.3dshapes/RK09K1130AH1.STEP"
       (offset (xyz 7 2.5 0))
@@
       (net 16 "Net-(CUTOFF1-Pad1)") (pinfunction "1") (pintype "passive"))
     (pad "2" thru_hole circle (at 0 -2.5 90) (size 1.8 1.8) (drill 1) (layers *.Cu *.Mask)
-      (net 17 "Net-(CUTOFF1-Pad2)") (pinfunction "2") (pintype "passive"))
+      (net 17 "Net-(R15-Pad2)") (pinfunction "2") (pintype "passive"))
     (pad "3" thru_hole circle (at 0 -5 90) (size 1.8 1.8) (drill 1) (layers *.Cu *.Mask)
-      (net 18 "Net-(CUTOFF1-Pad3)") (pinfunction "3") (pintype "passive"))
+      (net 18 "Net-(R18-Pad2)") (pinfunction "3") (pintype "passive"))
     (model "${KICAD6_3DMODEL_DIR}/Potentiometer_THT.3dshapes/RK09K1130AH1.STEP"
       (offset (xyz 7 2.5 0))
@@
       (net 28 "/Cutoff") (pintype "passive"))
     (pad "2" thru_hole oval (at 10.16 0 180) (size 1.6 1.6) (drill 0.8) (layers *.Cu *.Mask)
-      (net 14 "Net-(CUTCV1-Pad2)") (pintype "passive"))
+      (net 14 "Net-(R14-Pad2)") (pintype "passive"))
     (model "${KICAD6_3DMODEL_DIR}/Resistor_THT.3dshapes/R_Axial_DIN0207_L6.3mm_D2.5mm_P10.16mm_Horizontal.wrl"
       (offset (xyz 0 0 0))
@@
       (net 28 "/Cutoff") (pintype "passive"))
     (pad "2" thru_hole oval (at 10.16 0 90) (size 1.6 1.6) (drill 0.8) (layers *.Cu *.Mask)
-      (net 17 "Net-(CUTOFF1-Pad2)") (pintype "passive"))
+      (net 17 "Net-(R15-Pad2)") (pintype "passive"))
     (model "${KICAD6_3DMODEL_DIR}/Resistor_THT.3dshapes/R_Axial_DIN0207_L6.3mm_D2.5mm_P10.16mm_Horizontal.wrl"
       (offset (xyz 0 0 0))
@@
     (fp_line (start 10.16 0) (end 8.23 0) (layer "F.Fab") (width 0.1))
     (pad "1" thru_hole circle (at 0 0 180) (size 1.6 1.6) (drill 0.8) (layers *.Cu *.Mask)
-      (net 18 "Net-(CUTOFF1-Pad3)") (pintype "passive"))
+      (net 16 "Net-(CUTOFF1-Pad1)") (pintype "passive"))
     (pad "2" thru_hole oval (at 10.16 0 180) (size 1.6 1.6) (drill 0.8) (layers *.Cu *.Mask)
       (net 2 "+12V") (pintype "passive"))
@@
       (net 3 "-12V") (pintype "passive"))
     (pad "2" thru_hole oval (at 10.16 0) (size 1.6 1.6) (drill 0.8) (layers *.Cu *.Mask)
-      (net 16 "Net-(CUTOFF1-Pad1)") (pintype "passive"))
+      (net 18 "Net-(R18-Pad2)") (pintype "passive"))
     (model "${KICAD6_3DMODEL_DIR}/Resistor_THT.3dshapes/R_Axial_DIN0207_L6.3mm_D2.5mm_P10.16mm_Horizontal.wrl"
       (offset (xyz 0 0 0))
@@
     (pad "" np_thru_hole circle (at 7 -6.9 90) (size 4 4) (drill 2) (layers *.Cu *.Mask))
     (pad "1" thru_hole circle (at 0 0 90) (size 1.8 1.8) (drill 1) (layers *.Cu *.Mask)
-      (net 1 "GND") (pinfunction "1") (pintype "passive"))
+      (net 39 "Net-(R21-Pad1)") (pinfunction "1") (pintype "passive"))
     (pad "2" thru_hole circle (at 0 -2.5 90) (size 1.8 1.8) (drill 1) (layers *.Cu *.Mask)
       (net 29 "/ResOut") (pinfunction "2") (pintype "passive"))
     (pad "3" thru_hole circle (at 0 -5 90) (size 1.8 1.8) (drill 1) (layers *.Cu *.Mask)
-      (net 39 "Net-(R21-Pad1)") (pinfunction "3") (pintype "passive"))
+      (net 1 "GND") (pinfunction "3") (pintype "passive"))
     (model "${KICAD6_3DMODEL_DIR}/Potentiometer_THT.3dshapes/RK09K1130AH1.STEP"
       (offset (xyz 7 2.5 0))
@@
     )
   )
+  (gr_line (start 30 25) (end 30 31) (layer "Dwgs.User") (width 0.05))
   (gr_line (start 42 110) (end 42 143) (layer "Dwgs.User") (width 0.1))
   (gr_line (start 85 36.5) (end 85 146.5) (layer "Edge.Cuts") (width 0.05))
@@
     (effects (font (size 1.5 1.5) (thickness 0.3)) (justify mirror))
   )
-  (gr_text "MS-20 VCF\nV1.0 BleepSound\n2022" (at 42 39.5) (layer "F.SilkS")
+  (gr_text "MS-20 VCF\nV1.1 BleepSound\n2022" (at 42 39.5) (layer "F.SilkS")
+    (effects (font (size 1 1) (thickness 0.15)))
+  )
+  (gr_text "12HP\n" (at 62 32.5) (layer "Dwgs.User")
     (effects (font (size 1 1) (thickness 0.15)))
   )
+  (dimension (type aligned) (layer "Dwgs.User")
+    (pts (xy 30 25) (xy 30 158))
+    (height 8)
+    (gr_text "133.0000 mm" (at 20.85 91.5 90) (layer "Dwgs.User")
+      (effects (font (size 1 1) (thickness 0.15)))
+    )
+    (format (units 2) (units_format 1) (precision 4))
+    (style (thickness 0.15) (arrow_length 1.27) (text_position_mode 0) (extension_height 0.58642) (extension_offset 0) keep_text_aligned)
+  )
+  (dimension (type aligned) (layer "Dwgs.User")
+    (pts (xy 33 31) (xy 33 25))
+    (height -6)
+    (gr_text "6.0000 mm" (at 25.85 28 90) (layer "Dwgs.User")
+      (effects (font (size 1 1) (thickness 0.15)))
+    )
+    (format (units 2) (units_format 1) (precision 4))
+    (style (thickness 0.15) (arrow_length 1.27) (text_position_mode 0) (extension_height 0.58642) (extension_offset 0) keep_text_aligned)
+  )
   (segment (start 56.219954 78.2) (end 56.195388 78.224566) (width 0.3) (layer "F.Cu") (net 2))
   (segment (start 76.9 132.32) (end 73.18 132.32) (width 0.3) (layer "F.Cu") (net 2))
@@
   (segment (start 40.75 121.8) (end 42 123.05) (width 0.3) (layer "F.Cu") (net 14))
   (segment (start 36.42 124.362233) (end 38.982233 121.8) (width 0.3) (layer "F.Cu") (net 14))
-  (segment (start 42 140.9) (end 44.5 138.4) (width 0.3) (layer "F.Cu") (net 15))
-  (segment (start 44.5 128.05) (end 39.5 123.05) (width 0.3) (layer "F.Cu") (net 15))
-  (segment (start 44.5 138.4) (end 44.5 128.05) (width 0.3) (layer "F.Cu") (net 15))
-  (segment (start 62.5 52.4) (end 54.4 44.3) (width 0.3) (layer "F.Cu") (net 16))
-  (segment (start 62.5 56.05) (end 62.5 52.4) (width 0.3) (layer "F.Cu") (net 16))
-  (segment (start 54.4 44.3) (end 50.56 44.3) (width 0.3) (layer "F.Cu") (net 16))
+  (segment (start 44.5 138.4) (end 42 140.9) (width 0.3) (layer "F.Cu") (net 15))
+  (segment (start 44.5 123.05) (end 44.5 138.4) (width 0.3) (layer "F.Cu") (net 15))
+  (segment (start 50.56 47.4) (end 52.5 49.34) (width 0.3) (layer "F.Cu") (net 16))
+  (segment (start 59.45 53) (end 62.5 56.05) (width 0.3) (layer "F.Cu") (net 16))
+  (segment (start 52.5 50) (end 55.5 53) (width 0.3) (layer "F.Cu") (net 16))
+  (segment (start 52.5 49.34) (end 52.5 50) (width 0.3) (layer "F.Cu") (net 16))
+  (segment (start 55.5 53) (end 59.45 53) (width 0.3) (layer "F.Cu") (net 16))
   (segment (start 68.3 49.14) (end 68.3 52.017767) (width 0.3) (layer "F.Cu") (net 17))
   (segment (start 68.3 52.017767) (end 62.717767 57.6) (width 0.3) (layer "F.Cu") (net 17))
   (segment (start 62.717767 57.6) (end 60.7 57.6) (width 0.3) (layer "F.Cu") (net 17))
-  (segment (start 60 56.9) (end 60 56.05) (width 0.3) (layer "F.Cu") (net 17))
-  (segment (start 60.7 57.6) (end 60 56.9) (width 0.3) (layer "F.Cu") (net 17))
-  (segment (start 57.5 54.34) (end 50.56 47.4) (width 0.3) (layer "F.Cu") (net 18))
-  (segment (start 57.5 56.05) (end 57.5 54.34) (width 0.3) (layer "F.Cu") (net 18))
+  (segment (start 60 56.05) (end 60 56.9) (width 0.3) (layer "F.Cu") (net 17))
+  (segment (start 60 56.9) (end 60.7 57.6) (width 0.3) (layer "F.Cu") (net 17))
+  (segment (start 52.5 46.24) (end 50.56 44.3) (width 0.3) (layer "B.Cu") (net 18))
+  (segment (start 52.5 51.05) (end 52.5 46.24) (width 0.3) (layer "B.Cu") (net 18))
+  (segment (start 57.5 56.05) (end 52.5 51.05) (width 0.3) (layer "B.Cu") (net 18))
   (segment (start 76.9 142.48) (end 81.255 142.48) (width 0.3) (layer "F.Cu") (net 19))
   (segment (start 81.255 142.48) (end 81.4 142.335) (width 0.3) (layer "F.Cu") (net 19))
@@
   (segment (start 46 75.860661) (end 46 71.5) (width 0.3) (layer "B.Cu") (net 38))
   (segment (start 46.774339 76.635) (end 46 75.860661) (width 0.3) (layer "B.Cu") (net 38))
-  (segment (start 57.5 99.05) (end 63.55 105.1) (width 0.3) (layer "F.Cu") (net 39))
   (segment (start 63.55 105.1) (end 64.58 105.1) (width 0.3) (layer "F.Cu") (net 39))
+  (segment (start 62.5 104.05) (end 63.55 105.1) (width 0.3) (layer "F.Cu") (net 39))
+  (segment (start 62.5 99.05) (end 62.5 104.05) (width 0.3) (layer "F.Cu") (net 39))
   (zone (net 1) (net_name "GND") (layer "F.Cu") (hatch edge 0.508)
     (connect_pads (clearance 0.508))
