File: ms20_vcf/simple/Kicad/MS20-VCF.kicad_pcb (KiCad board)
At the start: 2 copper layers, 118 x 128 mm, 59 parts, among them J5 Power Input, J6 FilterCV1, J7 FilterIn1, J8 FilterOut1, Q1 BC559, Q2 BC559, SW1 Hpass/Lpass Switch, U1 LM13700, U2 TL072

Commit message: fix issues on ms20 vcf
Parts:
- moved H1 0.50 mm to (111.0, 30.0)
- moved H2 0.50 mm to (145.0, 30.0)
Connections:
- CUTCV1 pad 1: GND -> /CVIn
- CUTCV1 pad 3: /CVIn -> GND
- CUTOFF1 pad 3: Net-(CUTOFF1-Pad3) -> Net-(R18-Pad2)
- R17 pad 1: Net-(CUTOFF1-Pad3) -> Net-(CUTOFF1-Pad1)
- R18 pad 2: Net-(CUTOFF1-Pad1) -> Net-(R18-Pad2)
- Res1 pad 1: GND -> Net-(R21-Pad1)
- Res1 pad 3: Net-(R21-Pad1) -> GND
Routing:
- net Net-(R18-Pad2): track 0.00 -> 14.6 mm
- net Net-(CUTOFF1-Pad3): track 11.5 -> 0.00 mm
- net Net-(CUTOFF1-Pad1): track 18.9 -> 15.9 mm
- net Net-(R21-Pad1): track 9.59 -> 7.51 mm
- net /CVIn: track 21.0 -> 18.9 mm
Other:
- board size 118 x 128 mm -> 118 x 128.5 mm
- board text added: "MS-20 VCF Face plate V1.1 BleepSound 2022"
- board text added: "MS-20 VCF V1.1 BleepSound 2022"
- board text removed: "MS-20 VCF Face plate V1.0 BleepSound 2022"
- board text removed: "MS-20 VCF V1.0 BleepSound 2022"
