File: ms20_vcf/simple/Kicad/MS20-VCF.kicad_sch (KiCad schematic)
At the start: 59 parts, among them J5 Power Input, J6 FilterCV1, J7 FilterIn1, J8 FilterOut1, Q1 BC559, Q2 BC559, SW1 Hpass/Lpass Switch, U1 LM13700, U2 TL072

Commit message: fix issues on ms20 vcf
Connections:
- net CVIn: now also CUTCV1.1; no longer CUTCV1.3
- net GND: now also CUTCV1.3, Res1.3; no longer CUTCV1.1, Res1.1
- net at R21.1: now also Res1.1; no longer Res1.3
- net at CUTOFF1.1: now also R17.1; no longer R18.2
- net at CUTOFF1.3: now also R18.2; no longer R17.1
Other:
- moved on the sheet: CUTCV1, CUTOFF1, Res1
Changed lines of the file:
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@@
     (pin "2")
   )
-  (symbol (lib_id "Device:R_POT") (at 236.22 81.28 180) (unit 1)
-    (in_bom yes) (on_board yes)
-    (property "Reference" "Res1" (id 0) (at 237.49 80.01 0)
-      (effects (font (size 1.27 1.27)) (justify right))
-    )
-    (property "Value" "100k" (id 1) (at 237.49 82.55 0)
+  (symbol (lib_id "Device:R_POT") (at 236.22 81.28 0) (mirror y) (unit 1)
+    (in_bom yes) (on_board yes)
+    (property "Reference" "Res1" (id 0) (at 237.49 82.55 0)
+      (effects (font (size 1.27 1.27)) (justify right))
+    )
+    (property "Value" "100k" (id 1) (at 237.49 80.01 0)
       (effects (font (size 1.27 1.27)) (justify right))
     )
@@
     (pin "2")
   )
-  (symbol (lib_id "Device:R_POT") (at 185.42 148.59 180) (unit 1)
-    (in_bom yes) (on_board yes)
-    (property "Reference" "CUTOFF1" (id 0) (at 186.69 147.32 0)
-      (effects (font (size 1.27 1.27)) (justify right))
-    )
-    (property "Value" "100k" (id 1) (at 186.69 149.86 0)
+  (symbol (lib_id "Device:R_POT") (at 185.42 148.59 0) (mirror y) (unit 1)
+    (in_bom yes) (on_board yes)
+    (property "Reference" "CUTOFF1" (id 0) (at 186.69 149.86 0)
+      (effects (font (size 1.27 1.27)) (justify right))
+    )
+    (property "Value" "100k" (id 1) (at 186.69 147.32 0)
       (effects (font (size 1.27 1.27)) (justify right))
     )
@@
     (pin "2")
   )
-  (symbol (lib_id "Device:R_POT") (at 167.64 123.19 180) (unit 1)
-    (in_bom yes) (on_board yes)
-    (property "Reference" "CUTCV1" (id 0) (at 168.91 121.92 0)
-      (effects (font (size 1.27 1.27)) (justify right))
-    )
-    (property "Value" "100k" (id 1) (at 168.91 124.46 0)
-      (effects (font (size 1.27 1.27)) (justify right))
-    )
+  (symbol (lib_id "Device:R_POT") (at 167.64 123.19 0) (mirror y) (unit 1)
+    (in_bom yes) (on_board yes)
+    (property "Reference" "CUTCV1" (id 0) (at 168.91 124.46 0)
+      (effects (font (size 1.27 1.27)) (justify right))
+    )
+    (property "Value" "100k" (id 1) (at 168.91 121.92 0)
+      (effects (font (size 1.27 1.27)) (justify right))
+    )
