File: ms20_vcf/double/Kicad/MS20-VCF.kicad_pcb (KiCad board)
At the start: 2 copper layers, 207 x 128 mm, 110 parts, among them J1 Conn_CircuitBoard, J10 Conn_CircuitBoard, J11 Conn_JackBoard, J12 Conn_JackBoard, J13 FilterCV2, J14 FilterIn2, J15 FilterOut2, J2 Conn_CircuitBoard, J3 Conn_JackBoard, J4 Conn_JackBoard, J5 Power Input, J6 FilterCV1, J7 FilterIn1, J8 FilterOut1, J9 Conn_CircuitBoard, Q1 BC559, Q2 BC559, Q3 BC559, Q4 BC559, SW1 Hpass/Lpass Switch, SW2 Bandpass, SW3 Hpass/Lpass Switch, U1 LM13700, U2 TL072, U3 LM13700, U4 TL072

Commit message: Auto stash before merge of "main" and "origin/main"
Parts:
- removed the J5 at (41.9, 93.2)
- added C11: 100nF, Capacitor_THT:C_Disc_D7.0mm_W2.5mm_P5.00mm, B.Cu at (47.6, 103.0)
- added C12: 100nF, Capacitor_THT:C_Disc_D7.0mm_W2.5mm_P5.00mm, B.Cu at (41.2, 79.1)
- added C13: 100nF, Capacitor_THT:C_Disc_D7.0mm_W2.5mm_P5.00mm, F.Cu at (82.0, 123.3)
- added C14: 100nF, Capacitor_THT:C_Disc_D7.0mm_W2.5mm_P5.00mm, F.Cu at (80.6, 73.5)
- added C6: 100nF, Capacitor_THT:C_Disc_D7.0mm_W2.5mm_P5.00mm, F.Cu at (84.6, 109.4)
- added C9: 100nF, Capacitor_THT:C_Disc_D7.0mm_W2.5mm_P5.00mm, F.Cu at (83.2, 59.5)
- added J8: Power Input, Connector_IDC:IDC-Header_2x05_P2.54mm_Vertical, B.Cu at (50.1, 92.1)
- C7, C8: value 0.1µ -> 100nF; footprint Capacitor_THT:CP_Radial_D5.0mm_P2.00mm -> Capacitor_THT:C_Disc_D7.0mm_W2.5mm_P5.00mm
- FB1, FB2: footprint Inductor_THT:L_Axial_L9.5mm_D4.0mm_P12.70mm_Horizontal_Fastron_SMCC -> Inductor_THT:L_Axial_L7.0mm_D3.3mm_P10.16mm_Horizontal_Fastron_MICC
- Q1, Q2, Q3, Q4: footprint Package_TO_SOT_THT:TO-92_Inline -> Package_TO_SOT_THT:TO-92_Inline_Wide
- ResLv1, ResLv2, ResVol1, ResVol2: footprint Potentiometer_THT:Potentiometer_Bourns_3386C_Horizontal -> Potentiometer_THT:Potentiometer_Bourns_3386X_Horizontal
- U1, U3: footprint Package_DIP:DIP-16_W7.62mm_Socket -> Package_SO:SOIC-16_3.9x9.9mm_P1.27mm; moved to B.Cu
- moved C5 34.9 mm to (32.9, 98.5), turned to -90 degrees
- moved R10 31.5 mm to (33.4, 46.0)
- moved R5 31.5 mm to (36.5, 46.0)
- moved C8 31.3 mm to (51.8, 74.1), turned to -90 degrees
- moved FB1 30.8 mm to (32.3, 95.5), turned to 90 degrees
- moved R33 27.8 mm to (33.9, 114.4)
- moved R25 26.5 mm to (38.3, 122.6)
- moved R26 21.3 mm to (60.0, 120.6)
- moved C18 19.4 mm to (87.8, 113.8), turned to -90 degrees
- moved R23 19.2 mm to (44.5, 112.4)
- moved R28 18.9 mm to (41.4, 122.6)
- moved D1 18.0 mm to (83.2, 56.8), turned to 90 degrees
- moved C1 17.3 mm to (36.6, 76.6)
- moved R24 15.8 mm to (56.9, 110.4), turned to -90 degrees
- moved C7 15.1 mm to (37.0, 108.0), turned to 90 degrees
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- renumbered C6 to C1, C3 to C10, C14 to C15, C11 to C16, C13 to C17, C12 to C18, C1 to C2, C5 to C3, C2 to C5, D2 to D1, D12 to D10, D9 to D11, D11 to D12, D4 to D2, D6 to D3, D3 to D4, D7 to D6, D1 to D7, D10 to D9, J6 to J1, J11 to J10, J13 to J11, J15 to J12, J10 to J13, J12 to J14, J14 to J15, J8 to J2, J1 to J3, J3 to J4, J7 to J5, J2 to J6, J4 to J7, R6 to R1, R3 to R10, R13 to R11, R21 to R12, R20 to R13, R5 to R14, R8 to R15, R14 to R16, R7 to R17, R9 to R18, R17 to R19, R16 to R2, R15 to R20, R18 to R21, R4 to R22, R27 to R23, R37 to R24, R23 to R25, R33 to R26, R24 to R27, R32 to R28, R40 to R29, R1 to R3, R43 to R30, R25 to R32, R34 to R33, R42 to R34, R41 to R35, R26 to R36, R29 to R37, R35 to R38, R28 to R39, R12 to R4, R30 to R40, R38 to R41, R36 to R42, R39 to R43, R2 to R5, R11 to R6, R19 to R7, R22 to R8, R10 to R9
Connections:
- C8 pad 1: GND -> +12V
- C8 pad 2: -12V -> GND
Routing:
- net -12V: track 267.1 -> 133.6 mm, vias 2 -> 0
- net +12V: track 281.3 -> 183.0 mm, vias 1 -> 0
- net Net-(C1-Pad2): track 56.7 -> 0.00 mm
- net Net-(C2-Pad2): track 54.8 -> 0.00 mm
- net Net-(C4-Pad2): track 44.5 -> 0.00 mm
- net /Cutoff: track 78.6 -> 36.6 mm
- net Net-(D3-Pad1): track 37.6 -> 0.00 mm
- net Net-(R2-Pad1): track 35.3 -> 0.00 mm
- net Net-(R23-Pad2): track 46.3 -> 18.2 mm
- net Net-(C2-Pad1): track 26.4 -> 0.00 mm
- net Net-(R11-Pad2): track 26.3 -> 0.00 mm
- net Net-(R1-Pad2): track 24.2 -> 0.00 mm
- net Net-(C16-Pad1): track 35.1 -> 10.9 mm
- net /Out1: track 58.3 -> 37.5 mm
- net Net-(C4-Pad1): track 19.4 -> 0.00 mm
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Other:
- board text added: "Double MS-20 VCF V1.2 BleepSound 2022"
- board text removed: "Double MS-20 VCF V1.1 BleepSound 2022"

Commit message: updates front panel designs and gerbers before order
Parts:
- moved C2 23.3 mm to (56.5, 62.5)
- moved R18 23.1 mm to (51.2, 82.8)
- moved R4 22.3 mm to (66.5, 65.6)
- moved C3 22.0 mm to (37.4, 81.2), turned to 90 degrees
- moved R2 22.0 mm to (56.3, 68.7)
- moved R5 20.3 mm to (31.3, 65.6), turned to 0 degrees
- moved R10 16.6 mm to (31.3, 62.5), turned to 0 degrees
- moved R17 14.0 mm to (67.3, 82.5)
- moved R1 11.1 mm to (43.8, 65.6), turned to 0 degrees
- moved Q2 10.9 mm to (71.8, 81.3), turned to 90 degrees
- moved R7 10.1 mm to (64.2, 82.5), turned to 90 degrees
- moved R3 9.54 mm to (54.0, 68.7), turned to 180 degrees
- moved R6 9.36 mm to (58.0, 72.3), turned to -90 degrees
- moved R15 9.30 mm to (72.3, 72.2)
- moved R11 6.66 mm to (54.0, 62.5)
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Connections:
- CUTCV1 pad 1: GND -> /CVIn
- CUTCV1 pad 3: /CVIn -> GND
- CUTCV2 pad 1: GND -> /Filtre2/CVIn
- CUTCV2 pad 3: /Filtre2/CVIn -> GND
- CUTOFF1 pad 3: Net-(CUTOFF1-Pad3) -> Net-(R21-Pad2)
- R19 pad 1: Net-(CUTOFF1-Pad3) -> Net-(CUTOFF1-Pad1)
- R21 pad 2: Net-(CUTOFF1-Pad1) -> Net-(R21-Pad2)
- R41 pad 1: Net-(CUTOFF2-Pad3) -> Net-(CUTOFF2-Pad1)
- R43 pad 2: Net-(CUTOFF2-Pad1) -> Net-(CUTOFF2-Pad3)
- Res1 pad 1: GND -> Net-(R12-Pad1)
- Res1 pad 3: Net-(R12-Pad1) -> GND
- Res2 pad 1: GND -> Net-(R34-Pad1)
- Res2 pad 3: Net-(R34-Pad1) -> GND
Routing:
- net +12V: track 183.0 -> 268.3 mm, vias 0 -> 2
- net -12V: track 133.6 -> 214.1 mm
- net /Cutoff: track 36.6 -> 81.5 mm, vias 0 -> 1
- net Net-(C2-Pad2): track 0.00 -> 43.5 mm
- net Net-(D3-Pad1): track 0.00 -> 38.4 mm
- net Net-(C1-Pad2): track 0.00 -> 33.7 mm, vias 0 -> 1
- net Net-(C4-Pad2): track 0.00 -> 33.3 mm
- net Net-(R11-Pad2): track 0.00 -> 29.4 mm, vias 0 -> 1
- net Net-(C2-Pad1): track 0.00 -> 28.8 mm
- net Net-(R1-Pad2): track 0.00 -> 27.8 mm
- net Net-(R2-Pad1): track 0.00 -> 26.2 mm, vias 0 -> 1
- net Net-(Q1-Pad1): track 0.00 -> 22.8 mm
- net Net-(R21-Pad2): track 0.00 -> 19.0 mm
- net Net-(C3-Pad1): track 0.00 -> 18.9 mm, vias 0 -> 1
- net Net-(C4-Pad1): track 0.00 -> 18.9 mm
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Other:
- board size 207 x 128 mm -> 207 x 128.5 mm
- board text added: "Front"
- board text removed: "Double MS-20 VCF V1.0 BleepSound 2022"
