File: ms20_vcf/double/Kicad/MS20-VCF.kicad_sch (KiCad schematic)
At the start: 62 parts, among them J1 Conn_CircuitBoard, J2 Conn_CircuitBoard, J3 Conn_JackBoard, J4 Conn_JackBoard, J5 Power Input, J6 FilterCV1, J7 FilterIn1, J8 FilterOut1, Q1 BC559, Q2 BC559, SW1 Hpass/Lpass Switch, SW2 Bandpass, U1 LM13700, U2 TL072

Commit message: Auto stash before merge of "main" and "origin/main"
Parts:
- removed C7, C8: 0.1µ, Capacitor_THT:CP_Radial_D5.0mm_P2.00mm, symbol Device:CP1_Small
- removed J5: Power Input, Connector_PinHeader_2.54mm:PinHeader_2x05_P2.54mm_Vertical, symbol Connector:Conn_01x10_Male
- added C11, C12, C13, C14, C6, C7, C8, C9: 100nF, Capacitor_THT:C_Disc_D7.0mm_W2.5mm_P5.00mm, symbol Device:C_Small
- added J8: Power Input, Connector_IDC:IDC-Header_2x05_P2.54mm_Vertical, symbol Connector:Conn_01x10_Male
- FB1, FB2: footprint Inductor_THT:L_Axial_L9.5mm_D4.0mm_P12.70mm_Horizontal_Fastron_SMCC -> Inductor_THT:L_Axial_L7.0mm_D3.3mm_P10.16mm_Horizontal_Fastron_MICC
- Q1, Q2: footprint Package_TO_SOT_THT:TO-92_Inline -> Package_TO_SOT_THT:TO-92_Inline_Wide
- ResLv1, ResVol1: footprint Potentiometer_THT:Potentiometer_Bourns_3386C_Horizontal -> Potentiometer_THT:Potentiometer_Bourns_3386X_Horizontal
- U1: footprint Package_DIP:DIP-16_W7.62mm_Socket -> Package_SO:SOIC-16_3.9x9.9mm_P1.27mm
- renumbered C6 to C1, C3 to C10, C1 to C2, C5 to C3, C2 to C5, D2 to D1, D4 to D2, D6 to D3, D3 to D4, D7 to D6, D1 to D7, J6 to J1, J8 to J2, J1 to J3, J3 to J4, J7 to J5, J2 to J6, J4 to J7, R6 to R1, R3 to R10, R13 to R11, R21 to R12, R20 to R13, R5 to R14, R8 to R15, R14 to R16, R7 to R17, R9 to R18, R17 to R19, R16 to R2, R15 to R20, R18 to R21, R4 to R22, R1 to R3, R12 to R4, R2 to R5, R11 to R6, R19 to R7, R22 to R8, R10 to R9
Connections:
- net +12V: now also C6.1, C7.1, C8.1, C9.1
- net -12V: now also C11.2, C12.2, C13.2, C14.2
- net GND: now also C11.1, C12.1, C13.1, C14.1, C6.2, C7.2, C8.2, C9.2, J8.3 (Pin_3), J8.4 (Pin_4), J8.5 (Pin_5), J8.6 (Pin_6), J8.7 (Pin_7), J8.8 (Pin_8)
- net at FB1.2: now also J8.10 (Pin_10), J8.9 (Pin_9)
- net at FB2.2: now also J8.1 (Pin_1), J8.2 (Pin_2)
Other:
- moved on the sheet: C10, C5, D7, FB1, FB2, R22, U1E, U2C

Commit message: updates front panel designs and gerbers before order
Connections:
- net CVIn: now also CUTCV1.1; no longer CUTCV1.3
- net GND: now also CUTCV1.3, Res1.3; no longer CUTCV1.1, Res1.1
- net at R12.1: now also Res1.1; no longer Res1.3
- net at CUTOFF1.1: now also R19.1; no longer R21.2
- net at CUTOFF1.3: now also R21.2; no longer R19.1
Other:
- moved on the sheet: CUTCV1, CUTOFF1, Res1
Changed lines of the file:
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@@
     (pin "2")
   )
-  (symbol (lib_id "Device:R_POT") (at 236.22 81.28 180) (unit 1)
-    (in_bom yes) (on_board yes)
-    (property "Reference" "Res1" (id 0) (at 237.49 80.01 0)
-      (effects (font (size 1.27 1.27)) (justify right))
-    )
-    (property "Value" "100k" (id 1) (at 237.49 82.55 0)
+  (symbol (lib_id "Device:R_POT") (at 236.22 81.28 0) (mirror y) (unit 1)
+    (in_bom yes) (on_board yes)
+    (property "Reference" "Res1" (id 0) (at 237.49 82.55 0)
+      (effects (font (size 1.27 1.27)) (justify right))
+    )
+    (property "Value" "100k" (id 1) (at 237.49 80.01 0)
       (effects (font (size 1.27 1.27)) (justify right))
     )
@@
     (pin "2")
   )
-  (symbol (lib_id "Device:R_POT") (at 182.88 146.05 180) (unit 1)
-    (in_bom yes) (on_board yes)
-    (property "Reference" "CUTOFF1" (id 0) (at 184.15 144.78 0)
-      (effects (font (size 1.27 1.27)) (justify right))
-    )
-    (property "Value" "100k" (id 1) (at 184.15 147.32 0)
+  (symbol (lib_id "Device:R_POT") (at 182.88 146.05 0) (mirror y) (unit 1)
+    (in_bom yes) (on_board yes)
+    (property "Reference" "CUTOFF1" (id 0) (at 184.15 147.32 0)
+      (effects (font (size 1.27 1.27)) (justify right))
+    )
+    (property "Value" "100k" (id 1) (at 184.15 144.78 0)
       (effects (font (size 1.27 1.27)) (justify right))
     )
@@
     (pin "2")
   )
-  (symbol (lib_id "Device:R_POT") (at 166.37 123.19 180) (unit 1)
-    (in_bom yes) (on_board yes)
-    (property "Reference" "CUTCV1" (id 0) (at 167.64 121.92 0)
-      (effects (font (size 1.27 1.27)) (justify right))
-    )
-    (property "Value" "100k" (id 1) (at 167.64 124.46 0)
-      (effects (font (size 1.27 1.27)) (justify right))
-    )
+  (symbol (lib_id "Device:R_POT") (at 166.37 123.19 0) (mirror y) (unit 1)
+    (in_bom yes) (on_board yes)
+    (property "Reference" "CUTCV1" (id 0) (at 167.64 124.46 0)
+      (effects (font (size 1.27 1.27)) (justify right))
+    )
+    (property "Value" "100k" (id 1) (at 167.64 121.92 0)
+      (effects (font (size 1.27 1.27)) (justify right))
+    )
